File: communication-hub/communication-hub.kicad_pcb (KiCad board)
At the start: 2 copper layers, 82.6 x 54 mm, 50 parts, among them CON1 SM04B-GHS-TB, CON2 SM04B-GHS-TB, CON3 SM02B-GHS-TB, CON4 SM04B-GHS-TB, CON5 SM04B-GHS-TB, Q1 DMN5L06K, Q2 DMN5L06K, U1 TCAN1042HVDR, U2 TCAN1042HVDR

Commit message: Fixed some potential issues with TCAN/MCP parts
Parts:
- removed C1, C2: 10u, communication-hub:C0805
Connections:
- U1 pad 5: +3V3 -> Net-(U1-Pad5)
- U2 pad 5: +3V3 -> Net-(U2-Pad5)
Routing:
- net +3V3: track 131.7 -> 127.5 mm, vias 2 -> 1
