File: communication-hub/communication-hub.brd (EAGLE design)
At the start: 51.7 x 30.5 mm, 7 parts

Commit message: routed everything
Routing:
- net CAN_H: track 0.00 -> 22.7 mm, vias 0 -> 2
- net CAN_L: track 0.00 -> 22.7 mm, vias 0 -> 2
- net N$4: track 0.00 -> 18.1 mm
- net CAN_TXD: track 0.00 -> 17.5 mm
- net +3V3: track 0.00 -> 17.4 mm, vias 0 -> 2
- net CAN_RXD: track 0.00 -> 15.0 mm
- net GND: track 5.93 -> 18.5 mm, vias 0 -> 4
- net N$3: track 0.00 -> 11.4 mm
- net +5V: track 39.9 -> 48.3 mm
- added copper zone on layer 1, net GND
- added copper zone on layer 16, net GND
Other:
- board text added: "Communications Hub Revision"
- board text added: "Jack Opgenorth"
- board text added: "SPEAR"

Commit message: Larger CAN traces + removed useless ground
Routing:
- net GND: track 18.5 -> 11.7 mm, vias 4 -> 2
Changed lines of the file:
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@@
 <wire x1="79.673" y1="22.098" x2="77.089" y2="22.098" width="0.3048" layer="1"/>
 <wire x1="85.3" y1="23.495" x2="88.265" y2="23.495" width="0.1524" layer="1"/>
-<via x="89.281" y="17.907" extent="1-16" drill="0.35"/>
-<via x="96.012" y="6.223" extent="1-16" drill="0.35"/>
-<wire x1="92.71" y1="6.35" x2="95.885" y2="6.35" width="0.508" layer="1"/>
-<wire x1="95.885" y1="6.35" x2="96.012" y2="6.223" width="0.508" layer="1"/>
-<wire x1="92.71" y1="17.78" x2="89.408" y2="17.78" width="0.508" layer="1"/>
-<wire x1="89.408" y1="17.78" x2="89.281" y2="17.907" width="0.508" layer="1"/>
 <polygon width="0.1524" layer="16">
 <vertex x="49.53" y="29.21"/>
@@
 <contactref element="U$1" pad="7"/>
 <contactref element="JP3" pad="2"/>
-<wire x1="92.71" y1="22.86" x2="92.075" y2="22.225" width="0.1524" layer="1"/>
-<wire x1="92.075" y1="22.225" x2="86.614" y2="22.225" width="0.1524" layer="1"/>
+<wire x1="92.71" y1="22.86" x2="92.075" y2="22.225" width="0.381" layer="1"/>
+<wire x1="92.075" y1="22.225" x2="86.614" y2="22.225" width="0.381" layer="1"/>
 <via x="87.63" y="21.209" extent="1-16" drill="0.35"/>
 <via x="90.424" y="11.303" extent="1-16" drill="0.35"/>
-<wire x1="86.614" y1="22.225" x2="85.3" y2="22.225" width="0.1524" layer="1"/>
+<wire x1="86.614" y1="22.225" x2="85.3" y2="22.225" width="0.381" layer="1"/>
 <wire x1="92.71" y1="11.43" x2="92.583" y2="11.303" width="0.1524" layer="1"/>
-<wire x1="92.583" y1="11.303" x2="90.424" y2="11.303" width="0.1524" layer="1"/>
-<wire x1="87.63" y1="21.209" x2="86.614" y2="22.225" width="0.1524" layer="1"/>
-<wire x1="90.424" y1="11.303" x2="90.17" y2="11.557" width="0.1524" layer="16"/>
-<wire x1="90.17" y1="11.557" x2="90.17" y2="19.05" width="0.1524" layer="16"/>
-<wire x1="90.17" y1="19.05" x2="88.011" y2="21.209" width="0.1524" layer="16"/>
-<wire x1="88.011" y1="21.209" x2="87.63" y2="21.209" width="0.1524" layer="16"/>
+<wire x1="92.583" y1="11.303" x2="90.424" y2="11.303" width="0.381" layer="1"/>
+<wire x1="87.63" y1="21.209" x2="86.614" y2="22.225" width="0.381" layer="1"/>
+<wire x1="90.424" y1="11.303" x2="90.17" y2="11.557" width="0.381" layer="16"/>
+<wire x1="90.17" y1="11.557" x2="90.17" y2="19.05" width="0.381" layer="16"/>
+<wire x1="90.17" y1="19.05" x2="88.011" y2="21.209" width="0.381" layer="16"/>
+<wire x1="88.011" y1="21.209" x2="87.63" y2="21.209" width="0.381" layer="16"/>
 </signal>
 <signal name="N$3">
@@
 <contactref element="JP1" pad="3"/>
 <contactref element="U$1" pad="6"/>
-<wire x1="92.71" y1="20.32" x2="87.63" y2="20.32" width="0.1524" layer="1"/>
-<wire x1="87.63" y1="20.32" x2="85.935" y2="20.32" width="0.1524" layer="1"/>
-<wire x1="85.935" y1="20.32" x2="85.3" y2="20.955" width="0.1524" layer="1"/>
+<wire x1="92.71" y1="20.32" x2="87.63" y2="20.32" width="0.381" layer="1"/>
 <via x="90.17" y="8.89" extent="1-16" drill="0.35"/>
 <via x="88.265" y="16.51" extent="1-16" drill="0.35"/>
-<wire x1="90.17" y1="8.89" x2="88.265" y2="10.795" width="0.1524" layer="16"/>
-<wire x1="88.265" y1="10.795" x2="88.265" y2="16.51" width="0.1524" layer="16"/>
-<wire x1="88.265" y1="16.51" x2="88.265" y2="19.685" width="0.1524" layer="1"/>
-<wire x1="88.265" y1="19.685" x2="87.63" y2="20.32" width="0.1524" layer="1"/>
-<wire x1="90.17" y1="8.89" x2="92.71" y2="8.89" width="0.1524" layer="1"/>
+<wire x1="90.17" y1="8.89" x2="88.265" y2="10.795" width="0.381" layer="16"/>
+<wire x1="88.265" y1="10.795" x2="88.265" y2="16.51" width="0.381" layer="16"/>
+<wire x1="88.265" y1="16.51" x2="88.265" y2="19.685" width="0.381" layer="1"/>
+<wire x1="88.265" y1="19.685" x2="87.63" y2="20.32" width="0.381" layer="1"/>
+<wire x1="90.17" y1="8.89" x2="92.71" y2="8.89" width="0.381" layer="1"/>
+<wire x1="86.36" y1="20.32" x2="87.63" y2="20.32" width="0.381" layer="1"/>
+<wire x1="85.3" y1="20.955" x2="85.725" y2="20.955" width="0.381" layer="1"/>
+<wire x1="85.725" y1="20.955" x2="86.36" y2="20.32" width="0.381" layer="1"/>
 </signal>
 </signals>
