File: can_termination/can_termination.kicad_pcb (KiCad board)
At the start: 2 copper layers, 82 x 22 mm, 15 parts, among them J101 Conn_01x04_Male, J102 Conn_01x04_Male, J103 Conn_01x04_Male, J104 Conn_01x04_Male, J105 Conn_01x04_Male, J106 Conn_01x04_Male

Commit message: Added SPEAR logo.
Parts:
- added G***: LOGO, logos:spear_logo_12.7x12.7mm, B.Cu at (85.2, 80.2)
