File: can_indication/indication.sch (EAGLE design)
At the start: 1 part

Commit message: Added Cree RGB LED and PCA9685 to library.
Parts:
- added D1, D2, D3, D4, D5, D6, D7, D8: CLV1L-FKB-CHMMQEHBB7673673, SPEAR:CLV1L-FKB-CHMMQEHBB7673673
Changed lines of the file:
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@@
 <parts>
 <part name="U$1" library="SPEAR" deviceset="MCP2562-E/SN" device=""/>
+<part name="D1" library="SPEAR" deviceset="CLV1L-FKB-CHMMQEHBB7673673" device=""/>
+<part name="D2" library="SPEAR" deviceset="CLV1L-FKB-CHMMQEHBB7673673" device=""/>
+<part name="D3" library="SPEAR" deviceset="CLV1L-FKB-CHMMQEHBB7673673" device=""/>
+<part name="D4" library="SPEAR" deviceset="CLV1L-FKB-CHMMQEHBB7673673" device=""/>
+<part name="D5" library="SPEAR" deviceset="CLV1L-FKB-CHMMQEHBB7673673" device=""/>
+<part name="D6" library="SPEAR" deviceset="CLV1L-FKB-CHMMQEHBB7673673" device=""/>
+<part name="D7" library="SPEAR" deviceset="CLV1L-FKB-CHMMQEHBB7673673" device=""/>
+<part name="D8" library="SPEAR" deviceset="CLV1L-FKB-CHMMQEHBB7673673" device=""/>
 </parts>
 <sheets>
@@
 <instances>
 <instance part="U$1" gate="G$1" x="10.16" y="-5.08"/>
+<instance part="D1" gate="G$1" x="116.84" y="33.02"/>
+<instance part="D2" gate="G$1" x="137.16" y="33.02"/>
+<instance part="D3" gate="G$1" x="157.48" y="33.02"/>
+<instance part="D4" gate="G$1" x="175.26" y="33.02"/>
+<instance part="D5" gate="G$1" x="114.3" y="-17.78"/>
+<instance part="D6" gate="G$1" x="134.62" y="-17.78"/>
+<instance part="D7" gate="G$1" x="154.94" y="-17.78"/>
+<instance part="D8" gate="G$1" x="177.8" y="-17.78"/>
 </instances>
 <busses>

Commit message: Added STM32F103CB device.
Parts:
- added U$2, U$3: PCA9685PW, SPEAR:PCA9685PW
- added U1: STM32F103CB, SPEAR:STM32F103CB
Connections:
- new net +3V3: U1_PWR.VDDA, U1_PWR.VDD_1, U1_PWR.VDD_2, U1_PWR.VDD_3
- new net +5V: D1.AN, D2.AN, D3.AN, D4.AN, D5.AN, D6.AN, D7.AN, D8.AN
- new net BOOT0: U1_PWR.BOOT0
- new net GND: U1_PWR.VSSA, U1_PWR.VSS_1, U1_PWR.VSS_2, U1_PWR.VSS_3
- new net LEDA0: D1.R, U$2.LED0
- new net LEDA1: D1.G, U$2.LED1
- new net LEDA10: D3.B, U$2.LED10
- new net LEDA11: U$2.LED11
- new net LEDA12: D4.R, U$2.LED12
- new net LEDA13: D4.G, U$2.LED13
- new net LEDA14: D4.B, U$2.LED14
- new net LEDA15: U$2.LED15
- new net LEDA2: D1.B, U$2.LED2
- new net LEDA3: U$2.LED3
- new net LEDA4: D2.R, U$2.LED4
- new net LEDA5: D2.G, U$2.LED5
- new net LEDA6: D2.B, U$2.LED6
- new net LEDA7: U$2.LED7
- new net LEDA8: D3.R, U$2.LED8
- new net LEDA9: D3.G, U$2.LED9
- new net LEDB0: D5.R, U$3.LED0
- new net LEDB1: D5.G, U$3.LED1
- new net LEDB10: D7.B, U$3.LED10
- new net LEDB11: U$3.LED11
- new net LEDB12: D8.R, U$3.LED12
- new net LEDB13: D8.G, U$3.LED13
- new net LEDB14: D8.B, U$3.LED14
- new net LEDB15: U$3.LED15
- new net LEDB2: D5.B, U$3.LED2
- new net LEDB3: U$3.LED3
- new net LEDB4: D6.R, U$3.LED4
- new net LEDB5: D6.G, U$3.LED5
- new net LEDB6: D6.B, U$3.LED6
- new net LEDB7: U$3.LED7
- new net LEDB8: D7.R, U$3.LED8
- new net LEDB9: D7.G, U$3.LED9
- new net NRST: U1_PWR.NRST
Other:
- moved on the sheet: D1, D2, D3, D4, D5, D6, D7, D8

Commit message: Made more progress. Schematic mostly done.
Parts:
- added C1, C2, C3, C4, C5: 100n, resistor:C-EUC0805
- added C6: 4u7, resistor:C-EUC0805
- added C7: 10n, resistor:C-EUC0805
- added C8: 1u, resistor:C-EUC0805
- added CON1, CON2: SM04B-GHS-TB, ARVP:SM04B-GHS-TB
- added R1, R10, R13, R16, R19, R22, R4, R7: 66, resistor:R-EU_R0805
- added R11, R12, R14, R15, R17, R18, R2, R20, R21, R23, R24, R3, R5, R6, R8, R9: 10, resistor:R-EU_R0805
- added R25: 10K, resistor:R-EU_R0805
- added R26, R27, R28: 10k, resistor:R-EU_R0805
- added U$4: TE-CONN_5-103669-1, SPEAR:TE-CONN_5-103669-1
Connections:
- new net CANH: CON1-2.S, CON2-2.S, U$1.CANH
- new net CANL: CON1-3.S, CON2-3.S, U$1.CANL
- new net CAN_STBY: U$1.STBY, U1_PORTA.PA10
- new net I2C_SCL: R27.1, U$2.SCL, U$3.SCL, U1_PORTB.PB6
- new net I2C_SDA: R28.1, U$2.SDA, U$3.SDA, U1_PORTB.PB7
- new net LED_!OE: R26.1, U$2.!OE, U1_PORTB.PB5
- new net LED_~OE: U$3.!OE
- new net N$1: D5.R, R1.2
- new net N$10: D8.R, R10.2
- new net N$11: D8.G, R11.2
- new net N$12: D8.B, R12.2
- new net N$13: D1.R, R13.2
- new net N$14: D1.G, R14.2
- new net N$15: D1.B, R15.2
- new net N$16: D2.R, R16.2
- new net N$17: D2.G, R17.2
- new net N$18: D2.B, R18.2
- new net N$19: D3.R, R19.2
- new net N$2: D5.G, R2.2
- new net N$20: D3.G, R20.2
- new net N$21: D3.B, R21.2
- new net N$22: D4.R, R22.2
- new net N$23: D4.G, R23.2
- new net N$24: D4.B, R24.2
- new net N$27: R25.2, U$3.A0
- new net N$3: D5.B, R3.2
- new net N$4: D6.R, R4.2
- new net N$5: D6.G, R5.2
- new net N$6: D6.B, R6.2
- new net N$7: D7.R, R7.2
- new net N$8: D7.G, R8.2
- new net N$9: D7.B, R9.2
- new net STM_CANRX: U$1.RXD, U1_PORTA.PA11
- new net STM_CANTX: U$1.TXD, U1_PORTA.PA12
- new net SWCLK: U1_PORTA.PA14
- new net SWDIO: U1_PORTA.PA13
- net +3V3: now also C1.1, C2.1, C3.1, C4.1, C5.1, C6.1, C7.1, C8.1, D1.AN, D2.AN, D3.AN, D4.AN, D5.AN, D6.AN, D7.AN, D8.AN, R25.1, R26.2, R27.2, R28.2, U$1.VIO, U$2.VDD, U$3.VDD, U$4.1
- net +5V: now also CON1-1.S, CON2-1.S, U$1.VDD; no longer D1.AN, D2.AN, D3.AN, D4.AN, D5.AN, D6.AN, D7.AN, D8.AN
- net GND: now also C1.2, C2.2, C3.2, C4.2, C5.2, C6.2, C7.2, C8.2, CON1-4.S, CON1-TABS.S, CON2-4.S, CON2-TABS.S, U$1.VSS, U$2.A0, U$2.A1, U$2.A2, U$2.A3, U$2.A4, U$2.A5, U$2.VSS, U$3.A1, U$3.A2, U$3.A3, U$3.A4, U$3.A5, U$3.VSS, U$4.2
- net LEDA0: now also R13.1; no longer D1.R
- net LEDA1: now also R14.1; no longer D1.G
- net LEDA10: now also R21.1; no longer D3.B
- net LEDA12: now also R22.1; no longer D4.R
- net LEDA13: now also R23.1; no longer D4.G
- net LEDA14: now also R24.1; no longer D4.B
- net LEDA2: now also R15.1; no longer D1.B
- net LEDA4: now also R16.1; no longer D2.R
- net LEDA5: now also R17.1; no longer D2.G
- net LEDA6: now also R18.1; no longer D2.B
- net LEDA8: now also R19.1; no longer D3.R
- net LEDA9: now also R20.1; no longer D3.G
- net LEDB0: now also R1.1; no longer D5.R
- net LEDB1: now also R2.1; no longer D5.G
- net LEDB10: now also R9.1; no longer D7.B
- net LEDB12: now also R10.1; no longer D8.R
- net LEDB13: now also R11.1; no longer D8.G
- net LEDB14: now also R12.1; no longer D8.B
- net LEDB2: now also R3.1; no longer D5.B
- net LEDB4: now also R4.1; no longer D6.R
- net LEDB5: now also R5.1; no longer D6.G
- net LEDB6: now also R6.1; no longer D6.B
- net LEDB8: now also R7.1; no longer D7.R
- net LEDB9: now also R8.1; no longer D7.G
Other:
- note added: "4.7uF Capacitor must be connected to VDD_3"
- note added: "Analog Supply Decoupling"
- note added: "Digital Supply Decoupling"
- note added: "Pullup Resistors"
- moved on the sheet: D1, D2, D3, D4, D5, D6, D7, D8, U$1
