File: can_indication/indication.sch (EAGLE design)
At the start: 51 parts, among them CON1 SM04B-GHS-TB, CON2 SM04B-GHS-TB, U1 STM32F103CB

Commit message: Fixed some footprint issues and most of positioning.
I botched a few footprints so I had to fix them :/
Other:
- note added: "PIN 1"
- note added: "Pin 26"
- note added: "Pin 35"
- moved on the sheet: U1_PWR

Commit message: Finished a lot of routing.
Most of the PCA9685 stuff is routed.

Todo:
- Add programming header.
- Route everything else.
- Add planes.
Connections:
- removed net LED_~OE: U$3.!OE
- net LED_!OE: now also U$3.!OE
Changed lines of the file:
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@@
 <label x="-93.98" y="27.94" size="1.778" layer="95"/>
+</segment>
+<segment>
+<pinref part="U$3" gate="G$1" pin="!OE"/>
+<wire x1="55.88" y1="-15.24" x2="48.26" y2="-15.24" width="0.1524" layer="91"/>
+<label x="43.18" y="-15.24" size="1.778" layer="95"/>
 </segment>
 </net>
@@
 </segment>
 </net>
-<net name="LED_~OE" class="0">
-<segment>
-<pinref part="U$3" gate="G$1" pin="!OE"/>
-<wire x1="55.88" y1="-15.24" x2="48.26" y2="-15.24" width="0.1524" layer="91"/>
-<label x="43.18" y="-15.24" size="1.778" layer="95"/>
-</segment>
-</net>

Commit message: Changed the indication board so it uses higher power LED's now
Parts:
- removed D1, D2, D3, D4, D5, D6, D7, D8: CLV1L-FKB-CHMMQEHBB7673673, SPEAR:CLV1L-FKB-CHMMQEHBB7673673
- removed R11, R12, R14, R15, R17, R18, R20, R21, R23, R24, R5, R6, R8, R9: 10, resistor:R-EU_R0805
- removed R13, R16, R19, R22, R4, R7: 66, resistor:R-EU_R0805
- removed R25: 10K, resistor:R-EU_R0805
- removed U$2, U$3: PCA9685PW, SPEAR:PCA9685PW
- added C10, C11, C12, C13, C14, C9: (no value), rcl:C-EUC0805
- added IC1, IC2: TPS92630QPWPRQ1, TPS92630QPWPRQ1:TPS92630QPWPRQ1
- added JP1: (no value), pinhead:PINHD-1X2
- added LED1, LED2: AAAF5051-05, AAAF5051-05:AAAF5051-05
- added SV1, SV2: (no value), con-lstb:MA04-1
- R1: value 66 -> 10K
- R10: value 66 -> 815
- R2: value 10 -> 815
- R3: value 10 -> 10K
Connections:
- removed net LEDA0: R13.1, U$2.LED0
- removed net LEDA1: R14.1, U$2.LED1
- removed net LEDA10: R21.1, U$2.LED10
- removed net LEDA11: U$2.LED11
- removed net LEDA12: R22.1, U$2.LED12
- removed net LEDA13: R23.1, U$2.LED13
- removed net LEDA14: R24.1, U$2.LED14
- removed net LEDA15: U$2.LED15
- removed net LEDA2: R15.1, U$2.LED2
- removed net LEDA3: U$2.LED3
- removed net LEDA4: R16.1, U$2.LED4
- removed net LEDA5: R17.1, U$2.LED5
- removed net LEDA6: R18.1, U$2.LED6
- removed net LEDA7: U$2.LED7
- removed net LEDA8: R19.1, U$2.LED8
- removed net LEDA9: R20.1, U$2.LED9
- removed net LEDB0: R1.1, U$3.LED0
- removed net LEDB1: R2.1, U$3.LED1
- removed net LEDB10: R9.1, U$3.LED10
- removed net LEDB11: U$3.LED11
- removed net LEDB12: R10.1, U$3.LED12
- removed net LEDB13: R11.1, U$3.LED13
- removed net LEDB14: R12.1, U$3.LED14
- removed net LEDB15: U$3.LED15
- removed net LEDB2: R3.1, U$3.LED2
- removed net LEDB3: U$3.LED3
- removed net LEDB4: R4.1, U$3.LED4
- removed net LEDB5: R5.1, U$3.LED5
- removed net LEDB6: R6.1, U$3.LED6
- removed net LEDB7: U$3.LED7
- removed net LEDB8: R7.1, U$3.LED8
- removed net LEDB9: R8.1, U$3.LED9
- removed net N$10: D8.R, R10.2
- removed net N$11: D8.G, R11.2
- removed net N$13: D1.R, R13.2
- removed net N$15: D1.B, R15.2
- removed net N$16: D2.R, R16.2
- removed net N$17: D2.G, R17.2
- removed net N$18: D2.B, R18.2
- removed net N$19: D3.R, R19.2
- removed net N$20: D3.G, R20.2
- removed net N$21: D3.B, R21.2
- removed net N$22: D4.R, R22.2
- removed net N$23: D4.G, R23.2
- removed net N$24: D4.B, R24.2
- removed net N$27: R25.2, U$3.A0
- removed net N$4: D6.R, R4.2
- removed net N$5: D6.G, R5.2
- removed net N$6: D6.B, R6.2
- removed net N$7: D7.R, R7.2
- removed net N$8: D7.G, R8.2
- removed net N$9: D7.B, R9.2
- new net L1OUT1: C9.1, IC1.IOUT1, IC1.VSNS1, LED1.K_BLUE
- new net L1OUT2: C10.1, IC1.IOUT2, IC1.VSNS2, LED1.K_ORANGE
- new net L1OUT3: C11.1, IC1.IOUT3, IC1.VSNS3, LED1.K_GREEN
- new net L2OUT1: C12.1, IC2.IOUT1, IC2.VSNS1, LED2.K_BLUE
- new net L2OUT2: C13.1, IC2.IOUT2, IC2.VSNS2, LED2.K_ORANGE
- new net L2OUT3: C14.1, IC2.IOUT3, IC2.VSNS3, LED2.K_GREEN
- new net PA1: IC1.FAULT_S, U1_PORTA.PA1
- new net PA2: IC1.FAULT, U1_PORTA.PA2
- new net PA3: IC1.PWM3, U1_PORTA.PA3
- new net PA4: IC1.PWM2, U1_PORTA.PA4
- new net PA5: IC1.PWM1, U1_PORTA.PA5
- new net PA6: IC1.EN, U1_PORTA.PA6
- new net PA7: IC2.FAULT_S, U1_PORTA.PA7
- new net PB0: IC2.FAULT, U1_PORTB.PB0
- new net PB1: IC2.PWM3, U1_PORTB.PB1
- new net PB10: IC2.PWM1, U1_PORTB.PB10
- new net PB11: IC2.EN, U1_PORTB.PB11
- new net PB2: IC2.PWM2, U1_PORTB.PB2
- new net PB8: U1_PORTB.PB8
- net +3V3: no longer D1.AN, D2.AN, D3.AN, D4.AN, D5.AN, D6.AN, D7.AN, D8.AN, R25.1, U$2.VDD, U$3.VDD
- net +5V: now also IC1.VIN, IC2.VIN, JP1.1, SV1.4, SV2.4; no longer CON1-1.S, CON2-1.S
- net CANH: now also SV1.3, SV2.3; no longer CON1-2.S, CON2-2.S
- net CANL: now also SV1.2, SV2.2; no longer CON1-3.S, CON2-3.S
- net GND: now also C10.2, C11.2, C12.2, C13.2, C14.2, C9.2, IC1.GND, IC2.GND, JP1.2, R1.1, R10.1, R2.1, R3.1, SV1.1, SV2.1; no longer CON1-4.S, CON2-4.S, U$2.A0, U$2.A1, U$2.A2, U$2.A3, U$2.A4, U$2.A5, U$2.VSS, U$3.A1, U$3.A2, U$3.A3, U$3.A4, U$3.A5, U$3.VSS
- net I2C_SCL: no longer U$2.SCL, U$3.SCL
- net I2C_SDA: no longer U$2.SDA, U$3.SDA
- net LED_!OE: no longer U$2.!OE, U$3.!OE
- net N$1: now also IC1.REF, R10.2; no longer D5.R, R1.2
- net N$12: now also IC1.TEMP, R1.2; no longer D8.B, R12.2
- net N$14: now also U1_PORTB.PB9; no longer D1.G, R14.2
- net N$2: now also IC2.TEMP, R3.2; no longer D5.G, R2.2
- net N$3: now also IC2.REF, R2.2; no longer D5.B, R3.2
Other:
- note removed: "Pin 35"
- moved on the sheet: R1, R10, R2, R3

Commit message: Fixed everything that needed to be fixed (hopefully)
Parts:
- removed CON1, CON2: SM04B-GHS-TB, ARVP:SM04B-GHS-TB
- removed LED1, LED2: AAAF5051-05, AAAF5051-05:AAAF5051-05
- removed U1: STM32F103CB, SPEAR:STM32F103CB
- added U$2: STM-DEV-BOARD, SPEAR:STM-DEV-BOARD
- added U$3, U$5: R50RGB-4-0045, SPEAR-indication:R50RGB-4-0045
- C10, C11, C12, C13, C14, C9: value (none) -> 100n
Connections:
- removed net BOOT0: U1_PWR.BOOT0
- removed net N$14: U1_PORTB.PB9
- removed net NRST: U1_PWR.NRST
- removed net PA7: IC2.FAULT_S, U1_PORTA.PA7
- removed net PB0: IC2.FAULT, U1_PORTB.PB0
- removed net PB1: IC2.PWM3, U1_PORTB.PB1
- removed net PB10: IC2.PWM1, U1_PORTB.PB10
- removed net PB11: IC2.EN, U1_PORTB.PB11
- removed net PB2: IC2.PWM2, U1_PORTB.PB2
- removed net SWCLK: U1_PORTA.PA14
- removed net SWDIO: U1_PORTA.PA13
- new net PB4: IC1.FAULT_S, U$2.PB4
- new net PB5: IC1.FAULT, U$2.PB5
- new net PB6: IC1.PWM3, U$2.PB6
- new net PB7: IC1.PWM2, U$2.PB7
- new net PB9: IC1.EN, U$2.PB9
- net +3V3: no longer U1_PWR.VDDA, U1_PWR.VDD_1, U1_PWR.VDD_2, U1_PWR.VDD_3
- net CANH: now also U$2.CANH
- net CANL: now also U$2.CANL
- net CAN_STBY: no longer U1_PORTA.PA10
- net GND: now also U$2.GND@2, U$2.GND@3, U$3.C, U$5.C; no longer CON1-TABS.S, CON2-TABS.S, U1_PWR.VSSA, U1_PWR.VSS_1, U1_PWR.VSS_2, U1_PWR.VSS_3
- net I2C_SCL: now also U$2.PB14; no longer U1_PORTB.PB6
- net I2C_SDA: now also U$2.PB15; no longer U1_PORTB.PB7
- net L1OUT1: now also U$3.BLU; no longer LED1.K_BLUE
- net L1OUT2: now also U$3.RED; no longer LED1.K_ORANGE
- net L1OUT3: now also U$3.GRN; no longer LED1.K_GREEN
- net L2OUT1: now also U$5.BLU; no longer LED2.K_BLUE
- net L2OUT2: now also U$5.RED; no longer LED2.K_ORANGE
- net L2OUT3: now also U$5.GRN; no longer LED2.K_GREEN
- net LED_!OE: now also U$2.PB10; no longer U1_PORTB.PB5
- net PA1: now also IC2.EN, U$2.PA1; no longer IC1.FAULT_S, U1_PORTA.PA1
- net PA2: now also IC2.PWM1, U$2.PA2; no longer IC1.FAULT, U1_PORTA.PA2
- net PA3: now also IC2.PWM2, U$2.PA3; no longer IC1.PWM3, U1_PORTA.PA3
- net PA4: now also IC2.PWM3, U$2.PA4; no longer IC1.PWM2, U1_PORTA.PA4
- net PA5: now also IC2.FAULT, U$2.PA5; no longer IC1.PWM1, U1_PORTA.PA5
- net PA6: now also IC2.FAULT_S, U$2.PA6; no longer IC1.EN, U1_PORTA.PA6
- net PB8: now also IC1.PWM1, U$2.PB8; no longer U1_PORTB.PB8
- net STM_CANRX: now also U$2.PB13; no longer U1_PORTA.PA11
- net STM_CANTX: now also U$2.PB12; no longer U1_PORTA.PA12
Other:
- moved on the sheet: C1, C2, C3, C4, C5, C6, C7, C8, SV2

Commit message: new design to fix a bunch of problems
Parts:
- removed C6: 4u7, resistor:C-EUC0805
- removed C7: 10n, resistor:C-EUC0805
- removed C8: 1u, resistor:C-EUC0805
- removed JP1: (no value), pinhead:PINHD-1X2
- removed R26, R27, R28: 10k, resistor:R-EU_R0805
- removed U$2: STM-DEV-BOARD, SPEAR:STM-DEV-BOARD
- removed U$4: TE-CONN_5-103669-1, SPEAR:TE-CONN_5-103669-1
- added D1: CGRM4001-G, diode:CGRM4001-G
- added J1: (no value), SparkFun-Connectors:CONN_025MM
- C1: value 100n -> 100nf; device resistor:C-EUC0805 -> resistor:C-EUC1206
- C10, C11, C12, C13, C14, C9: value 100n -> 10n
- C2, C4: value 100n -> 10uF; device resistor:C-EUC0805 -> rcl:C-EUC1206
- C3, C5: value 100n -> 100nF; device resistor:C-EUC0805 -> rcl:C-EUC0805
- R1, R3: value 10K -> 100
- R10, R2: value 815 -> 2.5k
- U$1: value MCP2562-E/SN -> STM-DEV-BOARD; device SPEAR:MCP2562-E/SN -> SPEAR:STM-DEV-BOARD
Connections:
- removed net +5V: IC1.VIN, IC2.VIN, JP1.1, SV1.4, SV2.4, U$1.VDD
- removed net CAN_STBY: U$1.STBY
- removed net I2C_SCL: R27.1, U$2.PB14
- removed net I2C_SDA: R28.1, U$2.PB15
- removed net LED_!OE: R26.1, U$2.PB10
- removed net PA1: IC2.EN, U$2.PA1
- removed net PA2: IC2.PWM1, U$2.PA2
- removed net PA3: IC2.PWM2, U$2.PA3
- removed net PA4: IC2.PWM3, U$2.PA4
- removed net PA5: IC2.FAULT, U$2.PA5
- removed net PA6: IC2.FAULT_S, U$2.PA6
- removed net PB4: IC1.FAULT_S, U$2.PB4
- removed net PB5: IC1.FAULT, U$2.PB5
- removed net PB6: IC1.PWM3, U$2.PB6
- removed net PB7: IC1.PWM2, U$2.PB7
- removed net PB8: IC1.PWM1, U$2.PB8
- removed net PB9: IC1.EN, U$2.PB9
- removed net STM_CANRX: U$1.RXD, U$2.PB13
- removed net STM_CANTX: U$1.TXD, U$2.PB12
- new net 5V: C1.1, D1.C, U$1.5V
- new net EN1: IC1.EN, U$1.PA2
- new net EN2: IC2.EN, U$1.PA3
- new net FAULT1: IC1.FAULT, U$1.PB10
- new net FAULT2: IC2.FAULT, U$1.PA4
- new net FAULTS1: IC1.FAULT_S, U$1.PB11
- new net FAULTS2: IC2.FAULT_S, U$1.PA5
- new net N$4: D1.A, SV1.4, SV2.4
- new net TIM3_CH1: IC2.PWM1, U$1.PA6
- new net TIM3_CH2: IC2.PWM2, U$1.PA7
- new net TIM3_CH3: IC2.PWM3, U$1.PB0
- new net TIM4_CH1: IC1.PWM1, U$1.PB6
- new net TIM4_CH2: IC1.PWM2, U$1.PB7
- new net TIM4_CH3: IC1.PWM3, U$1.PB8
- new net VIN: C2.1, C3.1, C4.1, C5.1, IC1.VIN, IC2.VIN, J1.2
- net +3V3: now also U$1.3.3V@1, U$1.VBAT; no longer C1.1, C2.1, C3.1, C4.1, C5.1, C6.1, C7.1, C8.1, R26.2, R27.2, R28.2, U$1.VIO, U$4.1
- net CANH: no longer U$2.CANH
- net CANL: no longer U$2.CANL
- net GND: now also IC1.EP, IC1.REF, IC2.EP, IC2.REF, J1.1, U$1.GND@1, U$1.GND@2, U$1.GND@3; no longer C6.2, C7.2, C8.2, IC1.GND, IC2.GND, JP1.2, U$1.VSS, U$2.GND@2, U$2.GND@3, U$4.2
- net N$1: now also IC1.GND; no longer IC1.REF
- net N$3: now also IC2.GND; no longer IC2.REF
Other:
- note removed: "4.7uF Capacitor must be connected to VDD_3"
- note removed: "Analog Supply Decoupling"
- note removed: "Digital Supply Decoupling"
- note removed: "PIN 1"
- note removed: "Pullup Resistors"
- moved on the sheet: C1, C2, C3, C4, C5, R10, R2
