File: can_indication/indication.brd (EAGLE design)
At the start: 160 x 100 mm, 51 parts, among them CON1 SM04B-GHS-TB, CON2 SM04B-GHS-TB, U1 STM32F103CB

Commit message: Fixed some footprint issues and most of positioning.
I botched a few footprints so I had to fix them :/
Parts:
- moved D8 114.2 mm to (59.7, 5.08)
- moved R9 113.7 mm to (52.1, 10.2), turned to 270 degrees
- moved R8 111.2 mm to (54.6, 10.2), turned to 270 degrees
- moved R11 110.6 mm to (59.7, 10.2), turned to 270 degrees
- moved D7 101.9 mm to (52.1, 5.08)
- moved R7 101.7 mm to (49.5, 10.2), turned to 270 degrees
- moved R6 94.6 mm to (47.0, 10.2), turned to 270 degrees
- moved CON2 93.7 mm to (61.0, 33.0), turned to 90 degrees
- moved R12 92.9 mm to (62.2, 10.2), turned to 270 degrees
- moved D6 90.2 mm to (44.5, 5.08)
- moved CON1 88.4 mm to (61.0, 21.6), turned to 90 degrees
- moved R5 87.6 mm to (44.5, 10.2), turned to 270 degrees
- moved R23 86.9 mm to (29.2, 10.2), turned to 270 degrees
- moved D3 85.6 mm to (21.6, 5.08)
- moved R10 81.7 mm to (57.1, 10.2), turned to 270 degrees
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Connections:
- net +3V3: now also U$1.5, U1.24, U1.36, U1.48, U1.9; no longer U$1.7, U1.4, U1.5, U1.6, U1.7
- net +5V: now also U$1.3; no longer U$1.6
- net BOOT0: now also U1.44; no longer U1.1
- net CANH: now also U$1.7; no longer U$1.1
- net CANL: now also U$1.6; no longer U$1.2
- net CAN_STBY: now also U$1.8, U1.31; no longer U$1.4, U1.22
- net GND: now also U$1.2, U1.23, U1.35, U1.47; no longer U$1.8, U1.10, U1.11, U1.9
- net I2C_SCL: now also U1.42; no longer U1.34
- net I2C_SDA: now also U1.43; no longer U1.35
- net LED_!OE: now also U1.41; no longer U1.33
- net NRST: now also U1.7; no longer U1.2
- net STM_CANRX: now also U$1.4, U1.32; no longer U$1.3, U1.23
- net STM_CANTX: now also U$1.1, U1.33; no longer U$1.5, U1.24
- net SWCLK: now also U1.37; no longer U1.26
- net SWDIO: now also U1.34; no longer U1.25

Commit message: Finished placement.
Parts:
- moved C7 26.6 mm to (33.7, 22.7), turned to 180 degrees
- moved C8 25.8 mm to (38.1, 22.7)
- moved C4 25.3 mm to (40.0, 27.8), turned to 270 degrees
- moved C1 16.3 mm to (25.4, 31.6), turned to 90 degrees
- moved C5 16.1 mm to (40.0, 32.3), turned to 90 degrees
- moved C3 14.9 mm to (22.9, 27.2), turned to 270 degrees
- moved C2 13.6 mm to (22.9, 31.6), turned to 90 degrees
- moved R27 8.32 mm to (16.0, 24.6)
- moved R28 8.32 mm to (13.5, 24.6)
- moved R26 8.32 mm to (10.9, 24.6), turned to 90 degrees
- moved CON2 5.80 mm to (58.7, 27.7)
- moved U$4 5.71 mm to (3.81, 26.0)
- moved C6 4.75 mm to (25.4, 27.2), turned to 270 degrees
- moved CON1 4.44 mm to (58.7, 17.8)
- moved U1 4.32 mm to (33.0, 29.7)
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Other:
- board size 160 x 100 mm -> 63.5 x 38 mm

Commit message: Finished a lot of routing.
Most of the PCA9685 stuff is routed.

Todo:
- Add programming header.
- Route everything else.
- Add planes.
Parts:
- moved R25 21.3 mm to (29.3, 16.3)
- moved R8 2.54 mm to (50.0, 7.62)
- moved R9 2.54 mm to (52.6, 7.62)
Connections:
- removed net LED_~OE: U$3.23
- net LED_!OE: now also U$3.23
Routing:
- net LED_!OE: track 0.00 -> 47.5 mm, vias 0 -> 3
- net I2C_SDA: track 0.00 -> 36.7 mm, vias 0 -> 2
- net I2C_SCL: track 0.00 -> 34.6 mm
- net LEDB14: track 0.00 -> 31.3 mm
- net LEDA14: track 0.00 -> 30.9 mm
- net LEDA13: track 0.00 -> 28.3 mm, vias 0 -> 2
- net LEDB13: track 0.00 -> 27.4 mm
- net LEDA12: track 0.00 -> 25.0 mm, vias 0 -> 2
- net LEDB12: track 0.00 -> 23.7 mm
- net LEDB10: track 0.00 -> 23.1 mm, vias 0 -> 2
- net CANH: track 0.01 -> 21.8 mm
- net LEDA10: track 0.00 -> 21.7 mm, vias 0 -> 2
- net LEDB9: track 0.00 -> 20.9 mm, vias 0 -> 2
- net LEDA9: track 0.00 -> 18.8 mm, vias 0 -> 2
- net CANL: track 0.01 -> 18.1 mm, vias 0 -> 3
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
Commit message: Finished Layout.
- Passes DRC.
Routing:
- net +3V3: track 0.00 -> 88.7 mm, vias 0 -> 14
- net GND: track 0.00 -> 31.5 mm, vias 0 -> 25
- net CAN_STBY: track 0.00 -> 22.9 mm
- net +5V: track 12.7 -> 33.3 mm
- net STM_CANRX: track 0.00 -> 17.8 mm, vias 0 -> 2
- net STM_CANTX: track 0.00 -> 17.7 mm, vias 0 -> 2
- net I2C_SCL: track 34.6 -> 46.7 mm, vias 0 -> 2
- net LED_!OE: track 47.5 -> 57.5 mm, vias 3 -> 5
- net I2C_SDA: track 36.7 -> 45.5 mm
- net LEDB10: track 23.1 -> 22.3 mm
- net LEDA0: track 7.27 -> 6.71 mm
- added copper zone on layer 1, net +3V3
- added copper zone on layer 16, net +3V3
- added copper zone on layer 1, net GND
- added copper zone on layer 16, net GND

Commit message: Fixed a few little things I noticed.
Routing:
- net LED_!OE: track 57.5 -> 60.1 mm
- net GND: track 31.5 -> 32.4 mm
Changed lines of the file:
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@@
 <wire x1="25.7228" y1="28.128" x2="26.6728" y2="27.178" width="0.3048" layer="1"/>
 <via x="26.6728" y="27.178" extent="1-16" drill="0.35"/>
-<wire x1="26.6728" y1="27.178" x2="27.5618" y2="26.289" width="0.3048" layer="16"/>
-<wire x1="27.5618" y1="26.289" x2="28.067" y2="26.289" width="0.3048" layer="16"/>
-<via x="28.067" y="26.289" extent="1-16" drill="0.35"/>
-<wire x1="28.067" y1="26.289" x2="28.091" y2="26.289" width="0.3048" layer="1"/>
-<wire x1="28.091" y1="26.289" x2="28.77" y2="26.968" width="0.3048" layer="1"/>
+<wire x1="26.6728" y1="27.178" x2="27.8158" y2="26.035" width="0.3048" layer="16"/>
+<wire x1="27.8158" y1="26.035" x2="28.067" y2="26.035" width="0.3048" layer="16"/>
+<via x="28.067" y="26.035" extent="1-16" drill="0.35"/>
+<wire x1="28.067" y1="26.265" x2="28.067" y2="26.035" width="0.3048" layer="1"/>
+<wire x1="28.067" y1="26.265" x2="28.77" y2="26.968" width="0.3048" layer="1"/>
 <polygon width="0.3048" layer="1">
 <vertex x="20.193" y="36.195"/>
@@
 <via x="19.431" y="17.272" extent="1-16" drill="0.35"/>
 <via x="11.684" y="12.192" extent="1-16" drill="0.35"/>
-<via x="3.81" y="16.383" extent="1-16" drill="0.35"/>
+<via x="3.302" y="15.875" extent="1-16" drill="0.35"/>
 <via x="10.922" y="13.335" extent="1-16" drill="0.35"/>
 <via x="56.642" y="23.241" extent="1-16" drill="0.35"/>
@@
 <wire x1="35.306" y1="31.623" x2="35.306" y2="30.353" width="0.2032" layer="1"/>
 <via x="35.306" y="30.353" extent="1-16" drill="0.35"/>
-<wire x1="30.77" y1="33.968" x2="30.77" y2="32.929" width="0.2032" layer="1"/>
-<wire x1="30.77" y1="32.929" x2="30.734" y2="32.893" width="0.2032" layer="1"/>
-<via x="30.734" y="32.893" extent="1-16" drill="0.35"/>
+<wire x1="30.77" y1="33.968" x2="30.77" y2="32.421" width="0.2032" layer="1"/>
+<wire x1="30.77" y1="32.421" x2="30.48" y2="32.131" width="0.2032" layer="1"/>
+<via x="30.48" y="32.131" extent="1-16" drill="0.35"/>
 <via x="24.13" y="33.909" extent="1-16" drill="0.35"/>
 <wire x1="24.13" y1="33.909" x2="25.019" y2="33.909" width="0.2032" layer="1"/>
@@
 <wire x1="9.078" y1="21.844" x2="4.572" y2="21.844" width="0.2032" layer="1"/>
 <via x="4.572" y="21.844" extent="1-16" drill="0.35"/>
-<wire x1="4.572" y1="21.844" x2="4.572" y2="18.034" width="0.2032" layer="16"/>
-<via x="4.572" y="18.034" extent="1-16" drill="0.35"/>
-<wire x1="4.572" y1="18.034" x2="4.613" y2="18.075" width="0.2032" layer="1"/>
-<wire x1="4.613" y1="18.075" x2="4.613" y2="19.537" width="0.2032" layer="1"/>
+<wire x1="4.318" y1="21.59" x2="4.318" y2="17.145" width="0.2032" layer="16"/>
+<via x="4.318" y="17.145" extent="1-16" drill="0.35"/>
+<wire x1="4.318" y1="17.145" x2="4.613" y2="17.44" width="0.2032" layer="1"/>
+<wire x1="4.613" y1="17.44" x2="4.613" y2="19.537" width="0.2032" layer="1"/>
 <contactref element="U$3" pad="23"/>
 <wire x1="35.093" y1="19.41" x2="35.052" y2="19.369" width="0.2032" layer="1"/>
@@
 <wire x1="34.798" y1="18.034" x2="30.988" y2="18.034" width="0.2032" layer="1"/>
 <via x="10.668" y="19.558" extent="1-16" drill="0.35"/>
-<wire x1="10.668" y1="19.558" x2="9.144" y2="18.034" width="0.2032" layer="16"/>
+<wire x1="10.668" y1="19.558" x2="8.255" y2="17.145" width="0.2032" layer="16"/>
 <wire x1="18.288" y1="19.558" x2="10.668" y2="19.558" width="0.2032" layer="1"/>
-<wire x1="9.144" y1="18.034" x2="4.572" y2="18.034" width="0.2032" layer="16"/>
+<wire x1="8.255" y1="17.145" x2="4.318" y2="17.145" width="0.2032" layer="16"/>
 <wire x1="20.8026" y1="22.0726" x2="18.288" y2="19.558" width="0.2032" layer="1"/>
 <wire x1="30.988" y1="18.034" x2="27.3685" y2="21.6535" width="0.2032" layer="1"/>
@@
 <wire x1="27.3685" y1="21.6535" x2="27.3713" y2="21.6535" width="0.2032" layer="1"/>
 <wire x1="27.3713" y1="21.6535" x2="27.6662" y2="21.9484" width="0.2032" layer="1"/>
+<wire x1="4.572" y1="21.844" x2="4.318" y2="21.59" width="0.2032" layer="16"/>
 </signal>
 <signal name="N$27">
