File: can_indication/indication.brd (EAGLE design)
At the start: 63.5 x 38 mm, 51 parts, among them CON1 SM04B-GHS-TB, CON2 SM04B-GHS-TB, U1 STM32F103CB

Commit message: Changed the indication board so it uses higher power LED's now
Parts:
- removed D1, D2, D3, D4, D5, D6, D7, D8: CLV1L-FKB-CHMMQEHBB7673673, SPEAR:PLCC-4
- removed R11, R12, R14, R15, R17, R18, R20, R21, R23, R24, R5, R6, R8, R9: 10, resistor:R0805
- removed R13, R16, R19, R22, R4, R7: 66, resistor:R0805
- removed R25: 10K, resistor:R0805
- removed U$2, U$3: PCA9685PW, SPEAR:TSSOP28
- added C10, C11, C12, C13, C14, C9: (no value), rcl:C0805
- added IC1, IC2: TPS92630QPWPRQ1, TPS92630QPWPRQ1:SOP65P640X120-17N
- added JP1: (no value), pinhead:1X02
- added LED1, LED2: AAAF5051-05, AAAF5051-05:AAAF505105
- added SV1, SV2: (no value), con-lstb:MA04-1
- R1: value 66 -> 10K
- R10: value 66 -> 815
- R2: value 10 -> 815
- R3: value 10 -> 10K
- moved R2 42.1 mm to (67.3, 34.3), turned to 90 degrees
- moved C8 41.0 mm to (2.54, 43.2), turned to 90 degrees
- moved R3 37.4 mm to (63.5, 34.3), turned to 90 degrees
- moved CON1 36.1 mm to (64.8, 53.3), turned to 0 degrees
- moved CON2 34.9 mm to (63.5, 62.2), turned to 0 degrees
- moved C7 33.1 mm to (7.62, 43.2), turned to 90 degrees
- moved R1 26.2 mm to (55.9, 19.1), turned to 90 degrees
- moved C3 26.0 mm to (38.1, 48.3), turned to 90 degrees
- moved U$1 21.9 mm to (48.3, 52.1), turned to 90 degrees
- moved R26 21.7 mm to (27.9, 38.1)
- moved C4 21.6 mm to (33.0, 48.3), turned to 90 degrees
- moved C5 20.0 mm to (27.9, 48.3)
- moved C1 17.2 mm to (38.1, 43.2), turned to 270 degrees
- moved C6 16.2 mm to (27.9, 43.2)
- moved R27 15.7 mm to (24.1, 38.1)
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Connections:
- removed net LEDA0: R13.1, U$2.6
- removed net LEDA1: R14.1, U$2.7
- removed net LEDA10: R21.1, U$2.17
- removed net LEDA11: U$2.18
- removed net LEDA12: R22.1, U$2.19
- removed net LEDA13: R23.1, U$2.20
- removed net LEDA14: R24.1, U$2.21
- removed net LEDA15: U$2.22
- removed net LEDA2: R15.1, U$2.8
- removed net LEDA3: U$2.9
- removed net LEDA4: R16.1, U$2.10
- removed net LEDA5: R17.1, U$2.11
- removed net LEDA6: R18.1, U$2.12
- removed net LEDA7: U$2.13
- removed net LEDA8: R19.1, U$2.15
- removed net LEDA9: R20.1, U$2.16
- removed net LEDB0: R1.1, U$3.6
- removed net LEDB1: R2.1, U$3.7
- removed net LEDB10: R9.1, U$3.17
- removed net LEDB11: U$3.18
- removed net LEDB12: R10.1, U$3.19
- removed net LEDB13: R11.1, U$3.20
- removed net LEDB14: R12.1, U$3.21
- removed net LEDB15: U$3.22
- removed net LEDB2: R3.1, U$3.8
- removed net LEDB3: U$3.9
- removed net LEDB4: R4.1, U$3.10
- removed net LEDB5: R5.1, U$3.11
- removed net LEDB6: R6.1, U$3.12
- removed net LEDB7: U$3.13
- removed net LEDB8: R7.1, U$3.15
- removed net LEDB9: R8.1, U$3.16
- removed net N$10: D8.P$2, R10.2
- removed net N$11: D8.P$3, R11.2
- removed net N$13: D1.P$2, R13.2
- removed net N$15: D1.P$4, R15.2
- removed net N$16: D2.P$2, R16.2
- removed net N$17: D2.P$3, R17.2
- removed net N$18: D2.P$4, R18.2
- removed net N$19: D3.P$2, R19.2
- removed net N$20: D3.P$3, R20.2
- removed net N$21: D3.P$4, R21.2
- removed net N$22: D4.P$2, R22.2
- removed net N$23: D4.P$3, R23.2
- removed net N$24: D4.P$4, R24.2
- removed net N$27: R25.2, U$3.1
- removed net N$4: D6.P$2, R4.2
- removed net N$5: D6.P$3, R5.2
- removed net N$6: D6.P$4, R6.2
- removed net N$7: D7.P$2, R7.2
- removed net N$8: D7.P$3, R8.2
- removed net N$9: D7.P$4, R9.2
- new net L1OUT1: C9.1, IC1.11, IC1.16, LED1.1
- new net L1OUT2: C10.1, IC1.12, IC1.15, LED1.2
- new net L1OUT3: C11.1, IC1.13, IC1.14, LED1.3
- new net L2OUT1: C12.1, IC2.11, IC2.16, LED2.1
- new net L2OUT2: C13.1, IC2.12, IC2.15, LED2.2
- new net L2OUT3: C14.1, IC2.13, IC2.14, LED2.3
- new net PA1: IC1.7, U1.11
- new net PA2: IC1.6, U1.12
- new net PA3: IC1.5, U1.13
- new net PA4: IC1.4, U1.14
- new net PA5: IC1.3, U1.15
- new net PA6: IC1.2, U1.16
- new net PA7: IC2.7, U1.17
- new net PB0: IC2.6, U1.18
- new net PB1: IC2.5, U1.19
- new net PB10: IC2.3, U1.21
- new net PB11: IC2.2, U1.22
- new net PB2: IC2.4, U1.20
- new net PB8: U1.45
- net +3V3: no longer D1.P$1, D2.P$1, D3.P$1, D4.P$1, D5.P$1, D6.P$1, D7.P$1, D8.P$1, R25.1, U$2.28, U$3.28
- net +5V: now also IC1.1, IC2.1, JP1.1, SV1.4, SV2.4; no longer CON1.P$1, CON2.P$1
- net CANH: now also SV1.3, SV2.3; no longer CON1.P$2, CON2.P$2
- net CANL: now also SV1.2, SV2.2; no longer CON1.P$3, CON2.P$3
- net GND: now also C10.2, C11.2, C12.2, C13.2, C14.2, C9.2, IC1.9, IC2.9, JP1.2, R1.1, R10.1, R2.1, R3.1, SV1.1, SV2.1; no longer CON1.P$4, CON2.P$4, U$2.1, U$2.14, U$2.2, U$2.24, U$2.3, U$2.4, U$2.5, U$3.14, U$3.2, U$3.24, U$3.3, U$3.4, U$3.5
- net I2C_SCL: no longer U$2.26, U$3.26
- net I2C_SDA: no longer U$2.27, U$3.27
- net LED_!OE: no longer U$2.23, U$3.23
- net N$1: now also IC1.10, R10.2; no longer D5.P$2, R1.2
- net N$12: now also IC1.8, R1.2; no longer D8.P$4, R12.2
- net N$14: now also U1.46; no longer D1.P$3, R14.2
- net N$2: now also IC2.8, R3.2; no longer D5.P$3, R2.2
- net N$3: now also IC2.10, R2.2; no longer D5.P$4, R3.2
Routing:
- net GND: track 32.4 -> 148.9 mm, vias 25 -> 14
- net +5V: track 33.3 -> 82.3 mm, vias 0 -> 2
- net LED_!OE: track 60.1 -> 13.1 mm, vias 5 -> 0
- net LEDB14: track 31.3 -> 0.00 mm
- net L2OUT2: track 0.00 -> 31.0 mm, vias 0 -> 2
- net LEDA14: track 30.9 -> 0.00 mm
- net I2C_SCL: track 46.7 -> 17.2 mm, vias 2 -> 0
- net LEDA13: track 28.3 -> 0.00 mm, vias 2 -> 0
- net LEDB13: track 27.7 -> 0.00 mm
- net L2OUT1: track 0.00 -> 27.2 mm
- net L2OUT3: track 0.00 -> 25.1 mm
- net LEDA12: track 25.0 -> 0.00 mm, vias 2 -> 0
- net L1OUT2: track 0.00 -> 24.6 mm, vias 0 -> 2
- net I2C_SDA: track 45.5 -> 21.2 mm, vias 2 -> 0
- net +3V3: track 89.0 -> 112.8 mm, vias 14 -> 5
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- removed copper zone on layer 1, net +3V3
- removed copper zone on layer 16, net +3V3
- removed copper zone on layer 16, net GND
Other:
- board size 63.5 x 38 mm -> 100 x 80 mm
- board text added: "SPEAR Indication Board Revision Jack Opgenorth"

Commit message: Moved some silkscreen so they weren't on top of eachother
Parts:
- moved SV1 8.89 mm to (20.3, 58.4)
Routing:
- net GND: track 148.9 -> 140.1 mm
- net +5V: track 82.3 -> 73.4 mm
- net CANL: track 39.8 -> 30.9 mm
- net CANH: track 37.5 -> 28.6 mm
Other:
- board size 100 x 80 mm -> 98.7 x 50.8 mm
Changed lines of the file:
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@@
 <board>
 <plain>
-<wire x1="0" y1="0" x2="100" y2="0" width="0" layer="20"/>
-<wire x1="100" y1="0" x2="100" y2="80" width="0" layer="20"/>
-<wire x1="100" y1="80" x2="0" y2="80" width="0" layer="20"/>
-<wire x1="0" y1="80" x2="0" y2="0" width="0" layer="20"/>
+<wire x1="0" y1="15.24" x2="97.46" y2="15.24" width="0" layer="20"/>
+<wire x1="97.46" y1="15.24" x2="98.73" y2="66.03" width="0" layer="20"/>
+<wire x1="98.73" y1="66.03" x2="0" y2="66.03" width="0" layer="20"/>
+<wire x1="0" y1="66.03" x2="0" y2="15.24" width="0" layer="20"/>
 <text x="2.54" y="24.13" size="1.778" layer="121">SPEAR
 Indication Board Revision
@@
 <element name="R26" library="resistor" library_urn="urn:adsk.eagle:library:348" package="R0805" package3d_urn="urn:adsk.eagle:package:23553/2" value="10k" x="27.94" y="38.1" smashed="yes" rot="R90">
 <attribute name="NAME" x="26.67" y="37.465" size="1.27" layer="25" rot="R90"/>
-<attribute name="VALUE" x="30.48" y="37.465" size="1.27" layer="27" rot="R90"/>
+<attribute name="VALUE" x="26.67" y="33.655" size="1.27" layer="27" rot="R90"/>
 </element>
 <element name="R27" library="resistor" library_urn="urn:adsk.eagle:library:348" package="R0805" package3d_urn="urn:adsk.eagle:package:23553/2" value="10k" x="24.13" y="38.1" smashed="yes" rot="R90">
 <attribute name="NAME" x="22.86" y="37.465" size="1.27" layer="25" rot="R90"/>
-<attribute name="VALUE" x="26.67" y="37.465" size="1.27" layer="27" rot="R90"/>
+<attribute name="VALUE" x="22.86" y="33.655" size="1.27" layer="27" rot="R90"/>
 </element>
 <element name="R28" library="resistor" library_urn="urn:adsk.eagle:library:348" package="R0805" package3d_urn="urn:adsk.eagle:package:23553/2" value="10k" x="20.32" y="38.1" smashed="yes" rot="R90">
 <attribute name="NAME" x="19.05" y="37.465" size="1.27" layer="25" rot="R90"/>
-<attribute name="VALUE" x="22.86" y="37.465" size="1.27" layer="27" rot="R90"/>
+<attribute name="VALUE" x="19.05" y="33.655" size="1.27" layer="27" rot="R90"/>
 </element>
 <element name="U$1" library="SPEAR" package="SOIC8" value="MCP2562-E/SN" x="48.26" y="52.07" smashed="yes" rot="R90">
@@
 <element name="R3" library="resistor" library_urn="urn:adsk.eagle:library:348" package="R0805" package3d_urn="urn:adsk.eagle:package:23553/2" value="10K" x="63.5" y="34.29" smashed="yes" rot="R90">
 <attribute name="NAME" x="60.96" y="33.655" size="1.27" layer="25" rot="R90"/>
-<attribute name="VALUE" x="66.04" y="33.655" size="1.27" layer="27" rot="R90"/>
-</element>
-<element name="SV1" library="con-lstb" library_urn="urn:adsk.eagle:library:162" package="MA04-1" package3d_urn="urn:adsk.eagle:package:8337/1" value="" x="11.43" y="58.42" smashed="yes" rot="R90">
-<attribute name="MF" value="" x="11.43" y="58.42" size="1.778" layer="27" rot="R90" display="off"/>
-<attribute name="MPN" value="" x="11.43" y="58.42" size="1.778" layer="27" rot="R90" display="off"/>
-<attribute name="NAME" x="9.779" y="53.34" size="1.27" layer="25" ratio="10" rot="R90"/>
-<attribute name="OC_FARNELL" value="unknown" x="11.43" y="58.42" size="1.778" layer="27" rot="R90" display="off"/>
-<attribute name="OC_NEWARK" value="unknown" x="11.43" y="58.42" size="1.778" layer="27" rot="R90" display="off"/>
-<attribute name="POPULARITY" value="41" x="11.43" y="58.42" size="1.778" layer="27" rot="R90" display="off"/>
-<attribute name="VALUE" x="9.779" y="59.055" size="1.27" layer="27" ratio="10" rot="R90"/>
+<attribute name="VALUE" x="66.04" y="29.845" size="1.27" layer="27" rot="R90"/>
+</element>
+<element name="SV1" library="con-lstb" library_urn="urn:adsk.eagle:library:162" package="MA04-1" package3d_urn="urn:adsk.eagle:package:8337/1" value="" x="20.32" y="58.42" smashed="yes" rot="R90">
+<attribute name="MF" value="" x="20.32" y="58.42" size="1.778" layer="27" rot="R90" display="off"/>
+<attribute name="MPN" value="" x="20.32" y="58.42" size="1.778" layer="27" rot="R90" display="off"/>
+<attribute name="NAME" x="18.669" y="53.34" size="1.27" layer="25" ratio="10" rot="R90"/>
+<attribute name="OC_FARNELL" value="unknown" x="20.32" y="58.42" size="1.778" layer="27" rot="R90" display="off"/>
+<attribute name="OC_NEWARK" value="unknown" x="20.32" y="58.42" size="1.778" layer="27" rot="R90" display="off"/>
+<attribute name="POPULARITY" value="41" x="20.32" y="58.42" size="1.778" layer="27" rot="R90" display="off"/>
+<attribute name="VALUE" x="18.669" y="59.055" size="1.27" layer="27" ratio="10" rot="R90"/>
 </element>
 <element name="SV2" library="con-lstb" library_urn="urn:adsk.eagle:library:162" package="MA04-1" package3d_urn="urn:adsk.eagle:package:8337/1" value="" x="33.02" y="58.42" smashed="yes" rot="R90">
@@
 <contactref element="SV1" pad="4"/>
 <contactref element="SV2" pad="4"/>
-<wire x1="11.43" y1="62.23" x2="33.02" y2="62.23" width="0.1524" layer="1"/>
+<wire x1="20.32" y1="62.23" x2="33.02" y2="62.23" width="0.1524" layer="1"/>
 <wire x1="51.8546875" y1="53.4464" x2="51.7514" y2="53.4464" width="0.1524" layer="1"/>
 <wire x1="51.7514" y1="53.4464" x2="51.01" y2="52.705" width="0.1524" layer="1"/>
@@
 <wire x1="64.77" y1="18.1" x2="55.88" y2="18.1" width="0.1524" layer="1"/>
 <contactref element="SV2" pad="1"/>
-<wire x1="11.43" y1="54.61" x2="22.86" y2="54.61" width="0.1524" layer="1"/>
+<wire x1="20.32" y1="54.61" x2="22.86" y2="54.61" width="0.1524" layer="1"/>
 <wire x1="22.86" y1="54.61" x2="28.1" y2="49.37" width="0.1524" layer="1"/>
 <via x="63.5" y="57.15" extent="1-16" drill="0.35"/>
@@
 <contactref element="SV1" pad="3"/>
 <contactref element="SV2" pad="3"/>
-<wire x1="11.43" y1="59.69" x2="33.02" y2="59.69" width="0.1524" layer="1"/>
+<wire x1="20.32" y1="59.69" x2="33.02" y2="59.69" width="0.1524" layer="1"/>
 <wire x1="44.6653125" y1="52.1764" x2="44.7686" y2="52.1764" width="0.1524" layer="1"/>
 <wire x1="44.7686" y1="52.1764" x2="45.51" y2="51.435" width="0.1524" layer="1"/>
@@
 <contactref element="SV1" pad="2"/>
 <contactref element="SV2" pad="2"/>
-<wire x1="11.43" y1="57.15" x2="33.02" y2="57.15" width="0.1524" layer="1"/>
+<wire x1="20.32" y1="57.15" x2="33.02" y2="57.15" width="0.1524" layer="1"/>
 <wire x1="44.6653125" y1="50.9064" x2="46.3546875" y2="50.9064" width="0.1524" layer="1"/>
 <wire x1="46.3546875" y1="50.9064" x2="46.4886" y2="51.0403125" width="0.1524" layer="1"/>

Commit message: Fixed everything that needed to be fixed (hopefully)
Parts:
- removed CON1, CON2: SM04B-GHS-TB, ARVP:SM04B-GHS-TB
- removed LED1, LED2: AAAF5051-05, AAAF5051-05:AAAF505105
- removed U1: STM32F103CB, SPEAR:LQFP48
- added U$2: STM-DEV-BOARD, SPEAR:STM-DEV-BOARD
- added U$3, U$5: R50RGB-4-0045, SPEAR-indication:R50RGB-4-0045
- C10, C11, C12, C13, C14, C9: value (none) -> 100n
- moved R28 57.6 mm to (72.4, 62.6), turned to 180 degrees
- moved R27 53.0 mm to (72.4, 59.9), turned to 180 degrees
- moved R26 51.9 mm to (72.4, 64.9), turned to 180 degrees
- moved U$4 41.8 mm to (41.3, 62.2)
- moved C7 38.2 mm to (43.6, 56.0), turned to 270 degrees
- moved C8 38.0 mm to (38.4, 56.0), turned to 270 degrees
- moved SV1 35.7 mm to (55.9, 55.9), turned to 180 degrees
- moved SV2 35.7 mm to (68.6, 55.9), turned to 180 degrees
- moved C2 35.5 mm to (63.6, 61.1)
- moved C1 34.4 mm to (67.4, 61.1)
- moved C5 27.4 mm to (52.2, 61.1), turned to 270 degrees
- moved C6 27.2 mm to (48.4, 61.1)
- moved C11 26.7 mm to (45.7, 34.3), turned to 90 degrees
- moved C4 26.3 mm to (56.0, 61.1), turned to 270 degrees
- moved C3 25.2 mm to (59.8, 61.1), turned to 270 degrees
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Connections:
- removed net BOOT0: U1.44
- removed net N$14: U1.46
- removed net NRST: U1.7
- removed net PA7: IC2.7, U1.17
- removed net PB0: IC2.6, U1.18
- removed net PB1: IC2.5, U1.19
- removed net PB10: IC2.3, U1.21
- removed net PB11: IC2.2, U1.22
- removed net PB2: IC2.4, U1.20
- removed net SWCLK: U1.37
- removed net SWDIO: U1.34
- new net PB4: IC1.7, U$2.PB4
- new net PB5: IC1.6, U$2.PB5
- new net PB6: IC1.5, U$2.PB6
- new net PB7: IC1.4, U$2.PB7
- new net PB9: IC1.2, U$2.PB9
- net +3V3: no longer U1.24, U1.36, U1.48, U1.9
- net CANH: now also U$2.CANH
- net CANL: now also U$2.CANL
- net CAN_STBY: no longer U1.31
- net GND: now also U$2.GND@2, U$2.GND@3, U$3.P$2, U$5.P$2; no longer CON1.P$5, CON1.P$6, CON2.P$5, CON2.P$6, U1.23, U1.35, U1.47, U1.8
- net I2C_SCL: now also U$2.PB14; no longer U1.42
- net I2C_SDA: now also U$2.PB15; no longer U1.43
- net L1OUT1: now also U$3.P$3; no longer LED1.1
- net L1OUT2: now also U$3.P$4; no longer LED1.2
- net L1OUT3: now also U$3.P$1; no longer LED1.3
- net L2OUT1: now also U$5.P$3; no longer LED2.1
- net L2OUT2: now also U$5.P$4; no longer LED2.2
- net L2OUT3: now also U$5.P$1; no longer LED2.3
- net LED_!OE: now also U$2.PB10; no longer U1.41
- net PA1: now also IC2.2, U$2.PA1; no longer IC1.7, U1.11
- net PA2: now also IC2.3, U$2.PA2; no longer IC1.6, U1.12
- net PA3: now also IC2.4, U$2.PA3; no longer IC1.5, U1.13
- net PA4: now also IC2.5, U$2.PA4; no longer IC1.4, U1.14
- net PA5: now also IC2.6, U$2.PA5; no longer IC1.3, U1.15
- net PA6: now also IC2.7, U$2.PA6; no longer IC1.2, U1.16
- net PB8: now also IC1.3, U$2.PB8; no longer U1.45
- net STM_CANRX: now also U$2.PB13; no longer U1.32
- net STM_CANTX: now also U$2.PB12; no longer U1.33
Routing:
- net +3V3: track 112.8 -> 69.7 mm, vias 5 -> 2
- net PA1: track 12.4 -> 37.2 mm, vias 0 -> 2
- net PA3: track 10.2 -> 33.4 mm
- net PA2: track 11.4 -> 34.0 mm
- net PA4: track 10.1 -> 32.2 mm
- net PA6: track 10.0 -> 30.7 mm, vias 0 -> 2
- net PA5: track 10.1 -> 30.7 mm
- net LED_!OE: track 13.1 -> 31.5 mm
- net CAN_STBY: track 17.4 -> 0.00 mm
- net CANH: track 28.6 -> 45.6 mm, vias 0 -> 3
- net +5V: track 73.4 -> 89.1 mm, vias 2 -> 6
- net PB11: track 10.6 -> 0.00 mm
- net PB10: track 10.6 -> 0.00 mm
- net PB2: track 10.5 -> 0.00 mm
- net PB1: track 10.4 -> 0.00 mm
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Other:
- board size 98.7 x 50.8 mm -> 69.9 x 63.5 mm

Commit message: got rid of some useless ground traces
Routing:
- net GND: track 134.1 -> 110.9 mm, vias 10 -> 7
Changed lines of the file:
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@@
 <element name="C1" library="resistor" library_urn="urn:adsk.eagle:library:348" package="C0805" package3d_urn="urn:adsk.eagle:package:23617/2" value="100n" x="67.437" y="61.087" smashed="yes" rot="R270">
 <attribute name="NAME" x="64.897" y="62.357" size="1.27" layer="25" rot="R270"/>
-<attribute name="VALUE" x="62.103" y="66.167" size="1.27" layer="27"/>
+<attribute name="VALUE" x="65.913" y="63.627" size="1.27" layer="27"/>
 </element>
 <element name="C2" library="resistor" library_urn="urn:adsk.eagle:library:348" package="C0805" package3d_urn="urn:adsk.eagle:package:23617/2" value="100n" x="63.627" y="61.087" smashed="yes" rot="R270">
 <attribute name="NAME" x="61.087" y="62.357" size="1.27" layer="25" rot="R270"/>
-<attribute name="VALUE" x="63.627" y="62.23" size="1.27" layer="27"/>
+<attribute name="VALUE" x="62.357" y="63.5" size="1.27" layer="27"/>
 </element>
 <element name="C3" library="resistor" library_urn="urn:adsk.eagle:library:348" package="C0805" package3d_urn="urn:adsk.eagle:package:23617/2" value="100n" x="59.817" y="61.087" smashed="yes" rot="R270">
 <attribute name="NAME" x="61.087" y="62.357" size="1.27" layer="25" rot="R270"/>
-<attribute name="VALUE" x="59.817" y="62.23" size="1.27" layer="27"/>
+<attribute name="VALUE" x="58.547" y="63.5" size="1.27" layer="27"/>
 </element>
 <element name="C4" library="resistor" library_urn="urn:adsk.eagle:library:348" package="C0805" package3d_urn="urn:adsk.eagle:package:23617/2" value="100n" x="56.007" y="61.087" smashed="yes" rot="R270">
 <attribute name="NAME" x="57.277" y="62.357" size="1.27" layer="25" rot="R270"/>
-<attribute name="VALUE" x="56.007" y="62.23" size="1.27" layer="27"/>
+<attribute name="VALUE" x="54.737" y="63.5" size="1.27" layer="27"/>
 </element>
 <element name="C5" library="resistor" library_urn="urn:adsk.eagle:library:348" package="C0805" package3d_urn="urn:adsk.eagle:package:23617/2" value="100n" x="52.197" y="61.087" smashed="yes" rot="R270">
 <attribute name="NAME" x="53.467" y="62.357" size="1.27" layer="25" rot="R270"/>
-<attribute name="VALUE" x="52.197" y="62.23" size="1.27" layer="27"/>
+<attribute name="VALUE" x="50.927" y="63.5" size="1.27" layer="27"/>
 </element>
 <element name="C6" library="resistor" library_urn="urn:adsk.eagle:library:348" package="C0805" package3d_urn="urn:adsk.eagle:package:23617/2" value="4u7" x="48.387" y="61.087" smashed="yes" rot="R270">
 <attribute name="NAME" x="43.307" y="62.357" size="1.27" layer="25" rot="R270"/>
-<attribute name="VALUE" x="49.657" y="62.357" size="1.27" layer="27" rot="R270"/>
+<attribute name="VALUE" x="46.863" y="63.627" size="1.27" layer="27"/>
 </element>
 <element name="C7" library="resistor" library_urn="urn:adsk.eagle:library:348" package="C0805" package3d_urn="urn:adsk.eagle:package:23617/2" value="10n" x="43.561" y="56.007" smashed="yes" rot="R270">
@@
 <element name="R26" library="resistor" library_urn="urn:adsk.eagle:library:348" package="R0805" package3d_urn="urn:adsk.eagle:package:23553/2" value="10k" x="72.39" y="64.897" smashed="yes" rot="R180">
 <attribute name="NAME" x="76.835" y="66.167" size="1.27" layer="25" rot="R180"/>
-<attribute name="VALUE" x="70.485" y="64.897" size="1.27" layer="27" rot="R180"/>
+<attribute name="VALUE" x="73.025" y="67.437" size="1.27" layer="27" rot="R180"/>
 </element>
 <element name="R27" library="resistor" library_urn="urn:adsk.eagle:library:348" package="R0805" package3d_urn="urn:adsk.eagle:package:23553/2" value="10k" x="72.39" y="59.944" smashed="yes" rot="R180">
@@
 <via x="66.04" y="12.7" extent="1-16" drill="0.35"/>
 <via x="66.04" y="30.48" extent="1-16" drill="0.35"/>
-<via x="46.99" y="48.26" extent="1-16" drill="0.35"/>
 <wire x1="67.31" y1="31.75" x2="66.04" y2="30.48" width="0.1524" layer="1"/>
 <wire x1="63.5" y1="34.61" x2="63.5" y2="33.02" width="0.1524" layer="1"/>
@@
 <wire x1="67.31" y1="34.61" x2="67.31" y2="31.75" width="0.1524" layer="1"/>
 <via x="62.23" y="55.245" extent="1-16" drill="0.35"/>
-<via x="72.39" y="58.42" extent="1-16" drill="0.35"/>
-<wire x1="59.69" y1="55.88" x2="61.595" y2="55.88" width="0.1524" layer="1"/>
-<wire x1="61.595" y1="55.88" x2="62.23" y2="55.245" width="0.1524" layer="1"/>
-<wire x1="72.39" y1="55.88" x2="72.39" y2="58.42" width="0.381" layer="1"/>
 <wire x1="52.07" y1="51.75" x2="55.88" y2="51.75" width="0.1524" layer="1"/>
 <wire x1="55.88" y1="51.75" x2="59.69" y2="51.75" width="0.1524" layer="1"/>
@@
 <wire x1="38.354" y1="55.057" x2="40.64" y2="52.771" width="0.381" layer="1"/>
 <wire x1="40.64" y1="52.771" x2="40.64" y2="52.07" width="0.381" layer="1"/>
-<wire x1="43.561" y1="54.991" x2="40.64" y2="52.07" width="0.381" layer="1"/>
-<wire x1="41.91" y1="44.45" x2="45.72" y2="48.26" width="0.381" layer="1"/>
-<wire x1="45.72" y1="48.26" x2="46.99" y2="48.26" width="0.381" layer="1"/>
 <wire x1="62.8932" y1="49.27865" x2="62.8932" y2="49.78135" width="0.1524" layer="1"/>
 <wire x1="63.24865" y1="50.1368" x2="62.8932" y2="49.78135" width="0.1524" layer="1"/>
@@
 <wire x1="63.5" y1="16.83" x2="66.04" y2="14.29" width="0.1524" layer="1"/>
 <wire x1="66.04" y1="14.29" x2="66.04" y2="12.7" width="0.1524" layer="1"/>
-<wire x1="67.437" y1="60.137" x2="69.154" y2="58.42" width="0.508" layer="1"/>
-<wire x1="69.154" y1="58.42" x2="72.39" y2="58.42" width="0.508" layer="1"/>
 <via x="90.17" y="59.69" extent="1-16" drill="0.35"/>
 <polygon width="0.1524" layer="1">
@@
 <wire x1="62.23" y1="29.817" x2="62.23" y2="30.48" width="0.1524" layer="1"/>
 <wire x1="92.71" y1="57.15" x2="90.17" y2="59.69" width="0.1524" layer="1"/>
-<wire x1="49.53" y1="46.99" x2="48.26" y2="46.99" width="0.1524" layer="1"/>
-<wire x1="48.26" y1="46.99" x2="46.99" y2="48.26" width="0.1524" layer="1"/>
 <contactref element="U$2" pad="GND@3"/>
 <wire x1="97.409" y1="59.69" x2="90.17" y2="59.69" width="0.1524" layer="1"/>
-<via x="46.99" y="29.21" extent="1-16" drill="0.35"/>
-<wire x1="49.53" y1="29.21" x2="46.99" y2="29.21" width="0.1524" layer="1"/>
+<wire x1="43.561" y1="55.057" x2="40.64" y2="52.136" width="0.381" layer="1"/>
+<wire x1="40.64" y1="52.136" x2="40.64" y2="52.07" width="0.381" layer="1"/>
 </signal>
 <signal name="STM_CANRX">

Commit message: increased size of power traces and some other traces
Routing:
- net GND: track 110.9 -> 113.5 mm, vias 7 -> 4
- net +5V: track 89.1 -> 86.7 mm
- net L1OUT1: track 23.2 -> 20.9 mm
- net L2OUT1: track 24.2 -> 22.8 mm
- net L1OUT3: track 30.3 -> 29.2 mm
- net L1OUT2: track 24.0 -> 24.8 mm
- net N$12: track 10.7 -> 10.1 mm
