File: arm-controller-stm32f103cbt6/Arm controller.brd (EAGLE design)
At the start: 67 x 65 mm, 59 parts, among them CON1 SM04B-GHS-TB, J1 CORTEX_DEBUG_SMD, Q1 32.768kHz, U1 3.3V, U2 3.3V, X1 8MHz

Commit message: added step file for arm-controller with minor changes
Parts:
- removed C11, C12: 100uF, rcl:CT6032
- added C22, C23: (no value), rcl:CT7343
- FB1: device Sparkfun Coils:0603 -> SPEAR:0603
- Q1: device crystal-geyer_V1_0:3.2X1.5 -> SPEAR:3.2X1.5
- S1: value SWS004 -> SMS-004; device smd-special:SMS-004 -> SPEAR:SMS-004
- S2: device SparkFun-Retired:TACTILE-SWITCH-SMD -> SPEAR:TACTILE_SWITCH_SMD_5.2MM
- U$4: device IAD-Library:TO252-3 -> SPEAR:TO252-3
- moved D2 5.03 mm to (16.9, 31.5), turned to 0 degrees
- moved LED2 0.13 mm to (59.1, 33.3)
Connections:
- net GND: now also C22.-, C23.-; no longer C11.-, C12.-
- net VOUT: now also C22.+, C23.+; no longer C11.+, C12.+
Routing:
- net AGND: track 2.45 -> 5.00 mm

Commit message: Changes to PCB Design
Parts:
- added CON2: SM04B-GHS-TB, SPEAR:SM04B-GHS-TB
- moved MOTOR 0.51 mm to (66.5, 21.6)
- renumbered MOTOR1 to VIN
Connections:
- removed net N$27: CON1.P$1, D1.A
- new net VCCCAN: CON1.P$1, CON2.P$1, D1.A
- net 3.3V: now also R3.2, R4.2
- net 5V: no longer R3.2, R4.2
- net CANH: now also CON2.P$2
- net CANL: now also CON2.P$3
- net GND: now also CON2.P$4, CON2.P$5, CON2.P$6
Routing:
- net 5V: track 89.7 -> 63.1 mm, vias 4 -> 2
- net 3.3V: track 148.5 -> 172.8 mm, vias 3 -> 5
- net CANH: track 5.05 -> 20.3 mm, vias 0 -> 2
- net CANL: track 9.57 -> 22.9 mm, vias 0 -> 2
- net VCCCAN: track 0.00 -> 13.3 mm
- net N$27: track 8.20 -> 0.00 mm
- net OUTA: track 30.4 -> 30.9 mm
- net VOUT: vias 57 -> 65
