File: arm-controller-stm32f103cbt6/Arm controller.sch (EAGLE design)
At the start: 59 parts, among them CON1 SM04B-GHS-TB, J1 CORTEX_DEBUG_SMD, Q1 32.768kHz, U1 3.3V, U2 3.3V, X1 8MHz

Commit message: added step file for arm-controller with minor changes
Parts:
- removed C11, C12: 100uF, rcl:CPOL-USCT6032
- added C22, C23: (no value), rcl:CPOL-USCT7343
- FB1: device Sparkfun Coils:FERRITE_BEAD-0603 -> SPEAR:FERRITE_BEAD-0603
- Q1: device crystal-geyer_V1_0:KX-327-NHT -> SPEAR:KX-327
- S1: value SWS004 -> SMS-004; device smd-special:SWS004 -> SPEAR:SMS-004
- S2: device SparkFun-Retired:TAC_SWITCHSMD -> SPEAR:MOMENTARY-SWITCH-SPST-2-SMD-5.2MM
- U$4: device IAD-Library:MOSFET-NCH -> SPEAR:MOSFET-NCH
Connections:
- net GND: now also C22.-, C23.-; no longer C11.-, C12.-
- net VOUT: now also C22.+, C23.+; no longer C11.+, C12.+
Changed lines of the file:
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@@
 <part name="C7" library="rcl" library_urn="urn:adsk.eagle:library:334" deviceset="C-EU" device="C0805" package3d_urn="urn:adsk.eagle:package:23617/2" value="20pF"/>
 <part name="GND3" library="SparkFun-PowerSymbols" deviceset="DGND" device=""/>
-<part name="J1" library="SparkFun-Connectors" library_urn="urn:adsk.eagle:library:4716215" deviceset="CORTEX_DEBUG" device="_SMD" package3d_urn="urn:adsk.eagle:package:4717419/1"/>
+<part name="J1" library="SparkFun-Connectors" library_urn="urn:adsk.eagle:library:4716215" deviceset="CORTEX_DEBUG" device="_SMD" package3d_urn="urn:adsk.eagle:package:4717419/2"/>
 <part name="SUPPLY2" library="SparkFun-PowerSymbols" deviceset="3.3V" device=""/>
-<part name="S1" library="smd-special" library_urn="urn:adsk.eagle:library:362" deviceset="SWS004" device="" package3d_urn="urn:adsk.eagle:package:26474/1"/>
-<part name="S2" library="SparkFun-Retired" deviceset="TAC_SWITCH" device="SMD" value="TAC_SWITCHSMD"/>
+<part name="S1" library="SPEAR" library_urn="urn:adsk.eagle:library:5549496" deviceset="SMS-004" device="" package3d_urn="urn:adsk.eagle:package:5592163/2"/>
+<part name="S2" library="SPEAR" library_urn="urn:adsk.eagle:library:5549496" deviceset="MOMENTARY-SWITCH-SPST-2" device="-SMD-5.2MM" package3d_urn="urn:adsk.eagle:package:5592178/3" value="TAC_SWITCHSMD"/>
 <part name="R3" library="rcl" library_urn="urn:adsk.eagle:library:334" deviceset="R-US_" device="R0805" package3d_urn="urn:adsk.eagle:package:23553/2" value="4.7k"/>
 <part name="R4" library="rcl" library_urn="urn:adsk.eagle:library:334" deviceset="R-US_" device="R0805" package3d_urn="urn:adsk.eagle:package:23553/2" value="4.7k"/>
@@
 <part name="R7" library="rcl" library_urn="urn:adsk.eagle:library:334" deviceset="R-US_" device="R0805" package3d_urn="urn:adsk.eagle:package:23553/2" value="1k"/>
 <part name="R8" library="rcl" library_urn="urn:adsk.eagle:library:334" deviceset="R-US_" device="R0805" package3d_urn="urn:adsk.eagle:package:23553/2" value="1k"/>
-<part name="U$4" library="IAD-Library" deviceset="MOSFET-NCH" device=""/>
+<part name="U$4" library="SPEAR" library_urn="urn:adsk.eagle:library:5549496" deviceset="MOSFET-NCH" device="" package3d_urn="urn:adsk.eagle:package:5592143/2"/>
 <part name="SUPPLY3" library="SparkFun-PowerSymbols" deviceset="VIN" device=""/>
 <part name="R10" library="rcl" library_urn="urn:adsk.eagle:library:334" deviceset="R-US_" device="R0805" package3d_urn="urn:adsk.eagle:package:23553/2" value="1k"/>
@@
 <part name="SUPPLY4" library="SparkFun-PowerSymbols" deviceset="VOUT" device=""/>
 <part name="SUPPLY5" library="SparkFun-PowerSymbols" deviceset="VOUT" device=""/>
-<part name="C11" library="rcl" library_urn="urn:adsk.eagle:library:334" deviceset="CPOL-US" device="CT6032" package3d_urn="urn:adsk.eagle:package:23305/2" value="100uF"/>
-<part name="C12" library="rcl" library_urn="urn:adsk.eagle:library:334" deviceset="CPOL-US" device="CT6032" package3d_urn="urn:adsk.eagle:package:23305/2" value="100uF"/>
 <part name="GND8" library="SparkFun-PowerSymbols" deviceset="DGND" device=""/>
-<part name="Q1" library="crystal-geyer_V1_0" library_urn="urn:adsk.eagle:library:203" deviceset="KX-327" device="-NHT" package3d_urn="urn:adsk.eagle:package:11937/1" value="32.768kHz"/>
+<part name="Q1" library="SPEAR" library_urn="urn:adsk.eagle:library:5549496" deviceset="KX-327" device="" package3d_urn="urn:adsk.eagle:package:5592245/2" value="32.768kHz"/>
 <part name="C14" library="rcl" library_urn="urn:adsk.eagle:library:334" deviceset="C-EU" device="C0805" package3d_urn="urn:adsk.eagle:package:23617/2" value="6pF"/>
 <part name="C15" library="rcl" library_urn="urn:adsk.eagle:library:334" deviceset="C-EU" device="C0805" package3d_urn="urn:adsk.eagle:package:23617/2" value="6pF"/>
@@
 <part name="U$5" library="SparkFun-PowerSymbols" deviceset="AGND" device=""/>
 <part name="U$6" library="SparkFun-PowerSymbols" deviceset="AGND" device=""/>
-<part name="FB1" library="Sparkfun Coils" deviceset="FERRITE_BEAD" device="-0603" value="30O/1.8A"/>
+<part name="FB1" library="SPEAR" library_urn="urn:adsk.eagle:library:5549496" deviceset="FERRITE_BEAD" device="-0603" package3d_urn="urn:adsk.eagle:package:5592201/2" value="30O/1.8A"/>
 <part name="P+3" library="supply1" library_urn="urn:adsk.eagle:library:371" deviceset="VCC" device=""/>
 <part name="U$9" library="SparkFun-PowerSymbols" deviceset="AGND" device=""/>
@@
 <part name="MOTOR1" library="SparkFun-Connectors" library_urn="urn:adsk.eagle:library:4716215" deviceset="CONN_02" device="5MM" package3d_urn="urn:adsk.eagle:package:4717103/2"/>
 <part name="SUPPLY21" library="SparkFun-PowerSymbols" deviceset="5V" device=""/>
+<part name="C22" library="rcl" library_urn="urn:adsk.eagle:library:334" deviceset="CPOL-US" device="CT7343" package3d_urn="urn:adsk.eagle:package:23304/2"/>
+<part name="C23" library="rcl" library_urn="urn:adsk.eagle:library:334" deviceset="CPOL-US" device="CT7343" package3d_urn="urn:adsk.eagle:package:23304/2"/>
 </parts>
 <sheets>
@@
 <instance part="SUPPLY2" gate="G$1" x="175.26" y="-12.7"/>
 <instance part="S1" gate="G$1" x="208.28" y="-53.34" rot="R270"/>
-<instance part="S2" gate="S" x="-5.08" y="121.92"/>
+<instance part="S2" gate="G$1" x="-5.08" y="121.92"/>
 <instance part="R3" gate="G$1" x="185.42" y="48.26" rot="R90"/>
 <instance part="R4" gate="G$1" x="195.58" y="48.26" rot="R90"/>
@@
 <instance part="SUPPLY4" gate="G$1" x="198.12" y="15.24"/>
 <instance part="SUPPLY5" gate="G$1" x="256.54" y="50.8"/>
-<instance part="C11" gate="G$1" x="213.36" y="5.08"/>
-<instance part="C12" gate="G$1" x="223.52" y="5.08"/>
 <instance part="GND8" gate="G$1" x="218.44" y="-7.62"/>
 <instance part="Q1" gate="G$1" x="-55.88" y="58.42"/>
@@
 <instance part="MOTOR1" gate="G$1" x="281.94" y="-78.74" rot="MR0"/>
 <instance part="SUPPLY21" gate="G$1" x="193.04" y="58.42"/>
+<instance part="C22" gate="G$1" x="213.36" y="5.08"/>
+<instance part="C23" gate="G$1" x="223.52" y="5.08"/>
 </instances>
 <busses>
@@
 </segment>
 <segment>
-<pinref part="C11" gate="G$1" pin="-"/>
 <wire x1="213.36" y1="0" x2="213.36" y2="-2.54" width="0.1524" layer="91"/>
-<pinref part="C12" gate="G$1" pin="-"/>
 <wire x1="213.36" y1="-2.54" x2="218.44" y2="-2.54" width="0.1524" layer="91"/>
 <wire x1="218.44" y1="-2.54" x2="223.52" y2="-2.54" width="0.1524" layer="91"/>
@@
 <wire x1="218.44" y1="-5.08" x2="218.44" y2="-2.54" width="0.1524" layer="91"/>
 <junction x="218.44" y="-2.54"/>
+<pinref part="C22" gate="G$1" pin="-"/>
+<pinref part="C23" gate="G$1" pin="-"/>
 </segment>
 <segment>
@@
 </segment>
 <segment>
-<pinref part="S2" gate="S" pin="4"/>
+<pinref part="S2" gate="G$1" pin="4"/>
 <wire x1="0" y1="119.38" x2="7.62" y2="119.38" width="0.1524" layer="91"/>
-<pinref part="S2" gate="S" pin="3"/>
+<pinref part="S2" gate="G$1" pin="3"/>
 <wire x1="7.62" y1="119.38" x2="20.32" y2="119.38" width="0.1524" layer="91"/>
 <wire x1="0" y1="121.92" x2="7.62" y2="121.92" width="0.1524" layer="91"/>
@@
 </segment>
 <segment>
-<pinref part="S2" gate="S" pin="1"/>
+<pinref part="S2" gate="G$1" pin="1"/>
 <wire x1="-10.16" y1="121.92" x2="-12.7" y2="121.92" width="0.1524" layer="91"/>
 <wire x1="-12.7" y1="121.92" x2="-15.24" y2="121.92" width="0.1524" layer="91"/>
 <wire x1="-15.24" y1="121.92" x2="-15.24" y2="119.38" width="0.1524" layer="91"/>
-<pinref part="S2" gate="S" pin="2"/>
+<pinref part="S2" gate="G$1" pin="2"/>
 <wire x1="-15.24" y1="119.38" x2="-10.16" y2="119.38" width="0.1524" layer="91"/>
 <wire x1="-15.24" y1="119.38" x2="-30.48" y2="119.38" width="0.1524" layer="91"/>
@@
 <wire x1="198.12" y1="15.24" x2="198.12" y2="10.16" width="0.1524" layer="91"/>
 <junction x="198.12" y="10.16"/>
-<pinref part="C11" gate="G$1" pin="+"/>
 <wire x1="213.36" y1="7.62" x2="213.36" y2="10.16" width="0.1524" layer="91"/>
 <junction x="213.36" y="10.16"/>
 <wire x1="218.44" y1="10.16" x2="223.52" y2="10.16" width="0.1524" layer="91"/>
-<pinref part="C12" gate="G$1" pin="+"/>
 <wire x1="223.52" y1="10.16" x2="223.52" y2="7.62" width="0.1524" layer="91"/>
 <wire x1="223.52" y1="10.16" x2="243.84" y2="10.16" width="0.1524" layer="91"/>
@@
 <wire x1="243.84" y1="10.16" x2="243.84" y2="7.62" width="0.1524" layer="91"/>
 <pinref part="C9" gate="G$1" pin="1"/>
-</segment>
-<segment>
+<pinref part="C22" gate="G$1" pin="+"/>
+<pinref part="C23" gate="G$1" pin="+"/>
+</segment>
+<segment>

Commit message: Changes to PCB Design
Parts:
- added CON2: SM04B-GHS-TB, SPEAR:SM04B-GHS-TB
- renumbered MOTOR1 to VIN
Connections:
- removed net N$27: CON1-1.S, D1.A
- new net VCCCAN: CON1-1.S, CON2-1.S, D1.A
- net 3.3V: now also R3.2, R4.2
- net 5V: no longer R3.2, R4.2
- net CANH: now also CON2-2.S
- net CANL: now also CON2-3.S
- net GND: now also CON2-4.S, CON2-TABS.S
