File: arm-controller-stm32f303cct6/Arm controller.brd (EAGLE design)
At the start: 67 x 65 mm, 61 parts, among them CON1 SM04B-GHS-TB, CON2 SM04B-GHS-TB, J1 CORTEX_DEBUG_SMD, Q1 32.768kHz, U1 3.3V, U2 3.3V, X1 8MHz

Commit message: Updated some parts of the library, with changes in added
Parts:
- removed C15: 6pF, rcl:C0805
- removed C16: 100nF, resistor:C0805
- removed C17: 10uF, resistor:C1206
- removed C18: 10uF, rcl:C1206
- removed D2: (no value), adafruit:SOD-123
- removed JP1: (no value), pinhead:1X04
- removed Q1: 32.768kHz, SPEAR:3.2X1.5
- added C11: 4.7uF, rcl:C0805
- added C12: 10uF, rcl:C0805
- added J-LINK: CORTEX_DEBUG_SMD, SparkFun-Connectors:SAMTECH_FTSH-105-01
- added LED4: (no value), led:CHIPLED_0805
- added R12, R15, R17, R19: 1k, rcl:R0805
- added R16, R20: 2k, rcl:R0805
- added R18: 3.3k, rcl:R0805
- added ST-LINK-V2: (no value), pinhead:1X04
- C14: value 6pF -> 10nF
- J1: value CORTEX_DEBUG_SMD -> 5-103669-4; device SparkFun-Connectors:SAMTECH_FTSH-105-01 -> SPEAR:TE_5-103669-4
- R14: value 17.4k -> 17k
- U$8: value 3.3UH-6045-3.6A -> 3015-INDUCTOR; device LCSC:INDC6161X450 -> LCSC:3015
- moved D1 32.6 mm to (17.0, 31.5), turned to 0 degrees
- moved C14 21.2 mm to (12.3, 35.2), turned to 270 degrees
- moved POTENT 10.3 mm to (58.7, 65.9), turned to 180 degrees
- moved BOOT0 8.51 mm to (49.9, 65.9)
- moved BOOT1 7.62 mm to (41.9, 65.9)
- moved J1 6.23 mm to (66.2, 43.6)
- moved R13 3.98 mm to (12.4, 39.5), turned to 270 degrees
- moved CON2 3.94 mm to (13.3, 65.3)
- moved R14 3.45 mm to (11.4, 42.5), turned to 0 degrees
- moved CON1 1.27 mm to (30.5, 65.3)
- moved U$8 0.85 mm to (17.8, 36.8)
- moved U$7 0.18 mm to (8.76, 35.2)
- renumbered S1 to ID_SELECTION
Connections:
- removed net N$13: C15.1, Q1.2, U$1.4
- removed net N$16: C16.2, D2.C, U$7.6, U$8.1
- removed net N$21: C16.1, U$7.1
- removed net VCCCAN: CON1.P$1, CON2.P$1, D1.A
- new net A: R17.2, R18.1, U$1.21
- new net B: R15.2, R16.2, U$1.22
- new net INDEX: R19.1, R20.1, U$1.17
- new net LED: LED4.C, U$1.29
- new net N$11: J1.3, R17.1
- new net N$15: J1.4, R19.2
- new net N$5: LED4.A, R12.1
- new net N$6: C14.2, D1.C, U$7.6, U$8.1
- new net N$7: J1.1, R15.1
- net 3.3V: now also J-LINK.1, R12.2, ST-LINK-V2.4; no longer J1.1, JP1.4
- net 5V: now also C12.1, CON1.P$1, CON2.P$1, J1.2; no longer C18.1, D1.C
- net GND: now also C11.2, C12.2, D1.A, J-LINK.3, J-LINK.5, J-LINK.9, R16.1, R18.2, R20.2, ST-LINK-V2.1; no longer C14.2, C15.2, C17.2, C18.2, D2.A, J1.3, J1.9, JP1.1
- net N$4: now also U$7.1; no longer Q1.1, U$1.3
- net RST: now also J-LINK.10; no longer J1.10
- net SWDCLK: now also J-LINK.4, ST-LINK-V2.2; no longer J1.4, JP1.2
- net SWDIO: now also J-LINK.2, ST-LINK-V2.3; no longer J1.2, JP1.3
- net VOUT: now also C11.1; no longer C17.1
Routing:
- net 5V: track 63.1 -> 139.5 mm
- net INDEX: track 0.00 -> 61.9 mm, vias 0 -> 2
- net LED: track 0.00 -> 42.5 mm, vias 0 -> 4
- net A: track 0.00 -> 32.4 mm, vias 0 -> 2
- net B: track 0.00 -> 26.5 mm, vias 0 -> 2
- net 3.3V: track 169.4 -> 193.4 mm, vias 5 -> 7
- net N$13: track 17.5 -> 0.00 mm
- net VCCCAN: track 13.3 -> 0.00 mm
- net N$4: track 14.7 -> 2.75 mm
- net BOOT0: track 33.9 -> 25.6 mm
- net SWDIO: track 37.9 -> 45.5 mm
- net N$8: track 4.16 -> 9.99 mm
- net BOOT1: track 40.7 -> 45.8 mm
- net N$11: track 0.00 -> 4.71 mm
- net CANL: track 22.9 -> 27.6 mm
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- added copper zone on layer 1, net N$6
- removed copper zone on layer 1, net N$16
Other:
- board text added: "GND"
- board text added: "V+"
- board text added: "V-"
- board text added: "V-\"
- board text added: "VIN: 4.5V -22V"
