File: arm-controller-stm32f303cct6/Arm controller.sch (EAGLE design)
At the start: 61 parts, among them CON1 SM04B-GHS-TB, CON2 SM04B-GHS-TB, J1 CORTEX_DEBUG_SMD, Q1 32.768kHz, U1 3.3V, U2 3.3V, X1 8MHz

Commit message: Updated some parts of the library, with changes in added
Parts:
- removed C15: 6pF, rcl:C-EUC0805
- removed C16: 100nF, resistor:C-EUC0805
- removed C17: 10uF, resistor:C-EUC1206
- removed C18: 10uF, rcl:C-EUC1206
- removed D2: (no value), adafruit:DIODESOD-123
- removed JP1: (no value), pinhead:PINHD-1X4
- removed Q1: 32.768kHz, SPEAR:KX-327
- removed S1: SMS-004, SPEAR:SMS-004
- added C11: 4.7uF, rcl:C-EUC0805
- added C12: 10uF, rcl:C-EUC0805
- added ID_SELECTION: SMS-004, SPEAR:SMS-004
- added J-LINK: CORTEX_DEBUG_SMD, SparkFun-Connectors:CORTEX_DEBUG_SMD
- added LED4: (no value), led:LEDCHIPLED_0805
- added R12, R15, R17, R19: 1k, rcl:R-US_R0805
- added R16, R20: 2k, rcl:R-US_R0805
- added R18: 3.3k, rcl:R-US_R0805
- added ST-LINK-V2: (no value), pinhead:PINHD-1X4
- C14: value 6pF -> 10nF
- J1: value CORTEX_DEBUG_SMD -> 5-103669-4; device SparkFun-Connectors:CORTEX_DEBUG_SMD -> SPEAR:5-103669-4
- R14: value 17.4k -> 17k
- U$8: value 3.3UH-6045-3.6A -> 3015-INDUCTOR; device LCSC:3.3UH-6045-3.6A -> LCSC:3015-INDUCTOR
Connections:
- removed net N$13: C15.1, Q1.2, U$1.PC15-OSC32_OUT
- removed net N$16: C16.2, D2.C, U$7.PHASE, U$8.1
- removed net N$21: C16.1, U$7.BOOT
- removed net VCCCAN: CON1-1.S, CON2-1.S, D1.A
- new net A: R17.2, R18.1, U$1.PB10/I2C2_SCL/USART3_TX
- new net B: R15.2, R16.2, U$1.PB11/I2C2_SDA/USART3_RX
- new net INDEX: R19.1, R20.1, U$1.PA7/SPI1_MOSI/ADC12_IN7/TIM3_CH2
- new net LED: LED4.C, U$1.PA8/USART1_CK/TIM1_CH1/MCO
- new net N$11: J1.3, R17.1
- new net N$15: J1.4, R19.2
- new net N$5: LED4.A, R12.1
- new net N$6: C14.2, D1.C, U$7.PHASE, U$8.1
- new net N$7: J1.1, R15.1
- net 3.3V: now also ID_SELECTION.5, ID_SELECTION.6, ID_SELECTION.7, ID_SELECTION.8, J-LINK.VCC, R12.2, ST-LINK-V2.4; no longer J1.VCC, JP1.4, S1.5, S1.6, S1.7, S1.8
- net 5V: now also C12.1, CON1-1.S, CON2-1.S, J1.2; no longer C18.1, D1.C
- net GND: now also C11.2, C12.2, D1.A, J-LINK.GND@3, J-LINK.GND@5, J-LINK.GNDDTCT, J1.5, R16.1, R18.2, R20.2, ST-LINK-V2.1; no longer C14.2, C15.2, C17.2, C18.2, D2.A, J1.GND@3, J1.GND@5, J1.GNDDTCT, JP1.1
- net N$4: now also U$7.BOOT; no longer Q1.1, U$1.PC14-OSC32_IN
- net NODE1: now also ID_SELECTION.1; no longer S1.1
- net NODE2: now also ID_SELECTION.2; no longer S1.2
- net NODE3: now also ID_SELECTION.3; no longer S1.3
- net NODE4: now also ID_SELECTION.4; no longer S1.4
- net RST: now also J-LINK.!RESET; no longer J1.!RESET
- net SWDCLK: now also J-LINK.SWDCLK/TCK, ST-LINK-V2.2; no longer J1.SWDCLK/TCK, JP1.2
- net SWDIO: now also J-LINK.SWDIO/TMS, ST-LINK-V2.3; no longer J1.SWDIO/TMS, JP1.3
- net VOUT: now also C11.1; no longer C17.1
Other:
- note added: "CAN Bus Tranceiver (MCP2562)"
- note added: "LEDS"
- note added: "MCU (STM32F303CCT6/STM32F103CBT6)"
- note added: "Motor Driver (VNH5019)"
- note added: "Pinout"
- note added: "Power Regulator (RT6200 + AP2112 or RT9193)"
- note added: "Programming Port (ST - Link V2 and J Link Edu)"
- note added: "VIN: 4.5V - 22V"
- moved on the sheet: BOOT0, BOOT1, C1, C10, C13, C14, C19, C2, C20, C21, C22, C23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
