File: arm-controller-stm32f303cct6/Arm controller Mega.brd (EAGLE design)
At the start: 100 x 100 mm, 67 parts, among them CON1 SM04B-GHS-TB, CON2 SM04B-GHS-TB, J4 5-103669-4, J5 5-103669-4, U1 STM32F303RET6, U2 3.3V, X1 8MHz

Commit message: changes based on last pull request enter the commit message for your changes. Lines starting
Parts:
- moved J1 41.8 mm to (3.56, 22.5), turned to 270 degrees
- moved J6 40.9 mm to (3.56, 38.2), turned to 270 degrees
- moved J3 5.61 mm to (96.0, 33.0)
- moved U$1 5.61 mm to (69.3, 33.5)
- moved R7 5.43 mm to (56.3, 45.6)
- moved R9 5.31 mm to (53.5, 45.6)
- moved R6 5.25 mm to (66.2, 45.6)
- moved R13 5.25 mm to (59.1, 45.6)
- moved R4 5.25 mm to (63.8, 45.6)
- moved R5 5.25 mm to (61.5, 45.6)
- moved R8 5.25 mm to (45.3, 45.6)
- moved R12 5.25 mm to (68.5, 45.6)
- moved R17 5.22 mm to (50.7, 45.6)
- moved R16 5.21 mm to (48.0, 45.6)
- moved J2 4.33 mm to (96.3, 15.5)
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Routing:
- net OUTB1: track 0.00 -> 18.8 mm
- net OUTA1: track 0.00 -> 17.6 mm
- net INA1: track 55.2 -> 40.6 mm, vias 0 -> 2
- net N$14: track 60.8 -> 52.6 mm
- net VIN: track 39.1 -> 46.3 mm, vias 2 -> 4
- net PWM2: track 19.4 -> 12.3 mm
- net INB1: track 53.8 -> 47.6 mm
- net ENB1: track 18.5 -> 12.6 mm
- net PWM1: track 23.8 -> 18.0 mm
- net N$8: track 45.4 -> 39.7 mm
- net N$15: track 14.9 -> 19.9 mm
- net VOUT: track 9.71 -> 14.4 mm
- net ENA1: track 27.1 -> 22.4 mm
- net ENB2: track 19.5 -> 14.9 mm
- net +3V3: track 255.1 -> 250.9 mm
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
Commit message: Simplified resistors to 1k or 10k
Parts:
- R5, R6, R8, R9: value 4.7k -> 10k
Changed lines of the file:
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@@
 <?xml version="1.0" encoding="utf-8"?>
 <!DOCTYPE eagle SYSTEM "eagle.dtd">
-<eagle version="9.3.1">
+<eagle version="9.4.1">
 <drawing>
 <settings>
-<setting alwaysvectorfont="yes"/>
+<setting alwaysvectorfont="no"/>
 <setting verticaltext="up"/>
 </settings>
-<grid distance="5" unitdist="mil" unit="mil" style="lines" multiple="1" display="yes" altdistance="5" altunitdist="mil" altunit="mil"/>
+<grid distance="0.1" unitdist="mm" unit="mm" style="lines" multiple="1" display="yes" altdistance="5" altunitdist="mil" altunit="mil"/>
 <layers>
 <layer number="1" name="Top" color="4" fill="1" visible="yes" active="yes"/>
@@
 <attribute name="SPICEPREFIX" value="R" x="136.144" y="65.913" size="1.778" layer="27" rot="R90" display="off"/>
 </element>
-<element name="R5" library="rcl" library_urn="urn:adsk.eagle:library:334" package="R0805" package3d_urn="urn:adsk.eagle:package:23553/2" value="4.7k" x="61.468" y="45.593" smashed="yes" rot="R90">
+<element name="R5" library="rcl" library_urn="urn:adsk.eagle:library:334" package="R0805" package3d_urn="urn:adsk.eagle:package:23553/2" value="10k" x="61.468" y="45.593" smashed="yes" rot="R90">
 <attribute name="NAME" x="60.833" y="47.879" size="0.8128" layer="25"/>
 <attribute name="SPICEPREFIX" value="R" x="121.158" y="120.523" size="1.778" layer="27" rot="R90" display="off"/>
 </element>
-<element name="R6" library="rcl" library_urn="urn:adsk.eagle:library:334" package="R0805" package3d_urn="urn:adsk.eagle:package:23553/2" value="4.7k" x="66.167" y="45.593" smashed="yes" rot="R90">
+<element name="R6" library="rcl" library_urn="urn:adsk.eagle:library:334" package="R0805" package3d_urn="urn:adsk.eagle:package:23553/2" value="10k" x="66.167" y="45.593" smashed="yes" rot="R90">
 <attribute name="NAME" x="65.659" y="47.879" size="0.8128" layer="25"/>
 <attribute name="SPICEPREFIX" value="R" x="125.857" y="126.873" size="1.778" layer="27" rot="R90" display="off"/>
@@
 <attribute name="SPICEPREFIX" value="R" x="128.651" y="70.993" size="1.778" layer="27" rot="R90" display="off"/>
 </element>
-<element name="R8" library="rcl" library_urn="urn:adsk.eagle:library:334" package="R0805" package3d_urn="urn:adsk.eagle:package:23553/2" value="4.7k" x="45.339" y="45.593" smashed="yes" rot="R90">
+<element name="R8" library="rcl" library_urn="urn:adsk.eagle:library:334" package="R0805" package3d_urn="urn:adsk.eagle:package:23553/2" value="10k" x="45.339" y="45.593" smashed="yes" rot="R90">
 <attribute name="NAME" x="44.323" y="47.879" size="0.8128" layer="25"/>
 <attribute name="SPICEPREFIX" value="R" x="111.379" y="62.103" size="1.778" layer="27" rot="R90" display="off"/>
 </element>
-<element name="R9" library="rcl" library_urn="urn:adsk.eagle:library:334" package="R0805" package3d_urn="urn:adsk.eagle:package:23553/2" value="4.7k" x="53.467" y="45.593" smashed="yes" rot="R90">
+<element name="R9" library="rcl" library_urn="urn:adsk.eagle:library:334" package="R0805" package3d_urn="urn:adsk.eagle:package:23553/2" value="10k" x="53.467" y="45.593" smashed="yes" rot="R90">
 <attribute name="NAME" x="52.959" y="47.879" size="0.8128" layer="25"/>
 <attribute name="SPICEPREFIX" value="R" x="119.507" y="68.453" size="1.778" layer="27" rot="R90" display="off"/>

Commit message: Some more changes
Parts:
- added C16, C17: 0u1, resistor:C0805
Connections:
- net +3V3: now also C17.1
- net +5V: now also C16.1
- net GND: now also C16.2, C17.2
