File: arm-controller-stm32f303cct6/Arm controller Mega.sch (EAGLE design)
At the start: 67 parts, among them CON1 SM04B-GHS-TB, CON2 SM04B-GHS-TB, J4 5-103669-4, J5 5-103669-4, U1 STM32F303RET6, U2 3.3V, X1 8MHz

Commit message: changes based on last pull request enter the commit message for your changes. Lines starting
Other:
- note added: "2 AMP DUPONT"
- note added: "CAN BUS"
- note added: "ID SELECTION"
- note added: "Main MCU"
- note added: "Motor Driver"
- note added: "POWER SUPPLY"
- moved on the sheet: C1, C10, C11, C12, C13, C14, C15, C2, C3, C4, C5, C6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

Commit message: Simplified resistors to 1k or 10k
Parts:
- R5, R6, R8, R9: value 4.7k -> 10k
Changed lines of the file:
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@@
 <?xml version="1.0" encoding="utf-8"?>
 <!DOCTYPE eagle SYSTEM "eagle.dtd">
-<eagle version="9.3.1">
+<eagle version="9.4.1">
 <drawing>
 <settings>
@@
 <part name="GND14" library="SparkFun-PowerSymbols" deviceset="DGND" device=""/>
 <part name="R4" library="rcl" library_urn="urn:adsk.eagle:library:334" deviceset="R-US_" device="R0805" package3d_urn="urn:adsk.eagle:package:23553/2" value="1k"/>
-<part name="R5" library="rcl" library_urn="urn:adsk.eagle:library:334" deviceset="R-US_" device="R0805" package3d_urn="urn:adsk.eagle:package:23553/2" value="4.7k"/>
-<part name="R6" library="rcl" library_urn="urn:adsk.eagle:library:334" deviceset="R-US_" device="R0805" package3d_urn="urn:adsk.eagle:package:23553/2" value="4.7k"/>
+<part name="R5" library="rcl" library_urn="urn:adsk.eagle:library:334" deviceset="R-US_" device="R0805" package3d_urn="urn:adsk.eagle:package:23553/2" value="10k"/>
+<part name="R6" library="rcl" library_urn="urn:adsk.eagle:library:334" deviceset="R-US_" device="R0805" package3d_urn="urn:adsk.eagle:package:23553/2" value="10k"/>
 <part name="+3V10" library="supply1" library_urn="urn:adsk.eagle:library:371" deviceset="+3V3" device=""/>
 <part name="R7" library="rcl" library_urn="urn:adsk.eagle:library:334" deviceset="R-US_" device="R0805" package3d_urn="urn:adsk.eagle:package:23553/2" value="1k"/>
-<part name="R8" library="rcl" library_urn="urn:adsk.eagle:library:334" deviceset="R-US_" device="R0805" package3d_urn="urn:adsk.eagle:package:23553/2" value="4.7k"/>
-<part name="R9" library="rcl" library_urn="urn:adsk.eagle:library:334" deviceset="R-US_" device="R0805" package3d_urn="urn:adsk.eagle:package:23553/2" value="4.7k"/>
+<part name="R8" library="rcl" library_urn="urn:adsk.eagle:library:334" deviceset="R-US_" device="R0805" package3d_urn="urn:adsk.eagle:package:23553/2" value="10k"/>
+<part name="R9" library="rcl" library_urn="urn:adsk.eagle:library:334" deviceset="R-US_" device="R0805" package3d_urn="urn:adsk.eagle:package:23553/2" value="10k"/>
 <part name="+3V11" library="supply1" library_urn="urn:adsk.eagle:library:371" deviceset="+3V3" device=""/>
 <part name="U$3" library="SPEAR" library_urn="urn:adsk.eagle:library:5549496" deviceset="MOSFET-NCH" device="" package3d_urn="urn:adsk.eagle:package:5592143/2"/>

Commit message: Some more changes
Parts:
- added C16, C17: 0u1, resistor:C-EUC0805
Connections:
- net +3V3: now also C17.1
- net +5V: now also C16.1
- net GND: now also C16.2, C17.2
Changed lines of the file:
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@@
 <part name="JP4" library="SparkFun-Jumpers" deviceset="JUMPER-SMT_2_NO" device="_NO-SILK"/>
 <part name="FRAME1" library="frames" library_urn="urn:adsk.eagle:library:229" deviceset="FRAME_C_L" device=""/>
+<part name="C16" library="resistor" library_urn="urn:adsk.eagle:library:348" deviceset="C-EU" device="C0805" package3d_urn="urn:adsk.eagle:package:23617/2" value="0u1"/>
+<part name="C17" library="resistor" library_urn="urn:adsk.eagle:library:348" deviceset="C-EU" device="C0805" package3d_urn="urn:adsk.eagle:package:23617/2" value="0u1"/>
+<part name="GND19" library="SparkFun-PowerSymbols" deviceset="DGND" device=""/>
+<part name="P+7" library="supply1" library_urn="urn:adsk.eagle:library:371" deviceset="+5V" device=""/>
+<part name="+3V18" library="supply1" library_urn="urn:adsk.eagle:library:371" deviceset="+3V3" device=""/>
 </parts>
 <sheets>
@@
 <attribute name="DRAWING_NAME" x="162.56" y="-196.85" size="2.54" layer="94"/>
 </instance>
+<instance part="C16" gate="G$1" x="-121.92" y="-175.26" smashed="yes">
+<attribute name="NAME" x="-120.396" y="-174.879" size="1.778" layer="95"/>
+<attribute name="VALUE" x="-120.396" y="-179.959" size="1.778" layer="96"/>
+</instance>
+<instance part="C17" gate="G$1" x="-114.3" y="-175.26" smashed="yes">
+<attribute name="NAME" x="-112.776" y="-174.879" size="1.778" layer="95"/>
+<attribute name="VALUE" x="-112.776" y="-179.959" size="1.778" layer="96"/>
+</instance>
+<instance part="GND19" gate="G$1" x="-114.3" y="-187.96" smashed="yes">
+<attribute name="VALUE" x="-114.3" y="-188.214" size="1.778" layer="96" align="top-center"/>
+</instance>
+<instance part="P+7" gate="1" x="-121.92" y="-170.18" smashed="yes">
+<attribute name="VALUE" x="-124.46" y="-175.26" size="1.778" layer="96" rot="R90"/>
+</instance>
+<instance part="+3V18" gate="G$1" x="-114.3" y="-170.18" smashed="yes">
+<attribute name="VALUE" x="-116.84" y="-175.26" size="1.778" layer="96" rot="R90"/>
+</instance>
 </instances>
 <busses>
@@
 <junction x="213.36" y="-121.92"/>
 </segment>
+<segment>
+<pinref part="C17" gate="G$1" pin="1"/>
+<pinref part="+3V18" gate="G$1" pin="+3V3"/>
+</segment>
 </net>
 <net name="GND" class="0">
@@
 <junction x="-144.78" y="-142.24"/>
 </segment>
+<segment>
+<pinref part="C16" gate="G$1" pin="2"/>
+<pinref part="C17" gate="G$1" pin="2"/>
+<wire x1="-121.92" y1="-180.34" x2="-114.3" y2="-180.34" width="0.1524" layer="91"/>
+<wire x1="-114.3" y1="-180.34" x2="-114.3" y2="-185.42" width="0.1524" layer="91"/>
+<junction x="-114.3" y="-180.34"/>
+<pinref part="GND19" gate="G$1" pin="GND"/>
+</segment>
 </net>
 <net name="N$3" class="0">
@@
 <wire x1="-142.24" y1="-121.92" x2="-142.24" y2="-111.76" width="0.1524" layer="91"/>
 </segment>
+<segment>
+<pinref part="C16" gate="G$1" pin="1"/>
+<pinref part="P+7" gate="1" pin="+5V"/>
+</segment>
 </net>
