File: arm-controller-stm32f303cct6/arm controller single.brd (EAGLE design)
At the start: 100 x 50 mm, 32 parts, among them IC1 NC7SZ157P6X, IC2 DRV8701PRGER, IC3 TS5A3357DCUT, J3 5-103669-4

Commit message: fixed wire stub, changes based on request
Parts:
- removed C5: 100nF, rcl:C0805
- R3: value 0.01 -> 0.005
- moved R1 28.3 mm to (49.0, 18.5), turned to 180 degrees
- moved C11 10.8 mm to (62.9, 25.4), turned to 180 degrees
- moved R5 2.16 mm to (49.0, 16.4)
- moved R4 2.16 mm to (49.0, 11.8)
- moved R6 2.16 mm to (49.0, 14.1)
- moved C9 1.55 mm to (77.0, 22.1)
Connections:
- new net DAC: IC2.6, JP3.12
- net +3V3: no longer C5.1, IC2.6
- net GND: no longer C5.2
- net SNSOUT: now also JP4.18; no longer JP3.15
- net SO: now also JP3.15; no longer JP3.12
Routing:
- net DAC: track 0.00 -> 49.0 mm, vias 0 -> 2
- net SNSOUT: track 44.8 -> 61.2 mm, vias 2 -> 1
- net +3V3: track 163.2 -> 149.0 mm
- net SO: track 50.8 -> 47.5 mm
- net IN1: track 35.8 -> 37.4 mm
- net SLEEP: track 37.1 -> 38.6 mm
- net IN2: track 33.3 -> 34.6 mm
- net GL2: track 28.3 -> 29.4 mm
- net SP: track 20.9 -> 21.8 mm
- net N$11: track 7.98 -> 7.09 mm
- net IDRIVE: track 7.36 -> 8.26 mm
- net GH2: track 34.3 -> 34.9 mm
- net GND: track 6.89 -> 7.17 mm, vias 85 -> 146
