File: arm-controller-stm32f303cct6/arm controller single.brd (EAGLE design)
At the start: 100 x 50 mm, 31 parts, among them IC1 NC7SZ157P6X, IC2 DRV8701PRGER, IC3 TS5A3357DCUT, J3 5-103669-4

Commit message: fixed DRC
Parts:
- R3: device rcl:R2512 -> rcl:WSC4527
- moved R4 0.13 mm to (49.0, 11.9)
Routing:
- net GND: track 7.17 -> 0.00 mm, vias 146 -> 149
- net SO: track 47.5 -> 48.2 mm
