File: arm-controller-stm32f303cct6/arm controller single v1.1.brd (EAGLE design)
At the start: 100 x 50 mm, 49 parts, among them IC1 NC7SZ157P6X, IC2 DRV8701PRGER, IC3 TS5A3357DCUT, J1 1017503, J2 1017503, J3 5-103669-4, U1 4MB Flash

Commit message: changes for better load
Parts:
- added C18: 680uF, rcl:E5-10,5
- C5, C6: value 1000uF -> 680uF
- moved C5 4.19 mm to (71.9, 5.33)
- moved C11 4.06 mm to (79.6, 4.70)
Connections:
- net GND: now also C18.-
- net VIN: now also C18.+
Routing:
- net N$12: vias 0 -> 16
- added copper zone on layer 16, net N$12
Changed lines of the file:
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@@
 </layers>
 <board>
-<fusionsync huburn="a.cGVyc29uYWw6dWUyODBmY2U1" projecturn="a.cGVyc29uYWw6dWUyODBmY2U1IzIwMTYxMjExNTQ1ODE1NTE" f3durn="urn:adsk.wipprod:dm.lineage:ojb-Q2_iSFqqAIA-rjsEgw" pcbguid="0204553a-29ea-480a-9da3-94c9a21dd363" lastpulledtime="" lastsyncedchangeguid="fb8cb836-21fe-dc68-fe53-1fd710d2f1c4"/>
+<fusionsync huburn="a.cGVyc29uYWw6dWUyODBmY2U1" projecturn="a.cGVyc29uYWw6dWUyODBmY2U1IzIwMTYxMjExNTQ1ODE1NTE" f3durn="urn:adsk.wipprod:dm.lineage:ojb-Q2_iSFqqAIA-rjsEgw" pcbguid="0204553a-29ea-480a-9da3-94c9a21dd363" lastpulledtime="" lastsyncedchangeguid="38305143-55cc-b8b2-b888-7ce595eec31e"/>
 <plain>
 <wire x1="0" y1="50" x2="0" y2="5" width="0" layer="20"/>
@@
 <wire x1="83.566" y1="7.874" x2="88.011" y2="12.7" width="3.048" layer="30"/>
 <wire x1="67.691" y1="7.874" x2="83.566" y2="7.874" width="3.048" layer="30"/>
-<wire x1="47.371" y1="9.144" x2="67.183" y2="9.144" width="3.048" layer="30"/>
-<wire x1="67.183" y1="9.144" x2="68.199" y2="7.747" width="3.048" layer="30"/>
 <wire x1="76.835" y1="25.4" x2="76.835" y2="16.129" width="2.54" layer="30"/>
 <wire x1="91.885" y1="23.241" x2="83.185" y2="23.241" width="2.54" layer="30"/>
@@
 <text x="67.31" y="34.544" size="1.27" layer="25">V1.1</text>
 <text x="51.943" y="34.417" size="1.27" layer="25">minh7a6</text>
+<wire x1="37.084" y1="7.937" x2="37.084" y2="16.637" width="2.54" layer="30"/>
+<wire x1="60.96" y1="7.874" x2="71.882" y2="7.874" width="2.54" layer="30"/>
+<wire x1="51.435" y1="9.652" x2="48.133" y2="9.652" width="3.048" layer="30"/>
+<wire x1="53.213" y1="7.874" x2="51.435" y2="9.652" width="3.048" layer="30"/>
+<wire x1="60.96" y1="7.874" x2="53.213" y2="7.874" width="3.048" layer="30"/>
+<wire x1="60.96" y1="7.874" x2="71.882" y2="7.874" width="3.048" layer="30"/>
 </plain>
 <attributes>
@@
 <attribute name="SPICEPREFIX" value="C" x="-13.589" y="9.271" size="1.778" layer="27" rot="R270" display="off"/>
 </element>
-<element name="C11" library="rcl" library_urn="urn:adsk.eagle:library:334" package="C0603" package3d_urn="urn:adsk.eagle:package:23616/2" value="100nF" x="75.565" y="4.699" smashed="yes" rot="R270">
-<attribute name="NAME" x="74.041" y="6.477" size="1.27" layer="25"/>
-<attribute name="POPULARITY" value="73" x="-8.255" y="-35.941" size="1.778" layer="27" rot="R270" display="off"/>
-<attribute name="SPICEPREFIX" value="C" x="-8.255" y="-35.941" size="1.778" layer="27" rot="R270" display="off"/>
+<element name="C11" library="rcl" library_urn="urn:adsk.eagle:library:334" package="C0603" package3d_urn="urn:adsk.eagle:package:23616/2" value="100nF" x="79.629" y="4.699" smashed="yes" rot="R270">
+<attribute name="NAME" x="78.105" y="6.477" size="1.27" layer="25"/>
+<attribute name="POPULARITY" value="73" x="-4.191" y="-35.941" size="1.778" layer="27" rot="R270" display="off"/>
+<attribute name="SPICEPREFIX" value="C" x="-4.191" y="-35.941" size="1.778" layer="27" rot="R270" display="off"/>
 </element>
 <element name="C12" library="rcl" library_urn="urn:adsk.eagle:library:334" package="C0603" package3d_urn="urn:adsk.eagle:package:23616/2" value="100nF" x="46.609" y="30.734" smashed="yes">
@@
 <attribute name="SPICEPREFIX" value="C" x="-18.669" y="107.569" size="1.778" layer="27" rot="R180" display="off"/>
 </element>
-<element name="C5" library="rcl" library_urn="urn:adsk.eagle:library:334" package="E5-10,5" package3d_urn="urn:adsk.eagle:package:23372/2" value="1000uF" x="67.691" y="5.334" smashed="yes" rot="R270">
-<attribute name="NAME" x="66.167" y="11.049" size="1.778" layer="25" ratio="10"/>
-<attribute name="POPULARITY" value="12" x="58.801" y="-48.006" size="1.778" layer="27" rot="R270" display="off"/>
-<attribute name="SPICEPREFIX" value="C" x="58.801" y="-48.006" size="1.778" layer="27" rot="R270" display="off"/>
-</element>
-<element name="C6" library="rcl" library_urn="urn:adsk.eagle:library:334" package="E5-10,5" package3d_urn="urn:adsk.eagle:package:23372/2" value="1000uF" x="77.597" y="44.45" smashed="yes" rot="R90">
+<element name="C5" library="rcl" library_urn="urn:adsk.eagle:library:334" package="E5-10,5" package3d_urn="urn:adsk.eagle:package:23372/2" value="680uF" x="71.882" y="5.334" smashed="yes" rot="R270">
+<attribute name="NAME" x="70.358" y="11.049" size="1.778" layer="25" ratio="10"/>
+<attribute name="POPULARITY" value="12" x="62.992" y="-48.006" size="1.778" layer="27" rot="R270" display="off"/>
+<attribute name="SPICEPREFIX" value="C" x="62.992" y="-48.006" size="1.778" layer="27" rot="R270" display="off"/>
+</element>
+<element name="C6" library="rcl" library_urn="urn:adsk.eagle:library:334" package="E5-10,5" package3d_urn="urn:adsk.eagle:package:23372/2" value="680uF" x="77.597" y="44.45" smashed="yes" rot="R90">
 <attribute name="NAME" x="83.312" y="43.942" size="1.778" layer="25" ratio="10"/>
 <attribute name="POPULARITY" value="12" x="86.487" y="118.11" size="1.778" layer="27" rot="R90" display="off"/>
@@
 <attribute name="SPICEPREFIX" value="R" x="16.764" y="6.731" size="1.778" layer="27" display="off"/>
 <attribute name="VALUE" x="16.129" y="4.826" size="1.27" layer="27"/>
+</element>
+<element name="C18" library="rcl" library_urn="urn:adsk.eagle:library:334" package="E5-10,5" package3d_urn="urn:adsk.eagle:package:23372/2" value="680uF" x="60.96" y="5.334" smashed="yes" rot="R270">
+<attribute name="NAME" x="59.309" y="11.1252" size="1.27" layer="25" ratio="10"/>
+<attribute name="POPULARITY" value="12" x="60.96" y="5.334" size="1.778" layer="27" rot="R270" display="off"/>
+<attribute name="SPICEPREFIX" value="C" x="60.96" y="5.334" size="1.778" layer="27" rot="R270" display="off"/>
+<attribute name="VALUE" x="57.7342" y="8.4582" size="1.27" layer="27" ratio="10" rot="R270"/>
 </element>
 </elements>
@@
 <via x="7.366" y="10.033" extent="1-16" drill="0.35"/>
 <via x="43.307" y="21.336" extent="1-16" drill="0.35"/>
-<via x="58.928" y="2.667" extent="1-16" drill="0.35"/>
+<via x="56.134" y="2.667" extent="1-16" drill="0.35"/>
 <via x="52.578" y="1.397" extent="1-16" drill="0.35"/>
 <via x="34.544" y="3.048" extent="1-16" drill="0.35"/>
@@
 <via x="98.171" y="6.985" extent="1-16" drill="0.35"/>
 <via x="96.393" y="8.001" extent="1-16" drill="0.35"/>
+<contactref element="C18" pad="-"/>
 </signal>
 <signal name="IN1">
@@
 <via x="88.011" y="11.303" extent="1-16" drill="0.35"/>
 <via x="86.868" y="11.303" extent="1-16" drill="0.35"/>
+<via x="84.328" y="7.366" extent="1-16" drill="0.35"/>
+<via x="92.583" y="8.128" extent="1-16" drill="0.35"/>
+<via x="95.123" y="14.732" extent="1-16" drill="0.35"/>
+<via x="97.663" y="17.907" extent="1-16" drill="0.35"/>
+<via x="95.504" y="26.035" extent="1-16" drill="0.35"/>
+<via x="98.044" y="21.336" extent="1-16" drill="0.35"/>
+<via x="97.282" y="27.305" extent="1-16" drill="0.35"/>
+<via x="96.266" y="37.338" extent="1-16" drill="0.35"/>
+<via x="88.138" y="41.275" extent="1-16" drill="0.35"/>
+<via x="77.089" y="38.608" extent="1-16" drill="0.35"/>
+<via x="79.248" y="40.894" extent="1-16" drill="0.35"/>
+<via x="75.692" y="40.386" extent="1-16" drill="0.35"/>
+<via x="75.565" y="42.291" extent="1-16" drill="0.35"/>
+<via x="78.105" y="39.243" extent="1-16" drill="0.35"/>
+<via x="79.756" y="38.608" extent="1-16" drill="0.35"/>
+<via x="81.788" y="37.084" extent="1-16" drill="0.35"/>
+<via x="92.329" y="37.084" extent="1-16" drill="0.35"/>
+<via x="96.52" y="32.258" extent="1-16" drill="0.35"/>
+<via x="95.377" y="28.956" extent="1-16" drill="0.35"/>
+<via x="97.79" y="29.845" extent="1-16" drill="0.35"/>
+<via x="97.917" y="39.751" extent="1-16" drill="0.35"/>
+<via x="91.059" y="40.132" extent="1-16" drill="0.35"/>
+<via x="87.503" y="8.001" extent="1-16" drill="0.35"/>
+<via x="80.518" y="8.89" extent="1-16" drill="0.35"/>
+<via x="57.785" y="9.271" extent="1-16" drill="0.35"/>
+<via x="54.61" y="6.096" extent="1-16" drill="0.35"/>
+<via x="57.404" y="5.588" extent="1-16" drill="0.35"/>
+<via x="53.721" y="9.017" extent="1-16" drill="0.35"/>
+<via x="89.916" y="9.144" extent="1-16" drill="0.35"/>
+<via x="89.535" y="6.604" extent="1-16" drill="0.35"/>
+<via x="85.852" y="5.715" extent="1-16" drill="0.35"/>
+<via x="93.853" y="11.303" extent="1-16" drill="0.35"/>
+<via x="93.091" y="13.462" extent="1-16" drill="0.35"/>
+<contactref element="C18" pad="+"/>
 </signal>
 <signal name="SO">
@@
 <vertex x="34.29" y="5.969"/>
 </polygon>
+<polygon width="0.1524" layer="16" thermals="no">
+<vertex x="34.163" y="19.939"/>
+<vertex x="34.163" y="6.35"/>
+<vertex x="34.925" y="5.588"/>
+<vertex x="44.069" y="5.588"/>
+<vertex x="44.831" y="6.35"/>
+<vertex x="44.831" y="19.939"/>
+<vertex x="44.704" y="20.066"/>
+<vertex x="34.29" y="20.066"/>
+</polygon>
+<via x="40.894" y="17.145" extent="1-16" drill="0.35"/>
+<via x="43.434" y="18.161" extent="1-16" drill="0.35"/>
+<via x="42.291" y="13.462" extent="1-16" drill="0.35"/>
+<via x="40.894" y="11.684" extent="1-16" drill="0.35"/>
+<via x="41.529" y="9.652" extent="1-16" drill="0.35"/>
+<via x="42.291" y="7.747" extent="1-16" drill="0.35"/>
+<via x="42.799" y="10.795" extent="1-16" drill="0.35"/>
+<via x="40.259" y="15.367" extent="1-16" drill="0.35"/>
+<via x="42.672" y="16.51" extent="1-16" drill="0.35"/>
+<via x="41.91" y="18.161" extent="1-16" drill="0.35"/>
+<via x="40.005" y="13.589" extent="1-16" drill="0.35"/>
+<via x="39.37" y="10.033" extent="1-16" drill="0.35"/>
+<via x="39.878" y="8.255" extent="1-16" drill="0.35"/>
+<via x="42.418" y="14.732" extent="1-16" drill="0.35"/>
+<via x="40.513" y="6.35" extent="1-16" drill="0.35"/>
+<via x="40.64" y="18.923" extent="1-16" drill="0.35"/>
 </signal>
 <signal name="PB6">

Commit message: changed layout to fit the CAN Connector
Parts:
- added JP6: (no value), pinhead:1X02
- moved R10 7.50 mm to (23.5, 10.0), turned to 90 degrees
Connections:
- net CANH: now also JP6.1
- net CANL: now also JP6.2
Routing:
- net CANH: track 46.1 -> 56.9 mm, vias 2 -> 1
- net CANL: track 56.5 -> 65.7 mm
- net N$10: track 3.84 -> 10.9 mm
- net PB0: track 36.7 -> 35.9 mm
- net SLEEP: track 50.7 -> 50.1 mm
