File: arm-controller-stm32f303cct6/arm controller single v1.1.sch (EAGLE design)
At the start: 49 parts, among them IC1 NC7SZ157P6X, IC2 DRV8701PRGER, IC3 TS5A3357DCUT, J1 1017503, J2 1017503, J3 5-103669-4, U1 4MB Flash

Commit message: changes for better load
Parts:
- added C18: 680uF, rcl:CPOL-USE5-10.5
- C5, C6: value 1000uF -> 680uF
Connections:
- net GND: now also C18.-
- net VIN: now also C18.+
Changed lines of the file:
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@@
 <part name="LED1" library="led" library_urn="urn:adsk.eagle:library:259" deviceset="LED" device="CHIP-LED0805" package3d_urn="urn:adsk.eagle:package:15818/2"/>
 <part name="GND12" library="SparkFun-PowerSymbols" deviceset="DGND" device=""/>
-<part name="C5" library="rcl" library_urn="urn:adsk.eagle:library:334" deviceset="CPOL-US" device="E5-10.5" package3d_urn="urn:adsk.eagle:package:23372/2" value="1000uF"/>
-<part name="C6" library="rcl" library_urn="urn:adsk.eagle:library:334" deviceset="CPOL-US" device="E5-10.5" package3d_urn="urn:adsk.eagle:package:23372/2" value="1000uF"/>
+<part name="C5" library="rcl" library_urn="urn:adsk.eagle:library:334" deviceset="CPOL-US" device="E5-10.5" package3d_urn="urn:adsk.eagle:package:23372/2" value="680uF"/>
+<part name="C6" library="rcl" library_urn="urn:adsk.eagle:library:334" deviceset="CPOL-US" device="E5-10.5" package3d_urn="urn:adsk.eagle:package:23372/2" value="680uF"/>
 <part name="U1" library="LCSC" library_urn="urn:adsk.eagle:library:4712115" deviceset="AT25SF041" device="" package3d_urn="urn:adsk.eagle:package:5772235/2" value="4MB Flash"/>
 <part name="R9" library="rcl" library_urn="urn:adsk.eagle:library:334" deviceset="R-US_" device="R0603" package3d_urn="urn:adsk.eagle:package:23555/3" value="10k"/>
@@
 <part name="JP5" library="pinhead" library_urn="urn:adsk.eagle:library:325" deviceset="PINHD-1X2" device="" package3d_urn="urn:adsk.eagle:package:22435/2"/>
 <part name="R10" library="rcl" library_urn="urn:adsk.eagle:library:334" deviceset="R-US_" device="R0603" package3d_urn="urn:adsk.eagle:package:23555/3" value="120"/>
+<part name="C18" library="rcl" library_urn="urn:adsk.eagle:library:334" deviceset="CPOL-US" device="E5-10.5" package3d_urn="urn:adsk.eagle:package:23372/2" value="680uF"/>
 </parts>
 <sheets>
@@
 <attribute name="NAME" x="-49.53" y="80.2386" size="1.778" layer="95"/>
 <attribute name="VALUE" x="-49.53" y="75.438" size="1.778" layer="96"/>
+</instance>
+<instance part="C18" gate="G$1" x="-53.34" y="121.92" smashed="yes">
+<attribute name="NAME" x="-52.324" y="122.555" size="1.778" layer="95"/>
+<attribute name="VALUE" x="-52.324" y="117.729" size="1.778" layer="96"/>
 </instance>
 </instances>
@@
 <wire x1="-38.1" y1="109.22" x2="-38.1" y2="116.84" width="0.1524" layer="91"/>
 <junction x="-22.86" y="109.22"/>
+<pinref part="C18" gate="G$1" pin="-"/>
+<wire x1="-53.34" y1="116.84" x2="-53.34" y2="109.22" width="0.1524" layer="91"/>
+<wire x1="-53.34" y1="109.22" x2="-38.1" y2="109.22" width="0.1524" layer="91"/>
+<junction x="-38.1" y="109.22"/>
 </segment>
 <segment>
@@
 <wire x1="-22.86" y1="124.46" x2="-22.86" y2="132.08" width="0.1524" layer="91"/>
 <junction x="-22.86" y="132.08"/>
-</segment>
-<segment>
+<pinref part="C18" gate="G$1" pin="+"/>
+<wire x1="-53.34" y1="124.46" x2="-53.34" y2="132.08" width="0.1524" layer="91"/>
+<wire x1="-53.34" y1="132.08" x2="-38.1" y2="132.08" width="0.1524" layer="91"/>
+<junction x="-38.1" y="132.08"/>
+</segment>
+<segment>

Commit message: changed layout to fit the CAN Connector
Parts:
- added JP6: (no value), pinhead:PINHD-1X2
Connections:
- net CANH: now also JP6.1
- net CANL: now also JP6.2
Changed lines of the file:
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@@
 <part name="R10" library="rcl" library_urn="urn:adsk.eagle:library:334" deviceset="R-US_" device="R0603" package3d_urn="urn:adsk.eagle:package:23555/3" value="120"/>
 <part name="C18" library="rcl" library_urn="urn:adsk.eagle:library:334" deviceset="CPOL-US" device="E5-10.5" package3d_urn="urn:adsk.eagle:package:23372/2" value="680uF"/>
+<part name="JP6" library="pinhead" library_urn="urn:adsk.eagle:library:325" deviceset="PINHD-1X2" device="" package3d_urn="urn:adsk.eagle:package:22435/2"/>
 </parts>
 <sheets>
@@
 <attribute name="NAME" x="-52.324" y="122.555" size="1.778" layer="95"/>
 <attribute name="VALUE" x="-52.324" y="117.729" size="1.778" layer="96"/>
+</instance>
+<instance part="JP6" gate="G$1" x="-30.48" y="55.88" smashed="yes">
+<attribute name="NAME" x="-36.83" y="61.595" size="1.778" layer="95"/>
+<attribute name="VALUE" x="-36.83" y="50.8" size="1.778" layer="96"/>
 </instance>
 </instances>
@@
 <label x="-60.96" y="78.74" size="1.778" layer="95"/>
 </segment>
+<segment>
+<pinref part="JP6" gate="G$1" pin="1"/>
+<wire x1="-33.02" y1="58.42" x2="-53.34" y2="58.42" width="0.1524" layer="91"/>
+<label x="-48.26" y="58.42" size="1.778" layer="95"/>
+</segment>
 </net>
 <net name="CANL" class="0">
@@
 <label x="-53.34" y="71.12" size="1.778" layer="95"/>
 </segment>
+<segment>
+<pinref part="JP6" gate="G$1" pin="2"/>
+<wire x1="-33.02" y1="55.88" x2="-53.34" y2="55.88" width="0.1524" layer="91"/>
+<label x="-48.26" y="55.88" size="1.778" layer="95"/>
+</segment>
 </net>
