File: battery_monitor/battery_monitor.brd (EAGLE design)
At the start: 160 x 100 mm, 34 parts, among them CON1 SM04B-GHS-TB, CON2 SM04B-GHS-TB, U1 STM32F303CB

Commit message: Schematic is finished (maybe)
Parts:
- removed R10: (no value), resistor:R0805
- removed R9: 40, resistor:R0805
- added C10, C9: 1uF, rcl:C0805
- U$8: value LP2981 -> RICHTEK_RT9058; device SPEAR-battery-monitor:SOT23-5 -> SPEAR-battery-monitor:SOT23
- moved U$1 22.9 mm to (-41.9, 2.54)
Connections:
- removed net N$8: R10.2, R9.2, U$8.1, U$8.3
- net +3V3: now also C9.1, U$8.2; no longer U$8.5
- net +VBAT: now also C10.1, U$8.1; no longer R9.1
- net GND: now also C10.2, C9.2, U$8.3; no longer R10.1, U$8.2
Changed lines of the file:
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@@
 </element>
 <element name="STM32-1" library="SPEAR-battery-monitor" package="TE_5-103669-3" value="STM32_SWD-HDR" x="26.67" y="40.64" rot="R90"/>
-<element name="U$1" library="SPEAR-battery-monitor" package="INFINEON_PG-TO263-3-2" value="IPB120P04P4L03ATMA1" x="-19.05" y="2.54"/>
+<element name="U$1" library="SPEAR-battery-monitor" package="INFINEON_PG-TO263-3-2" value="IPB120P04P4L03ATMA1" x="-41.91" y="2.54"/>
 <element name="U$2" library="SPEAR-battery-monitor" package="INFINEON_PG-TO263-3-2" value="IPB120P04P4L03ATMA1" x="-30.48" y="2.54"/>
 <element name="U$3" library="SPEAR-battery-monitor" package="SOT23" value="T2N7002AK,LM" x="-64.77" y="53.34"/>
@@
 <element name="U$7" library="SPEAR-general" package="SOIC8" value="MCP2562-E/SN" x="-58.42" y="24.13"/>
 <element name="U1" library="SPEAR-general" package="LQFP48" value="STM32F303CB" x="-49.53" y="41.91"/>
-<element name="U$8" library="SPEAR-battery-monitor" package="SOT23-5" value="LP2981" x="-64.77" y="-3.81"/>
-<element name="R9" library="resistor" library_urn="urn:adsk.eagle:library:348" package="R0805" package3d_urn="urn:adsk.eagle:package:23553/2" value="40" x="-64.77" y="-11.43"/>
-<element name="R10" library="resistor" library_urn="urn:adsk.eagle:library:348" package="R0805" package3d_urn="urn:adsk.eagle:package:23553/2" value="" x="-64.77" y="-16.51"/>
+<element name="U$8" library="SPEAR-battery-monitor" package="SOT23" value="RICHTEK_RT9058" x="-64.77" y="-3.81"/>
+<element name="C9" library="rcl" library_urn="urn:adsk.eagle:library:334" package="C0805" package3d_urn="urn:adsk.eagle:package:23617/2" value="1uF" x="-64.77" y="-11.43">
+<attribute name="SPICEPREFIX" value="C" x="-64.77" y="-11.43" size="1.778" layer="27" display="off"/>
+</element>
+<element name="C10" library="rcl" library_urn="urn:adsk.eagle:library:334" package="C0805" package3d_urn="urn:adsk.eagle:package:23617/2" value="1uF" x="-64.77" y="-16.51">
+<attribute name="SPICEPREFIX" value="C" x="-64.77" y="-16.51" size="1.778" layer="27" display="off"/>
+</element>
 </elements>
 <signals>
@@
 <wire x1="-64.77" y1="54.44" x2="-37.78" y2="68.58" width="0" layer="19" extent="1-1"/>
 <wire x1="-33.02" y1="2.54" x2="-64.77" y2="54.44" width="0" layer="19" extent="1-1"/>
-<wire x1="-21.59" y1="2.54" x2="-33.02" y2="2.54" width="0" layer="19" extent="1-1"/>
+<wire x1="-44.45" y1="2.54" x2="-33.02" y2="2.54" width="0" layer="19" extent="1-1"/>
 </signal>
 <signal name="+VBAT">
@@
 <contactref element="R1" pad="2"/>
 <contactref element="PCON1" pad="+"/>
-<contactref element="R9" pad="1"/>
+<contactref element="U$8" pad="1"/>
+<contactref element="C10" pad="1"/>
 <wire x1="-35.88" y1="68.58" x2="55.88" y2="90.17" width="0" layer="19" extent="1-1"/>
 <wire x1="-27.94" y1="2.54" x2="-35.88" y2="68.58" width="0" layer="19" extent="1-1"/>
-<wire x1="-16.51" y1="2.54" x2="-27.94" y2="2.54" width="0" layer="19" extent="1-1"/>
-<wire x1="-65.72" y1="-11.43" x2="-27.94" y2="2.54" width="0" layer="19" extent="1-1"/>
+<wire x1="-39.37" y1="2.54" x2="-27.94" y2="2.54" width="0" layer="19" extent="1-1"/>
+<wire x1="-65.72" y1="-4.91" x2="-27.94" y2="2.54" width="0" layer="19" extent="1-1"/>
+<wire x1="-65.72" y1="-16.51" x2="-65.72" y2="-4.91" width="0" layer="19" extent="1-1"/>
 </signal>
 <signal name="GND">
@@
 <contactref element="LED1" pad="C"/>
 <contactref element="LED2" pad="C"/>
-<contactref element="R10" pad="1"/>
-<contactref element="U$8" pad="2"/>
+<contactref element="U$8" pad="3"/>
+<contactref element="C10" pad="2"/>
+<contactref element="C9" pad="2"/>
 <wire x1="26.67" y1="40.64" x2="74.93" y2="90.17" width="0" layer="19" extent="1-1"/>
 <wire x1="-15.56" y1="68.58" x2="26.67" y2="40.64" width="0" layer="19" extent="1-1"/>
@@
 <wire x1="-59.055" y1="21.38" x2="-49.784" y2="24.003" width="0" layer="19" extent="1-1"/>
 <wire x1="-60.325" y1="26.88" x2="-59.055" y2="21.38" width="0" layer="19" extent="1-1"/>
-<wire x1="-64.77" y1="-5.01" x2="-59.055" y2="21.38" width="0" layer="19" extent="1-1"/>
-<wire x1="-65.72" y1="-16.51" x2="-64.77" y2="-5.01" width="0" layer="19" extent="1-1"/>
+<wire x1="-64.77" y1="-2.71" x2="-59.055" y2="21.38" width="0" layer="19" extent="1-1"/>
+<wire x1="-63.82" y1="-11.43" x2="-64.77" y2="-2.71" width="0" layer="19" extent="1-1"/>
+<wire x1="-63.82" y1="-16.51" x2="-63.82" y2="-11.43" width="0" layer="19" extent="1-1"/>
 </signal>
 <signal name="OUT_EN">
@@
 <contactref element="U$4" pad="P$1"/>
 <wire x1="-30.48" y1="11.69" x2="68.58" y2="46.44" width="0" layer="19" extent="1-1"/>
-<wire x1="-19.05" y1="11.69" x2="-30.48" y2="11.69" width="0" layer="19" extent="1-1"/>
+<wire x1="-41.91" y1="11.69" x2="-30.48" y2="11.69" width="0" layer="19" extent="1-1"/>
 </signal>
 <signal name="N$2">
@@
 <contactref element="STM32-1" pad="P$4"/>
 <contactref element="R7" pad="2"/>
-<contactref element="U$8" pad="5"/>
+<contactref element="U$8" pad="2"/>
+<contactref element="C9" pad="1"/>
 <wire x1="-23.18" y1="62.23" x2="26.67" y2="48.26" width="0" layer="19" extent="1-1"/>
 <wire x1="-22.54" y1="68.58" x2="-23.18" y2="62.23" width="0" layer="19" extent="1-1"/>
@@
 <wire x1="-56.515" y1="26.88" x2="-52.28" y2="37.66" width="0" layer="19" extent="1-1"/>
 <wire x1="-63.82" y1="62.23" x2="-50.48" y2="62.23" width="0" layer="19" extent="1-1"/>
-<wire x1="-65.72" y1="-2.61" x2="-56.515" y2="26.88" width="0" layer="19" extent="1-1"/>
+<wire x1="-63.82" y1="-4.91" x2="-56.515" y2="26.88" width="0" layer="19" extent="1-1"/>
+<wire x1="-65.72" y1="-11.43" x2="-63.82" y2="-4.91" width="0" layer="19" extent="1-1"/>
 </signal>
 <signal name="N$3">
@@
 <wire x1="-47.94" y1="68.58" x2="-19.05" y2="72.61" width="0" layer="19" extent="1-1"/>
 </signal>
-<signal name="N$8">
-<contactref element="U$8" pad="1"/>
-<contactref element="R10" pad="2"/>
-<contactref element="R9" pad="2"/>
-<contactref element="U$8" pad="3"/>
-<wire x1="-63.82" y1="-11.43" x2="-63.82" y2="-16.51" width="0" layer="19" extent="1-1"/>
-<wire x1="-63.82" y1="-5.01" x2="-63.82" y2="-11.43" width="0" layer="19" extent="1-1"/>
-<wire x1="-65.72" y1="-5.01" x2="-63.82" y2="-5.01" width="0" layer="19" extent="1-1"/>
-</signal>
 </signals>

Commit message: Mostly finished layout.
Parts:
- added J1: 2PIN_HDR, SPEAR-battery-monitor:2PIN-HDR
- moved U$2 124.0 mm to (71.1, 73.7), turned to 180 degrees
- moved C10 124.0 mm to (33.0, 59.7), turned to 270 degrees
- moved U$1 123.0 mm to (58.4, 73.7), turned to 180 degrees
- moved C9 114.8 mm to (25.4, 59.7), turned to 270 degrees
- moved U$8 113.4 mm to (29.2, 59.7), turned to 180 degrees
- moved U$5 108.4 mm to (64.8, 8.89), turned to 270 degrees
- moved U$3 94.8 mm to (29.2, 66.0)
- moved R3 89.3 mm to (26.7, 39.4)
- moved C4 84.6 mm to (34.3, 50.8), turned to 90 degrees
- moved C3 83.3 mm to (39.4, 50.8), turned to 90 degrees
- moved R6 81.0 mm to (15.4, 50.3), turned to 180 degrees
- moved R2 80.1 mm to (25.4, 66.0), turned to 90 degrees
- moved U$6 79.8 mm to (29.2, 34.3), turned to 90 degrees
- moved C2 78.0 mm to (39.4, 45.7), turned to 270 degrees
- moved U1 76.5 mm to (26.7, 48.3)
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Connections:
- removed net +VOUT: U$1.P$2, U$2.P$2, U$4.P$1
- removed net ISENSE_B: U$4.P$4, U$6.3
- removed net N$2: U$4.P$2, U$5.+_1, U$5.+_2
- new net MCU_OUT_EN: J1.P$1, U1.38
- new net VOUT: U$4.P$2, U$4.P$4, U$5.+_1, U$5.+_2, U$6.3
- net ISENSE_A: now also U$1.P$2, U$2.P$2, U$4.P$1
- net ISENSE_OUT: now also U1.10
- net OUT_EN: now also J1.P$2
Routing:
- net +3V3: track 0.00 -> 120.3 mm, vias 0 -> 1
- net N$1: track 0.00 -> 54.6 mm, vias 0 -> 2
- net +VBAT: track 0.00 -> 39.0 mm
- net +5V: track 0.00 -> 36.6 mm
- net CANTX: track 0.00 -> 27.7 mm, vias 0 -> 2
- net OUT_EN: track 0.00 -> 26.5 mm
- net MCU_OUT_EN: track 0.00 -> 24.8 mm
- net CANRX: track 0.00 -> 21.6 mm
- net N$5: track 0.00 -> 21.6 mm, vias 0 -> 2
- net NRST: track 0.00 -> 20.2 mm, vias 0 -> 2
- net ISENSE_OUT: track 0.00 -> 20.1 mm
- net ISENSE_A: track 0.00 -> 20.0 mm
- net VOUT: track 0.00 -> 20.0 mm, vias 0 -> 2
- net N$6: track 0.00 -> 18.6 mm, vias 0 -> 2
- net CANL: track 0.00 -> 17.4 mm, vias 0 -> 2
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- added copper zone on layer 1, net +VBAT
- added copper zone on layer 16, net GND
- added copper zone on layer 1, net ISENSE_A
- added copper zone on layer 1, net VOUT
Other:
- board size 160 x 100 mm -> 91.7 x 100.1 mm

Commit message: Finished layout.
Parts:
- added S2: (no value), SPEAR-arm-control:TACTILE_SWITCH_SMD_4.6X2.8MM
Connections:
- new net USR_BTN: S2.1, S2.2, U1.11
- net GND: now also S2.3, S2.4
Routing:
- net GND: track 0.00 -> 96.1 mm, vias 0 -> 20
- net +3V3: track 120.3 -> 145.1 mm, vias 1 -> 3
- net USR_BTN: track 0.00 -> 14.0 mm, vias 0 -> 2
- net CANTX: track 27.7 -> 28.4 mm
- net N$5: track 21.6 -> 22.2 mm

Commit message: Improved Silkscreen and finished dimensioning.
Parts:
- moved C10 20.3 mm to (33.0, 80.0)
- moved C2 20.3 mm to (39.4, 66.0)
- moved C3 20.3 mm to (39.4, 71.1)
- moved C4 20.3 mm to (34.3, 71.1)
- moved C5 20.3 mm to (36.8, 71.1)
- moved C6 20.3 mm to (34.3, 66.0)
- moved C7 20.3 mm to (36.8, 66.0)
- moved C9 20.3 mm to (25.4, 80.0)
- moved U$1 20.3 mm to (58.4, 94.0)
- moved U$2 20.3 mm to (71.1, 94.0)
- moved U$8 20.3 mm to (29.2, 80.0)
- moved C1 20.3 mm to (31.4, 59.7)
- moved C8 20.3 mm to (16.4, 56.4)
- moved CON2 20.3 mm to (7.62, 61.0)
- moved LED1 20.3 mm to (16.5, 77.5)
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Routing:
- net +3V3: track 145.1 -> 141.9 mm
Other:
- board size 91.7 x 100.1 mm -> 89.7 x 109.4 mm
- board text added: "Battery Monitor Board Rev. A"
- board text added: "David Lenfesty"
- board text added: "OUT_EN"
- board text added: "PWR"
- board text added: "Reset"
- board text added: "SPEAR"
- board text added: "Toggle Output"
