File: battery_monitor/battery_monitor.brd (EAGLE design)
At the start: 89.7 x 109.4 mm, 36 parts, among them CON1 SM04B-GHS-TB, CON2 SM04B-GHS-TB, J1 2PIN_HDR, U1 STM32F303CB

Commit message: Updated battery monitor design.
- Added cortex debug header.
- Added voltage divider to read voltage from batteries.
- Added 8MHz crystal oscillator
Parts:
- removed STM32-1: STM32_SWD-HDR, SPEAR-battery-monitor:TE_5-103669-3
- added C11, C12: 22pF, resistor:C0805
- added JP1: CORTEX-M-DBG, SPEAR-general:FTSH-105-01-F-DV-007
- added R10: 10K, resistor:R0805
- added R9: 90K, resistor:R0805
- added Y1: NX5032, SPEAR-general:NX5032
Connections:
- removed net N$5: STM32-1.P$3, U1.34
- removed net N$6: STM32-1.P$2, U1.37
- new net OSC_IN: C11.1, U1.5, Y1.P$2
- new net OSC_OUT: C12.1, U1.6, Y1.P$1
- new net SWCLK: JP1.4, U1.37
- new net SWDIO: JP1.2, U1.34
- new net SWO: JP1.6, U1.39
- new net VBAT_MEASURE: R10.1, R9.2, U1.12
- net +3V3: now also JP1.1; no longer STM32-1.P$4
- net +VBAT: now also R9.1
- net GND: now also C11.2, C12.2, JP1.3, JP1.5, JP1.9, R10.2; no longer STM32-1.P$1
- net NRST: now also JP1.10
Routing:
- net OSC_IN: track 0.00 -> 37.7 mm, vias 0 -> 2
- net OSC_OUT: track 0.00 -> 37.5 mm, vias 0 -> 2
- net VBAT_MEASURE: track 0.00 -> 24.8 mm, vias 0 -> 2
- net N$5: track 22.2 -> 0.00 mm, vias 2 -> 0
- net SWDIO: track 0.00 -> 21.4 mm, vias 0 -> 2
- net N$6: track 18.6 -> 0.00 mm, vias 2 -> 0
- net SWCLK: track 0.00 -> 16.0 mm, vias 0 -> 2
- net SWO: track 0.00 -> 15.9 mm
- net GND: track 96.1 -> 106.2 mm, vias 20 -> 23
- net NRST: track 20.2 -> 26.9 mm
- net +3V3: track 141.9 -> 145.8 mm, vias 3 -> 6
- net +VBAT: track 39.0 -> 42.7 mm
Other:
- board size 89.7 x 109.4 mm -> 90 x 110 mm
- board text added: "Battery Monitor Board Rev. B"
- board text removed: "Battery Monitor Board Rev. A"
