File: battery_monitor/battery_monitor.sch (EAGLE design)
At the start: 5 parts

Commit message: Added current sense.
Parts:
- added U$4: 20U_PC_SHUNT, SPEAR-battery-monitor:20U_PC_SHUNT
- added U$5: PP45_HOR_4GRD, SPEAR-general:PP45_HOR_4GRD
Connections:
- new net ISENSE_A: U$4.SA
- new net ISENSE_B: U$4.SB
- new net N$2: U$4.B, U$5.+
- net +VOUT: now also U$4.A
- net GND: now also U$5.-
Other:
- note added: "Current Sense Diff. Amplifier"
- note removed: "Rsens goes here."
Changed lines of the file:
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@@
 <part name="GND1" library="supply1" library_urn="urn:adsk.eagle:library:371" deviceset="GND" device=""/>
 <part name="R2" library="resistor" library_urn="urn:adsk.eagle:library:348" deviceset="R-EU_" device="R0805" package3d_urn="urn:adsk.eagle:package:23553/2" value="10K"/>
+<part name="U$4" library="SPEAR-battery-monitor" deviceset="20U_PC_SHUNT" device=""/>
+<part name="U$5" library="SPEAR-general" deviceset="PP45_HOR_4GRD" device=""/>
+<part name="GND2" library="supply1" library_urn="urn:adsk.eagle:library:371" deviceset="GND" device=""/>
 </parts>
 <sheets>
 <sheet>
 <plain>
-<wire x1="0" y1="58.42" x2="0" y2="-35.56" width="0.1524" layer="94" style="shortdash"/>
-<wire x1="0" y1="-35.56" x2="129.54" y2="-35.56" width="0.1524" layer="94" style="shortdash"/>
-<wire x1="129.54" y1="-35.56" x2="127" y2="-35.56" width="0.1524" layer="94" style="shortdash"/>
-<wire x1="127" y1="-35.56" x2="127" y2="58.42" width="0.1524" layer="94" style="shortdash"/>
-<wire x1="127" y1="58.42" x2="127" y2="63.5" width="0.1524" layer="94" style="shortdash"/>
-<wire x1="127" y1="63.5" x2="0" y2="63.5" width="0.1524" layer="94" style="shortdash"/>
-<wire x1="0" y1="63.5" x2="0" y2="58.42" width="0.1524" layer="94" style="shortdash"/>
+<wire x1="0" y1="-35.56" x2="124.46" y2="-35.56" width="0.1524" layer="94" style="shortdash"/>
+<wire x1="124.46" y1="-35.56" x2="121.92" y2="-35.56" width="0.1524" layer="94" style="shortdash"/>
+<wire x1="124.46" y1="58.42" x2="124.46" y2="63.5" width="0.1524" layer="94" style="shortdash"/>
 <text x="0" y="63.5" size="1.778" layer="94">MOSFET Control</text>
-<text x="86.36" y="-15.24" size="1.778" layer="94">Rsens goes here.</text>
+<wire x1="124.46" y1="58.42" x2="124.46" y2="-35.56" width="0.1524" layer="94" style="shortdash"/>
+<wire x1="0" y1="-35.56" x2="0" y2="63.5" width="0.1524" layer="94" style="shortdash"/>
+<wire x1="0" y1="63.5" x2="124.46" y2="63.5" width="0.1524" layer="94" style="shortdash"/>
+<text x="149.86" y="38.1" size="1.778" layer="94">Current Sense Diff. Amplifier</text>
 </plain>
 <instances>
@@
 <instance part="GND1" gate="1" x="50.8" y="-30.48"/>
 <instance part="R2" gate="G$1" x="27.94" y="-20.32" rot="R90"/>
+<instance part="U$4" gate="G$1" x="93.98" y="-10.16" rot="R90"/>
+<instance part="U$5" gate="G$1" x="104.14" y="-45.72"/>
+<instance part="GND2" gate="1" x="93.98" y="-58.42"/>
 </instances>
 <busses>
@@
 <junction x="50.8" y="-25.4"/>
 </segment>
+<segment>
+<pinref part="U$5" gate="G$1" pin="-"/>
+<wire x1="99.06" y1="-50.8" x2="93.98" y2="-50.8" width="0.1524" layer="91"/>
+<wire x1="93.98" y1="-50.8" x2="93.98" y2="-55.88" width="0.1524" layer="91"/>
+<pinref part="GND2" gate="1" pin="GND"/>
+</segment>
 </net>
 <net name="OUT_EN" class="0">
@@
 <junction x="81.28" y="5.08"/>
 <wire x1="93.98" y1="5.08" x2="93.98" y2="-2.54" width="0.1524" layer="91"/>
+<pinref part="U$4" gate="G$1" pin="A"/>
+<wire x1="93.98" y1="-2.54" x2="93.98" y2="-5.08" width="0.1524" layer="91"/>
 </segment>
 </net>
@@
 <segment>
 <wire x1="93.98" y1="-20.32" x2="93.98" y2="-25.4" width="0.1524" layer="91"/>
+<pinref part="U$4" gate="G$1" pin="B"/>
+<wire x1="93.98" y1="-17.78" x2="93.98" y2="-20.32" width="0.1524" layer="91"/>
+<wire x1="93.98" y1="-25.4" x2="93.98" y2="-40.64" width="0.1524" layer="91"/>
+<wire x1="93.98" y1="-40.64" x2="99.06" y2="-40.64" width="0.1524" layer="91"/>
+<pinref part="U$5" gate="G$1" pin="+"/>
 </segment>
 </net>
+<net name="ISENSE_A" class="0">
+<segment>
+<pinref part="U$4" gate="G$1" pin="SA"/>
+<wire x1="96.52" y1="-5.08" x2="109.22" y2="-5.08" width="0.1524" layer="91"/>
+<label x="109.22" y="-5.08" size="1.778" layer="95"/>
+</segment>
+</net>
+<net name="ISENSE_B" class="0">
+<segment>
+<pinref part="U$4" gate="G$1" pin="SB"/>
+<wire x1="96.52" y1="-17.78" x2="109.22" y2="-17.78" width="0.1524" layer="91"/>
+<label x="109.22" y="-17.78" size="1.778" layer="95"/>
+</segment>
+</net>

Commit message: Finished design block
Parts:
- added C1: 0u1F, resistor:C-EUC0805
- added C2, C3, C4: 100n, resistor:C-EUC0805
- added C5: 4u7, resistor:C-EUC0805
- added C6: 1uF, resistor:C-EUC0805
- added C7: 10nF, resistor:C-EUC0805
- added C8: 0u1, resistor:C-EUC0805
- added CON1, CON2: SM04B-GHS-TB, SPEAR-general:SM04B-GHS-TB
- added LED1, LED2: (no value), led:LEDCHIPLED_0805
- added PCON1: WIREPAD_DUAL-10AWG, SPEAR-battery-monitor:WIREPAD_DUAL-10AWG
- added R10: (no value), resistor:R-EU_R0805
- added R3, R6: 10K, resistor:R-EU_R0805
- added R4: 100, resistor:R-EU_R0805
- added R5: 100K, resistor:R-EU_R0805
- added R7, R8: 1K, resistor:R-EU_R0805
- added R9: 40, resistor:R-EU_R0805
- added S1: (no value), SPEAR-arm-control:MOMENTARY-SWITCH-SPST-2-SMD-4.6X2.8MM
- added STM32-1: STM32_SWD-HDR, SPEAR-battery-monitor:STM32_SWD-HDR
- added U$6: INA145, SPEAR-battery-monitor:INA145
- added U$7: MCP2562-E/SN, SPEAR-general:MCP2562-E/SN
- added U$8: LP2981, SPEAR-battery-monitor:LP2981
- added U1: STM32F303CB, SPEAR-general:STM32F303CB
Connections:
- new net +3V3: C1.2, C2.1, C3.1, C4.1, C5.1, C6.1, C7.1, R6.2, R7.2, STM32-1+3V3.S, U$6.V+, U$7.VIO, U$8.VOUT, U1-MISC.VBAT, U1-PWR.VDDA, U1-PWR.VDD_1, U1-PWR.VDD_2, U1-PWR.VDD_3
- new net +5V: C8.1, CON1-1.S, CON2-1.S, U$7.VDD
- new net CANH: CON1-2.S, CON2-2.S, U$7.CANH
- new net CANL: CON1-3.S, CON2-3.S, U$7.CANL
- new net CANRX: U$7.RXD, U1-PORTA.PA11
- new net CANTX: U$7.TXD, U1-PORTA.PA12
- new net ISENSE_OUT: R5.1, U$6.OUT
- new net N$3: R3.1, U$6.VG
- new net N$4: R3.2, R4.1, R5.2
- new net N$5: STM32-1SWDIO.S, U1-PORTA.PA13
- new net N$6: STM32-1SWCLK.S, U1-PORTA.PA14
- new net N$7: LED1.A, R7.1
- new net N$8: R10.2, R9.2, U$8.EN, U$8.VIN
- new net N$9: LED2.A, R8.1
- new net NRST: R6.1, S1.3, S1.4, U1-MISC.NRST
- net +VBAT: now also PCON1-VBAT.P, R9.1
- net GND: now also C1.1, C2.2, C3.2, C4.2, C5.2, C6.2, C7.2, C8.2, CON1-4.S, CON1-TABS.S, CON2-4.S, CON2-TABS.S, LED1.C, LED2.C, PCON1-GND.P, R10.1, R4.2, S1.1, S1.2, STM32-1GND.S, U$6.REF, U$6.V-, U$7.STBY, U$7.VSS, U$8.GND, U1-MISC.BOOT0, U1-PWR.VSSA/VREF-, U1-PWR.VSS_1, U1-PWR.VSS_2, U1-PWR.VSS_3
- net ISENSE_A: now also U$6.IN-
- net ISENSE_B: now also U$6.IN+
- net OUT_EN: now also R8.2
Other:
- note added: "1% Tolerance Resistors"
- note added: "Analog Supply Decoupling"
- note added: "CAN Bus"
- note added: "Datasheet Recommended"
- note added: "Digital Supply Decoupling"
- note added: "Indication"
- note added: "MCU Power"
- note added: "NOTE: No isolation protection on 3v3 rail. Only plug in programming header when unplugged."
- note added: "Output Enable"
- note added: "Power"
- note added: "Power Input"
- note added: "Voltage Regulation"
- moved on the sheet: R1, R2, U$1, U$2, U$3, U$4

Commit message: Schematic is finished (maybe)
Parts:
- removed R10: (no value), resistor:R-EU_R0805
- removed R9: 40, resistor:R-EU_R0805
- added C10, C9: 1uF, rcl:C-EUC0805
- U$8: value LP2981 -> RICHTEK_RT9058; device SPEAR-battery-monitor:LP2981 -> SPEAR-battery-monitor:RICHTEK_RT9058
Connections:
- removed net N$8: R10.2, R9.2, U$8.EN, U$8.VIN
- net +3V3: now also C9.1
- net +VBAT: now also C10.1, U$8.VIN; no longer R9.1
- net GND: now also C10.2, C9.2; no longer R10.1
Other:
- note added: "Power Regulation"
- note removed: "Voltage Regulation"
Changed lines of the file:
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@@
 <part name="GND16" library="supply1" library_urn="urn:adsk.eagle:library:371" deviceset="GND" device=""/>
 <part name="GND17" library="supply1" library_urn="urn:adsk.eagle:library:371" deviceset="GND" device=""/>
-<part name="U$8" library="SPEAR-battery-monitor" deviceset="LP2981" device=""/>
-<part name="R9" library="resistor" library_urn="urn:adsk.eagle:library:348" deviceset="R-EU_" device="R0805" package3d_urn="urn:adsk.eagle:package:23553/2" value="40"/>
-<part name="R10" library="resistor" library_urn="urn:adsk.eagle:library:348" deviceset="R-EU_" device="R0805" package3d_urn="urn:adsk.eagle:package:23553/2"/>
+<part name="U$8" library="SPEAR-battery-monitor" deviceset="RICHTEK_RT9058" device=""/>
 <part name="GND18" library="supply1" library_urn="urn:adsk.eagle:library:371" deviceset="GND" device=""/>
-<part name="GND19" library="supply1" library_urn="urn:adsk.eagle:library:371" deviceset="GND" device=""/>
 <part name="+3V9" library="supply1" library_urn="urn:adsk.eagle:library:371" deviceset="+3V3" device=""/>
+<part name="C9" library="rcl" library_urn="urn:adsk.eagle:library:334" deviceset="C-EU" device="C0805" package3d_urn="urn:adsk.eagle:package:23617/2" value="1uF"/>
+<part name="C10" library="rcl" library_urn="urn:adsk.eagle:library:334" deviceset="C-EU" device="C0805" package3d_urn="urn:adsk.eagle:package:23617/2" value="1uF"/>
 </parts>
 <sheets>
@@
 <wire x1="223.52" y1="129.54" x2="165.1" y2="129.54" width="0.1524" layer="94" style="shortdash"/>
 <wire x1="165.1" y1="129.54" x2="165.1" y2="175.26" width="0.1524" layer="94" style="shortdash"/>
-<text x="195.58" y="170.18" size="1.778" layer="94">Voltage Regulation</text>
+<text x="200.66" y="170.18" size="1.778" layer="94">Power Regulation</text>
 </plain>
 <instances>
@@
 <instance part="GND16" gate="1" x="261.62" y="129.54"/>
 <instance part="GND17" gate="1" x="281.94" y="129.54"/>
-<instance part="U$8" gate="G$1" x="185.42" y="144.78"/>
-<instance part="R9" gate="G$1" x="170.18" y="162.56" rot="R270"/>
-<instance part="R10" gate="G$1" x="170.18" y="147.32" rot="R90"/>
-<instance part="GND18" gate="1" x="170.18" y="137.16"/>
-<instance part="GND19" gate="1" x="195.58" y="134.62"/>
-<instance part="+3V9" gate="G$1" x="218.44" y="160.02"/>
+<instance part="U$8" gate="G$1" x="185.42" y="147.32"/>
+<instance part="GND18" gate="1" x="193.04" y="134.62"/>
+<instance part="+3V9" gate="G$1" x="215.9" y="162.56"/>
+<instance part="C9" gate="G$1" x="215.9" y="149.86"/>
+<instance part="C10" gate="G$1" x="172.72" y="149.86"/>
 </instances>
 <busses>
@@
 </segment>
 <segment>
-<pinref part="R9" gate="G$1" pin="1"/>
-<wire x1="170.18" y1="167.64" x2="170.18" y2="170.18" width="0.1524" layer="91"/>
-<label x="170.18" y="170.18" size="1.778" layer="95"/>
+<pinref part="U$8" gate="G$1" pin="VIN"/>
+<wire x1="180.34" y1="154.94" x2="172.72" y2="154.94" width="0.1524" layer="91"/>
+<wire x1="172.72" y1="154.94" x2="172.72" y2="165.1" width="0.1524" layer="91"/>
+<label x="172.72" y="165.1" size="1.778" layer="95"/>
+<pinref part="C10" gate="G$1" pin="1"/>
+<wire x1="172.72" y1="154.94" x2="172.72" y2="152.4" width="0.1524" layer="91"/>
+<junction x="172.72" y="154.94"/>
 </segment>
 </net>
@@
 </segment>
 <segment>
-<pinref part="R10" gate="G$1" pin="1"/>
-<wire x1="170.18" y1="142.24" x2="170.18" y2="139.7" width="0.1524" layer="91"/>
+<pinref part="U$8" gate="G$1" pin="GND"/>
 <pinref part="GND18" gate="1" pin="GND"/>
-</segment>
-<segment>
-<pinref part="U$8" gate="G$1" pin="GND"/>
-<pinref part="GND19" gate="1" pin="GND"/>
-<wire x1="195.58" y1="139.7" x2="195.58" y2="137.16" width="0.1524" layer="91"/>
+<wire x1="193.04" y1="142.24" x2="193.04" y2="139.7" width="0.1524" layer="91"/>
+<pinref part="C10" gate="G$1" pin="2"/>
+<wire x1="193.04" y1="139.7" x2="193.04" y2="137.16" width="0.1524" layer="91"/>
+<wire x1="172.72" y1="144.78" x2="172.72" y2="139.7" width="0.1524" layer="91"/>
+<wire x1="172.72" y1="139.7" x2="193.04" y2="139.7" width="0.1524" layer="91"/>
+<junction x="193.04" y="139.7"/>
+<pinref part="C9" gate="G$1" pin="2"/>
+<wire x1="193.04" y1="139.7" x2="215.9" y2="139.7" width="0.1524" layer="91"/>
+<wire x1="215.9" y1="139.7" x2="215.9" y2="144.78" width="0.1524" layer="91"/>
 </segment>
 </net>
@@
 <segment>
 <pinref part="U$8" gate="G$1" pin="VOUT"/>
-<wire x1="210.82" y1="152.4" x2="218.44" y2="152.4" width="0.1524" layer="91"/>
-<wire x1="218.44" y1="152.4" x2="218.44" y2="157.48" width="0.1524" layer="91"/>
+<wire x1="208.28" y1="154.94" x2="215.9" y2="154.94" width="0.1524" layer="91"/>
+<wire x1="215.9" y1="154.94" x2="215.9" y2="160.02" width="0.1524" layer="91"/>
 <pinref part="+3V9" gate="G$1" pin="+3V3"/>
+<pinref part="C9" gate="G$1" pin="1"/>
+<wire x1="215.9" y1="154.94" x2="215.9" y2="152.4" width="0.1524" layer="91"/>
+<junction x="215.9" y="154.94"/>
 </segment>
 </net>
@@
 <pinref part="LED2" gate="G$1" pin="A"/>
 <wire x1="281.94" y1="149.86" x2="281.94" y2="144.78" width="0.1524" layer="91"/>
-</segment>
-</net>
-<net name="N$8" class="0">
-<segment>
-<pinref part="U$8" gate="G$1" pin="VIN"/>
-<pinref part="R10" gate="G$1" pin="2"/>
-<wire x1="170.18" y1="152.4" x2="177.8" y2="152.4" width="0.1524" layer="91"/>
-<pinref part="R9" gate="G$1" pin="2"/>
-<wire x1="177.8" y1="152.4" x2="180.34" y2="152.4" width="0.1524" layer="91"/>
-<wire x1="170.18" y1="157.48" x2="170.18" y2="152.4" width="0.1524" layer="91"/>
-<junction x="170.18" y="152.4"/>
-<wire x1="177.8" y1="152.4" x2="177.8" y2="147.32" width="0.1524" layer="91"/>
-<junction x="177.8" y="152.4"/>
-<pinref part="U$8" gate="G$1" pin="EN"/>
-<wire x1="177.8" y1="147.32" x2="180.34" y2="147.32" width="0.1524" layer="91"/>
 </segment>
 </net>
@@
 packages will not be understood (or retained) with this version.
 </note>
+<note version="8.4" severity="warning">
+Since Version 8.4, EAGLE supports properties for SPICE simulation.
+Probes in schematics and SPICE mapping objects found in parts and library devices
+will not be understood with this version. Update EAGLE to the latest version
+for full support of SPICE simulation.
+</note>
 </compatibility>

Commit message: Mostly finished layout.
Parts:
- added J1: 2PIN_HDR, SPEAR-battery-monitor:2PIN_HDR
Connections:
- removed net +VOUT: U$1.D1, U$2.D1, U$4.A
- removed net ISENSE_B: U$4.SB, U$6.IN+
- removed net N$2: U$4.B, U$5.+
- new net MCU_OUT_EN: J1-1.S, U1-PORTA.PA15
- new net VOUT: U$4.2, U$5.+, U$6.IN+
- net ISENSE_A: now also U$1.D1, U$2.D1, U$4.1; no longer U$4.SA
- net ISENSE_OUT: now also U1-PORTA.PA0
- net OUT_EN: now also J1-2.S
Changed lines of the file:
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@@
 <part name="GND1" library="supply1" library_urn="urn:adsk.eagle:library:371" deviceset="GND" device=""/>
 <part name="R2" library="resistor" library_urn="urn:adsk.eagle:library:348" deviceset="R-EU_" device="R0805" package3d_urn="urn:adsk.eagle:package:23553/2" value="10K"/>
-<part name="U$4" library="SPEAR-battery-monitor" deviceset="20U_PC_SHUNT" device=""/>
 <part name="U$5" library="SPEAR-general" deviceset="PP45_HOR_4GRD" device=""/>
 <part name="GND2" library="supply1" library_urn="urn:adsk.eagle:library:371" deviceset="GND" device=""/>
@@
 <part name="C9" library="rcl" library_urn="urn:adsk.eagle:library:334" deviceset="C-EU" device="C0805" package3d_urn="urn:adsk.eagle:package:23617/2" value="1uF"/>
 <part name="C10" library="rcl" library_urn="urn:adsk.eagle:library:334" deviceset="C-EU" device="C0805" package3d_urn="urn:adsk.eagle:package:23617/2" value="1uF"/>
+<part name="U$4" library="SPEAR-battery-monitor" deviceset="20U_PC_SHUNT" device=""/>
+<part name="J1" library="SPEAR-battery-monitor" deviceset="2PIN_HDR" device=""/>
 </parts>
 <sheets>
@@
 <instance part="GND1" gate="1" x="66.04" y="40.64"/>
 <instance part="R2" gate="G$1" x="43.18" y="50.8" rot="R90"/>
-<instance part="U$4" gate="G$1" x="109.22" y="60.96" rot="R90"/>
 <instance part="U$5" gate="G$1" x="119.38" y="25.4"/>
 <instance part="GND2" gate="1" x="109.22" y="12.7"/>
@@
 <instance part="C9" gate="G$1" x="215.9" y="149.86"/>
 <instance part="C10" gate="G$1" x="172.72" y="149.86"/>
+<instance part="U$4" gate="G$1" x="109.22" y="60.96" rot="R270"/>
+<instance part="J1" gate="-1" x="144.78" y="200.66"/>
+<instance part="J1" gate="-2" x="160.02" y="200.66" rot="R180"/>
 </instances>
 <busses>
@@
 <label x="276.86" y="165.1" size="1.778" layer="95"/>
 </segment>
-</net>
-<net name="+VOUT" class="0">
-<segment>
-<pinref part="U$1" gate="G$1" pin="D1"/>
-<wire x1="50.8" y1="86.36" x2="50.8" y2="76.2" width="0.1524" layer="91"/>
-<wire x1="50.8" y1="76.2" x2="96.52" y2="76.2" width="0.1524" layer="91"/>
-<pinref part="U$2" gate="G$1" pin="D1"/>
-<wire x1="96.52" y1="76.2" x2="96.52" y2="86.36" width="0.1524" layer="91"/>
-<wire x1="96.52" y1="76.2" x2="109.22" y2="76.2" width="0.1524" layer="91"/>
-<junction x="96.52" y="76.2"/>
-<wire x1="109.22" y1="76.2" x2="109.22" y2="68.58" width="0.1524" layer="91"/>
-<pinref part="U$4" gate="G$1" pin="A"/>
-<wire x1="109.22" y1="68.58" x2="109.22" y2="66.04" width="0.1524" layer="91"/>
-</segment>
-</net>
-<net name="N$2" class="0">
-<segment>
-<wire x1="109.22" y1="50.8" x2="109.22" y2="45.72" width="0.1524" layer="91"/>
-<pinref part="U$4" gate="G$1" pin="B"/>
-<wire x1="109.22" y1="53.34" x2="109.22" y2="50.8" width="0.1524" layer="91"/>
-<wire x1="109.22" y1="45.72" x2="109.22" y2="30.48" width="0.1524" layer="91"/>
+<segment>
+<pinref part="J1" gate="-2" pin="S"/>
+<wire x1="162.56" y1="200.66" x2="167.64" y2="200.66" width="0.1524" layer="91"/>
+<label x="167.64" y="200.66" size="1.778" layer="95"/>
+</segment>
+</net>
+<net name="VOUT" class="0">
+<segment>
+<pinref part="U$6" gate="G$1" pin="IN+"/>
+<pinref part="U$4" gate="G$1" pin="2"/>
+<wire x1="165.1" y1="55.88" x2="109.22" y2="55.88" width="0.1524" layer="91"/>
+<junction x="109.22" y="55.88"/>
+<label x="109.22" y="43.18" size="1.778" layer="95"/>
+<wire x1="109.22" y1="55.88" x2="109.22" y2="30.48" width="0.1524" layer="91"/>
+<pinref part="U$5" gate="G$1" pin="+"/>
 <wire x1="109.22" y1="30.48" x2="114.3" y2="30.48" width="0.1524" layer="91"/>
-<pinref part="U$5" gate="G$1" pin="+"/>
-</segment>
-</net>
-<net name="ISENSE_A" class="0">
-<segment>
-<pinref part="U$4" gate="G$1" pin="SA"/>
-<wire x1="111.76" y1="66.04" x2="124.46" y2="66.04" width="0.1524" layer="91"/>
-<label x="124.46" y="66.04" size="1.778" layer="95"/>
-<wire x1="124.46" y1="66.04" x2="147.32" y2="66.04" width="0.1524" layer="91"/>
-<pinref part="U$6" gate="G$1" pin="IN-"/>
-<wire x1="165.1" y1="66.04" x2="160.02" y2="66.04" width="0.1524" layer="91"/>
-<wire x1="147.32" y1="66.04" x2="160.02" y2="66.04" width="0.1524" layer="91"/>
-</segment>
-</net>
-<net name="ISENSE_B" class="0">
-<segment>
-<pinref part="U$4" gate="G$1" pin="SB"/>
-<wire x1="111.76" y1="53.34" x2="124.46" y2="53.34" width="0.1524" layer="91"/>
-<label x="124.46" y="53.34" size="1.778" layer="95"/>
-<wire x1="154.94" y1="53.34" x2="124.46" y2="53.34" width="0.1524" layer="91"/>
-<pinref part="U$6" gate="G$1" pin="IN+"/>
-<wire x1="165.1" y1="55.88" x2="154.94" y2="55.88" width="0.1524" layer="91"/>
-<wire x1="154.94" y1="55.88" x2="154.94" y2="53.34" width="0.1524" layer="91"/>
 </segment>
 </net>
@@
 <label x="205.74" y="60.96" size="1.778" layer="95"/>
 </segment>
+<segment>
+<pinref part="U1" gate="-PORTA" pin="PA0"/>
+<wire x1="119.38" y1="238.76" x2="127" y2="238.76" width="0.1524" layer="91"/>
+<label x="127" y="238.76" size="1.778" layer="95"/>
+</segment>
 </net>
 <net name="NRST" class="0">
@@
 </segment>
 </net>
+<net name="ISENSE_A" class="0">
+<segment>
+<pinref part="U$1" gate="G$1" pin="D1"/>
+<wire x1="50.8" y1="86.36" x2="50.8" y2="76.2" width="0.1524" layer="91"/>
+<wire x1="50.8" y1="76.2" x2="96.52" y2="76.2" width="0.1524" layer="91"/>
+<pinref part="U$2" gate="G$1" pin="D1"/>
+<wire x1="96.52" y1="76.2" x2="96.52" y2="86.36" width="0.1524" layer="91"/>
+<wire x1="96.52" y1="76.2" x2="109.22" y2="76.2" width="0.1524" layer="91"/>
+<junction x="96.52" y="76.2"/>
+<wire x1="109.22" y1="76.2" x2="109.22" y2="66.04" width="0.1524" layer="91"/>
+<wire x1="109.22" y1="66.04" x2="165.1" y2="66.04" width="0.1524" layer="91"/>
+<pinref part="U$6" gate="G$1" pin="IN-"/>
+<pinref part="U$4" gate="G$1" pin="1"/>
+<junction x="109.22" y="66.04"/>
+</segment>
+</net>
+<net name="MCU_OUT_EN" class="0">
+<segment>
+<pinref part="U1" gate="-PORTA" pin="PA15"/>
+<wire x1="119.38" y1="200.66" x2="124.46" y2="200.66" width="0.1524" layer="91"/>
+<label x="124.46" y="200.66" size="1.778" layer="95"/>
+<pinref part="J1" gate="-1" pin="S"/>
+<wire x1="124.46" y1="200.66" x2="142.24" y2="200.66" width="0.1524" layer="91"/>
+</segment>
+</net>

Commit message: Finished layout.
Parts:
- added S2: (no value), SPEAR-arm-control:MOMENTARY-SWITCH-SPST-2-SMD-4.6X2.8MM
Connections:
- new net USR_BTN: S2.1, S2.2, U1-PORTA.PA1
- net GND: now also S2.3, S2.4
Changed lines of the file:
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@@
 <part name="U$4" library="SPEAR-battery-monitor" deviceset="20U_PC_SHUNT" device=""/>
 <part name="J1" library="SPEAR-battery-monitor" deviceset="2PIN_HDR" device=""/>
+<part name="S2" library="SPEAR-arm-control" deviceset="MOMENTARY-SWITCH-SPST-2" device="-SMD-4.6X2.8MM" package3d_urn="urn:adsk.eagle:package:5592177/1"/>
+<part name="GND19" library="supply1" library_urn="urn:adsk.eagle:library:371" deviceset="GND" device=""/>
 </parts>
 <sheets>
@@
 <instance part="J1" gate="-1" x="144.78" y="200.66"/>
 <instance part="J1" gate="-2" x="160.02" y="200.66" rot="R180"/>
+<instance part="S2" gate="G$1" x="175.26" y="233.68"/>
+<instance part="GND19" gate="1" x="180.34" y="220.98"/>
 </instances>
 <busses>
@@
 <wire x1="215.9" y1="139.7" x2="215.9" y2="144.78" width="0.1524" layer="91"/>
 </segment>
+<segment>
+<pinref part="S2" gate="G$1" pin="3"/>
+<pinref part="S2" gate="G$1" pin="4"/>
+<wire x1="180.34" y1="233.68" x2="180.34" y2="231.14" width="0.1524" layer="91"/>
+<wire x1="180.34" y1="231.14" x2="180.34" y2="223.52" width="0.1524" layer="91"/>
+<junction x="180.34" y="231.14"/>
+<pinref part="GND19" gate="1" pin="GND"/>
+</segment>
 </net>
 <net name="OUT_EN" class="0">
@@
 </segment>
 </net>
+<net name="USR_BTN" class="0">
+<segment>
+<pinref part="S2" gate="G$1" pin="2"/>
+<pinref part="S2" gate="G$1" pin="1"/>
+<wire x1="170.18" y1="231.14" x2="170.18" y2="233.68" width="0.1524" layer="91"/>
+<wire x1="170.18" y1="233.68" x2="132.08" y2="233.68" width="0.1524" layer="91"/>
+<wire x1="132.08" y1="233.68" x2="132.08" y2="236.22" width="0.1524" layer="91"/>
+<junction x="170.18" y="233.68"/>
+<pinref part="U1" gate="-PORTA" pin="PA1"/>
+<wire x1="132.08" y1="236.22" x2="119.38" y2="236.22" width="0.1524" layer="91"/>
+<label x="144.78" y="233.68" size="1.778" layer="95"/>
+</segment>
+</net>
