File: drive_pdu/drive_pdu.sch (EAGLE design)
At the start: 0 parts

Commit message: Created Drive PDU
Parts:
- added SV1, SV2: (no value), con-lstb:MA04-1
- added U$1, U$2, U$3, U$4, U$5: PP45-DG, SPEAR:PP45-DG
Connections:
- new net +5V: SV1.1, SV1.3, SV2.1, SV2.3, U$1.+, U$2.+, U$3.+, U$4.+, U$5.+
- new net GND: SV1.2, SV1.4, SV2.2, SV2.4, U$1.-, U$2.-, U$3.-, U$4.-, U$5.-
