File: drive_pdu/DrivePDU.brd (EAGLE design)
At the start: 105.1 x 100.3 mm, 17 parts

Commit message: Added dimensioning and tweaked dimensions slightly.
Parts:
- moved U$8 8.00 mm to (93.6, 25.4)
Routing:
- net N$2: track 23.4 -> 15.4 mm
Other:
- board size 105.1 x 100.3 mm -> 100.1 x 100.3 mm
Changed lines of the file:
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@@
 <setting verticaltext="up"/>
 </settings>
-<grid distance="50" unitdist="mil" unit="mm" style="lines" multiple="1" display="no" altdistance="5" altunitdist="mil" altunit="mil"/>
+<grid distance="1" unitdist="mm" unit="mm" style="lines" multiple="1" display="no" altdistance="5" altunitdist="mil" altunit="mil"/>
 <layers>
 <layer number="1" name="Top" color="4" fill="1" visible="yes" active="yes"/>
@@
 <board>
 <plain>
-<wire x1="0" y1="0" x2="105.08" y2="0" width="0" layer="20"/>
-<wire x1="105.08" y1="0" x2="105.08" y2="100.32" width="0" layer="20"/>
-<wire x1="105.08" y1="100.32" x2="0" y2="100.32" width="0" layer="20"/>
+<wire x1="0" y1="0" x2="100.08" y2="0" width="0" layer="20"/>
+<wire x1="100.08" y1="0" x2="100.08" y2="100.32" width="0" layer="20"/>
+<wire x1="100.08" y1="100.32" x2="0" y2="100.32" width="0" layer="20"/>
 <wire x1="0" y1="100.32" x2="0" y2="0" width="0" layer="20"/>
-<dimension x1="0" y1="100.32" x2="104.14" y2="100.33" x3="52.0695125" y3="105.405121875" textsize="1.778" layer="1"/>
-<dimension x1="105.08" y1="100.32" x2="105.08" y2="0" x3="124.46" y3="50.16" textsize="1.778" layer="1"/>
 <hole x="95" y="5" drill="4.5"/>
 <hole x="5" y="95" drill="4.5"/>
 <hole x="5" y="5" drill="4.5"/>
+<dimension x1="2" y1="95" x2="2" y2="5" x3="-21" y3="50" textsize="1.778" layer="49" dtype="diameter"/>
+<dimension x1="5" y1="2" x2="95" y2="2" x3="50" y3="-8" textsize="1.778" layer="49" dtype="diameter"/>
+<dimension x1="100.08" y1="100.32" x2="0" y2="100.32" x3="50.04" y3="103" textsize="1.778" layer="49"/>
+<dimension x1="100.08" y1="0" x2="100.08" y2="100.32" x3="117" y3="50.16" textsize="1.778" layer="49"/>
 </plain>
 <attributes>
@@
 <element name="U$6" library="SPEAR" package="PP45_HOR_2BOT" value="PP45_HOR_2BOT" x="11.43" y="36.83" rot="R180"/>
 <element name="U$7" library="SPEAR" package="PP45_HOR_2BOT" value="PP45_HOR_2BOT" x="11.43" y="16.51" rot="R180"/>
-<element name="U$8" library="SPEAR" package="AMP-MTE-2MALE" value="AMP-MTE-2MALE" x="101.6" y="25.4" rot="R90"/>
+<element name="U$8" library="SPEAR" package="AMP-MTE-2MALE" value="AMP-MTE-2MALE" x="93.6" y="25.4" rot="R90"/>
 <element name="U$9" library="SPEAR-PDU" package="R-78E3.3-0.5" value="R-78E3.3-0.5" x="76.2" y="22.86"/>
 <element name="U$10" library="SPEAR-PDU" package="01220090Z" value="30A_FUSE" x="57.15" y="88.9" rot="R90"/>
@@
 <contactref element="U$9" pad="VOUT"/>
 <contactref element="U$8" pad="P$1"/>
-<wire x1="78.74" y1="22.86" x2="100.33" y2="22.86" width="0.8128" layer="1"/>
-<wire x1="100.33" y1="22.86" x2="101.6" y2="24.13" width="0.8128" layer="1"/>
+<wire x1="78.74" y1="22.86" x2="92.33" y2="22.86" width="0.8128" layer="1"/>
+<wire x1="92.33" y1="22.86" x2="93.6" y2="24.13" width="0.8128" layer="1"/>
 </signal>
 <signal name="N$3">
