File: position_feedback/Main.kicad_pcb (KiCad board)
At the start: 2 copper layers, 30 x 30 mm, 6 parts, among them J1 Conn_01x03, U1 Potentiometer

Commit message: Fixed footprint stuff and added 3d model for pot.
Parts:
- U1: footprint SPEAR Arm Encoder:Potentiometer -> pot:Potentiometer
- moved U1 1.00 mm to (135.0, 100.0)
Routing:
- net /SIGNAL: track 16.2 -> 19.2 mm
- net /VCC: track 12.0 -> 13.5 mm
Changed lines of the file:
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@@
     (links 5)
     (no_connects 0)
-    (area 119.924999 69.924999 150.075001 115.075001)
+    (area 119.924999 84.924999 150.075001 115.075001)
     (thickness 1.6)
     (drawings 17)
-    (tracks 8)
+    (tracks 9)
     (zones 0)
     (modules 6)
@@
     (pad ~ thru_hole circle (at 0 0) (size 6.5 6.5) (drill 3.2) (layers *.Cu *.Mask))
   )
-  (module "SPEAR Arm Encoder:Potentiometer" (layer F.Cu)
-    (at 135 101)
-    (fp_text reference U1 (at 0 7.1) (layer F.SilkS)
-      (effects (font (size 1 1) (thickness 0.15)))
-    )
-    (fp_text value Potentiometer (at 0 -8.2) (layer F.Fab)
-      (effects (font (size 1 1) (thickness 0.15)))
-    )
-    (fp_line (start 3 -2.5) (end -0.9 -5.3) (layer F.SilkS) (width 0.15))
-    (fp_circle (center 0 -2.5) (end 3 -2.5) (layer F.SilkS) (width 0.15))
-    (fp_line (start -5 -7.5) (end -5 4) (layer F.SilkS) (width 0.15))
-    (fp_line (start 5 -7.5) (end -5 -7.5) (layer F.SilkS) (width 0.15))
-    (fp_line (start 5 4) (end 5 -7.5) (layer F.SilkS) (width 0.15))
-    (fp_line (start -5 4) (end 5 4) (layer F.SilkS) (width 0.15))
-    (fp_text user GND (at -6 -5 90) (layer F.SilkS)
-      (effects (font (size 1 1) (thickness 0.15)))
-    )
-    (fp_text user GND (at 6 -5 90) (layer F.SilkS)
-      (effects (font (size 1 1) (thickness 0.15)))
-    )
-    (fp_text user GND (at 2.5 2.6 270) (layer F.SilkS)
-      (effects (font (size 1 1) (thickness 0.15)))
-    )
-    (fp_text user SIG (at 0 2.5 90) (layer F.SilkS)
-      (effects (font (size 1 1) (thickness 0.15)))
-    )
-    (fp_text user VCC (at -2.6 2.6 270) (layer F.SilkS)
-      (effects (font (size 1 1) (thickness 0.15)))
-    )
-    (pad 1 thru_hole circle (at -2.5 5) (size 1.5 1.5) (drill 1) (layers *.Cu *.Mask)
+  (module pot:Potentiometer (layer F.Cu)
+    (at 135 100)
+    (fp_text reference U1 (at 0 9.6) (layer F.SilkS)
+      (effects (font (size 1 1) (thickness 0.15)))
+    )
+    (fp_text value Potentiometer (at 0 -5.7) (layer F.Fab)
+      (effects (font (size 1 1) (thickness 0.15)))
+    )
+    (fp_line (start 3 0) (end -0.9 -2.8) (layer F.SilkS) (width 0.15))
+    (fp_circle (center 0 0) (end 3 0) (layer F.SilkS) (width 0.15))
+    (fp_line (start -5 -5) (end -5 6.5) (layer F.SilkS) (width 0.15))
+    (fp_line (start 5 -5) (end -5 -5) (layer F.SilkS) (width 0.15))
+    (fp_line (start 5 6.5) (end 5 -5) (layer F.SilkS) (width 0.15))
+    (fp_line (start -5 6.5) (end 5 6.5) (layer F.SilkS) (width 0.15))
+    (fp_text user GND (at -6 -2.5 90) (layer F.SilkS)
+      (effects (font (size 1 1) (thickness 0.15)))
+    )
+    (fp_text user GND (at 6 -2.5 90) (layer F.SilkS)
+      (effects (font (size 1 1) (thickness 0.15)))
+    )
+    (fp_text user GND (at 2.5 5.1 270) (layer F.SilkS)
+      (effects (font (size 1 1) (thickness 0.15)))
+    )
+    (fp_text user SIG (at 0 5 90) (layer F.SilkS)
+      (effects (font (size 1 1) (thickness 0.15)))
+    )
+    (fp_text user VCC (at -2.6 5.1 270) (layer F.SilkS)
+      (effects (font (size 1 1) (thickness 0.15)))
+    )
+    (pad 1 thru_hole circle (at -2.5 7.5) (size 1.5 1.5) (drill 1) (layers *.Cu *.Mask)
       (net 2 /VCC))
-    (pad 2 thru_hole circle (at 0 5) (size 1.5 1.5) (drill 1) (layers *.Cu *.Mask)
+    (pad 2 thru_hole circle (at 0 7.5) (size 1.5 1.5) (drill 1) (layers *.Cu *.Mask)
       (net 3 /SIGNAL))
-    (pad 3 thru_hole circle (at 2.5 5) (size 1.5 1.5) (drill 1) (layers *.Cu *.Mask)
+    (pad 3 thru_hole circle (at 2.5 7.5) (size 1.5 1.5) (drill 1) (layers *.Cu *.Mask)
       (net 1 /GND))
-    (pad 4 thru_hole circle (at -5.7 -2.5) (size 1.5 1.5) (drill 1) (layers *.Cu *.Mask)
+    (pad 4 thru_hole circle (at -5.7 0) (size 1.5 1.5) (drill 1) (layers *.Cu *.Mask)
       (net 1 /GND))
-    (pad 5 thru_hole circle (at 5.6 -2.5) (size 1.5 1.5) (drill 1) (layers *.Cu *.Mask)
+    (pad 5 thru_hole circle (at 5.6 0) (size 1.5 1.5) (drill 1) (layers *.Cu *.Mask)
       (net 1 /GND))
+    (model C:/Users/David/13150-L5.wrl
+      (at (xyz 0 0 0.45))
+      (scale (xyz 1 1 1))
+      (rotate (xyz -90 0 0))
+    )
   )
   (dimension 20 (width 0.3) (layer Cmts.User)
@@
   (gr_line (start 120 115) (end 120 85) (layer Edge.Cuts) (width 0.15))
   (gr_line (start 150 115) (end 150 115) (layer Edge.Cuts) (width 0.15))
-  (gr_text SPEAR (at 135 111.75 360) (layer F.SilkS)
+  (gr_text SPEAR (at 135 111.75) (layer F.SilkS)
     (effects (font (size 1.5 1.5) (thickness 0.3)))
   )
-  (gr_text Top (at 140.75 92.1 360) (layer B.SilkS)
+  (gr_text Top (at 140.75 92.1) (layer B.SilkS)
     (effects (font (size 1.5 1.5) (thickness 0.3)) (justify mirror))
   )
@@
   )
   (gr_line (start 150 115) (end 120 115) (layer Edge.Cuts) (width 0.15))
-  (segment (start 132.5 106) (end 135 103.5) (width 0.25) (layer F.Cu) (net 2))
-  (segment (start 135 103.5) (end 135 95) (width 0.25) (layer F.Cu) (net 2))
-  (segment (start 135 106) (end 133.924999 107.075001) (width 0.25) (layer F.Cu) (net 3))
-  (segment (start 133.924999 107.075001) (end 131.983999 107.075001) (width 0.25) (layer F.Cu) (net 3))
-  (segment (start 131.983999 107.075001) (end 131.424999 106.516001) (width 0.25) (layer F.Cu) (net 3))
-  (segment (start 131.424999 106.516001) (end 131.424999 96.035001) (width 0.25) (layer F.Cu) (net 3))
-  (segment (start 131.424999 96.035001) (end 131.610001 95.849999) (width 0.25) (layer F.Cu) (net 3))
-  (segment (start 131.610001 95.849999) (end 132.46 95) (width 0.25) (layer F.Cu) (net 3))
+  (segment (start 132.5 106.31) (end 135 103.81) (width 0.25) (layer F.Cu) (net 2))
+  (segment (start 135 103.81) (end 135 95) (width 0.25) (layer F.Cu) (net 2))
+  (segment (start 132.5 107.5) (end 132.5 106.31) (width 0.25) (layer F.Cu) (net 2))
+  (segment (start 135 107.5) (end 133.85 108.65) (width 0.25) (layer F.Cu) (net 3))
+  (segment (start 133.85 108.65) (end 131.43 108.65) (width 0.25) (layer F.Cu) (net 3))
+  (segment (start 131.43 108.65) (end 130.16 107.38) (width 0.25) (layer F.Cu) (net 3))
+  (segment (start 130.16 107.38) (end 130.16 104.84) (width 0.25) (layer F.Cu) (net 3))
+  (segment (start 130.16 104.84) (end 132.46 102.54) (width 0.25) (layer F.Cu) (net 3))
+  (segment (start 132.46 102.54) (end 132.46 95) (width 0.25) (layer F.Cu) (net 3))
   (zone (net 1) (net_name /GND) (layer F.Cu) (hatch edge 0.508)
     (connect_pads (clearance 0.508))
