File: raspberrypi_canbus_hat/can bus hat.brd (EAGLE design)
At the start: 32 x 55 mm, 15 parts, among them CON1 SM04B-GHS-TB, J1 RASPBERRYPI-40-PIN-GPIO_PTH_N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, U1 MCP2515

Commit message: fixed footprint mcp2562 and modify raspberry pi HAT
Parts:
- added C3, C4: 100nF, rcl:C0805
- added CON2: SM04B-GHS-TB, ARVP:SM04B-GHS-TB
- added LED2: (no value), led:CHIP-LED0805
- added R1: 1k, rcl:R0805
- moved LED1 4.40 mm to (12.2, 30.6), turned to 270 degrees
- moved U$1 3.78 mm to (21.2, 41.4), turned to 0 degrees
- moved CON1 2.79 mm to (27.2, 48.3), turned to 90 degrees
- moved R5 0.89 mm to (11.7, 37.8)
- moved C7 0.89 mm to (11.7, 42.2)
- moved C8 0.89 mm to (11.7, 40.0)
- moved C2 0.28 mm to (23.1, 17.1)
Connections:
- new net N$8: LED2.A, R1.2
- net 3.3V: now also C4.1, U$1.5; no longer U$1.7
- net 5V: now also C3.1, CON2.P$1, R1.1, U$1.3; no longer U$1.6
- net CANH: now also CON2.P$2, U$1.7; no longer U$1.1
- net CANL: now also CON2.P$3, U$1.6; no longer U$1.2
- net GND: now also C3.2, C4.2, CON2.P$4, CON2.P$5, CON2.P$6, LED2.C, U$1.2; no longer U$1.4
- net N$3: now also U$1.1; no longer U$1.5
- net N$5: now also U$1.4; no longer U$1.3
Routing:
- net GPIO25: track 0.00 -> 34.4 mm, vias 0 -> 4
- net 5V: track 22.1 -> 43.3 mm, vias 0 -> 5
- net CE0: track 0.00 -> 19.2 mm, vias 0 -> 1
- net CANH: track 4.27 -> 19.7 mm
- net N$8: track 0.00 -> 13.0 mm, vias 0 -> 2
- net CANL: track 4.26 -> 16.5 mm, vias 0 -> 2
- net N$6: track 0.00 -> 8.44 mm
- net N$5: track 24.3 -> 17.9 mm
- net 3.3V: track 65.3 -> 67.9 mm
- net MOSI: track 22.1 -> 24.6 mm, vias 1 -> 2
- net N$3: track 19.8 -> 21.5 mm
Other:
- outline, holes or cut-outs redrawn
- board text added: "Raspberry Pi CAN Bus HAT"
- board text added: "v1.0"

Commit message: fixed raspberrypi pinout
Parts:
- CON1, CON2: device ARVP:SM04B-GHS-TB -> SPEAR:SM04B-GHS-TB
- D1: device _mod_diode:SOD123 -> adafruit:SOD-123
- U1: device SparkFun-IC-Comms:SO18W -> SPEAR:SO18W
- moved J1 48.3 mm to (6.35, 2.54), turned to 90 degrees
- moved U1 0.63 mm to (22.4, 28.7)
- moved C1 0.52 mm to (26.3, 16.6)
- moved C2 0.51 mm to (23.1, 16.6)
- moved X1 0.38 mm to (24.6, 20.7)
Routing:
- net N$4: track 0.00 -> 59.5 mm
- net 3.3V: track 67.9 -> 87.8 mm, vias 2 -> 4
- net GPIO22: track 6.34 -> 19.7 mm, vias 0 -> 1
- net CE0: track 19.2 -> 25.8 mm, vias 1 -> 0
- net CLK: track 25.3 -> 19.6 mm
- net GPIO25: track 34.4 -> 38.8 mm, vias 4 -> 2
- net MOSI: track 24.6 -> 20.3 mm, vias 2 -> 1
- net MISO: track 22.7 -> 18.5 mm, vias 0 -> 1
- net CANH: track 19.7 -> 19.0 mm
- net N$6: track 8.44 -> 9.07 mm
- net N$5: track 17.9 -> 18.6 mm
- net N$3: track 21.5 -> 22.1 mm
- removed copper zone on layer 1, net N$4
Other:
- outline, holes or cut-outs redrawn
- board text added: "-->"
- board text added: "v1.1"
- board text removed: "v1.0"
