File: raspberrypi_canbus_hat/can bus hat.sch (EAGLE design)
At the start: 15 parts, among them CON1 SM04B-GHS-TB, J1 RASPBERRYPI-40-PIN-GPIO_PTH_N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, U1 MCP2515

Commit message: fixed footprint mcp2562 and modify raspberry pi HAT
Parts:
- added C3, C4: 100nF, rcl:C-EUC0805
- added CON2: SM04B-GHS-TB, ARVP:SM04B-GHS-TB
- added LED2: (no value), led:LEDCHIP-LED0805
- added R1: 1k, rcl:R-US_R0805
Connections:
- new net N$8: LED2.A, R1.2
- net 3.3V: now also C4.1
- net 5V: now also C3.1, CON2-1.S, R1.1
- net CANH: now also CON2-2.S
- net CANL: now also CON2-3.S
- net GND: now also C3.2, C4.2, CON2-4.S, CON2-TABS.S, LED2.C

Commit message: fixed raspberrypi pinout
Parts:
- CON1, CON2: device ARVP:SM04B-GHS-TB -> SPEAR:SM04B-GHS-TB
- D1: device _mod_diode:DIODE-SOD123 -> adafruit:DIODESOD-123
- U1: device SparkFun-IC-Comms:MCP2515(MCP2510)SO -> SPEAR:MCP2515(MCP2510)SO
Other:
- note added: "Changes"
- note added: "V1.1: change the orientation of raspberry pi pinout"
- moved on the sheet: C3, C4, C5, C6, C7, C8, CON1-1, CON1-2, CON1-3, CON1-4, CON1-TABS, CON2-1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
