File: science_controller/science_controller.sch (EAGLE design)
At the start: 3 parts, among them U1 STM32F303CB

Commit message: Did stuff.
Still need to add bypass caps, CAN bus stuff,
and possibly an I2C multiplexer.
Parts:
- added C1, C2: 22pF, resistor:C-EUC0805
- added C3, C4: 1uF, resistor:C-EUC0805
- added J1: ED350/2, SPEAR-science-controller:ED350/2
- added JP1: CORTEX-M-DBG, SPEAR-general:CORTEX-M-DBG
- added JP2, JP3, JP4: (no value), pinhead:PINHD-1X16
- added U2: AP2112K-3.3TRG1, SPEAR-general:AP2112K-3.3TRG1
- added U3: PCA9685PW, SPEAR-science-controller:PCA9685PW
- added Y1: NX5032, SPEAR-general:NX5032
Connections:
- new net N$1: C1.1, U1-MISC.PF0/OSC_IN, Y1.2
- new net N$2: C2.1, U1-MISC.PF1/OSC_OUT, Y1.1
- new net NRST: JP1.!RESET, U1-MISC.NRST
- new net SERVO0: JP2.1, U3.LED0
- new net SERVO1: JP2.2, U3.LED1
- new net SERVO10: JP2.11, U3.LED10
- new net SERVO11: JP2.12, U3.LED11
- new net SERVO12: JP2.13, U3.LED12
- new net SERVO13: JP2.14, U3.LED13
- new net SERVO14: JP2.15, U3.LED14
- new net SERVO15: JP2.16, U3.LED15
- new net SERVO2: JP2.3, U3.LED2
- new net SERVO3: JP2.4, U3.LED3
- new net SERVO4: JP2.5, U3.LED4
- new net SERVO5: JP2.6, U3.LED5
- new net SERVO6: JP2.7, U3.LED6
- new net SERVO7: JP2.8, U3.LED7
- new net SERVO8: JP2.9, U3.LED8
- new net SERVO9: JP2.10, U3.LED9
- new net SERVO_!OE: U3.!OE
- new net SWCLK: JP1.SWCLK/TCK, U1-PORTA.PA14
- new net SWDIO: JP1.SWDIO/TMS, U1-PORTA.PA13
- new net SWO: JP1.SWO/TDO, U1-PORTB.PB3
- new net VCC: J1.1, JP3.1, JP3.10, JP3.11, JP3.12, JP3.13, JP3.14, JP3.15, JP3.16, JP3.2, JP3.3, JP3.4, JP3.5, JP3.6, JP3.7, JP3.8, JP3.9
- net +3V3: now also C4.1, JP1.VCC, U2.VOUT
- net +5V: now also C3.1, U2.EN, U2.VIN, U3.VDD
- net GND: now also C1.2, C2.2, C3.2, C4.2, J1.2, JP1.GND_1, JP1.GND_2, JP1.GND_DETECT, JP4.1, JP4.10, JP4.11, JP4.12, JP4.13, JP4.14, JP4.15, JP4.16, JP4.2, JP4.3, JP4.4, JP4.5, JP4.6, JP4.7, JP4.8, JP4.9, U2.GND, U3.A0, U3.A1, U3.A2, U3.A3, U3.A4, U3.A5, U3.VSS
- net SCL: now also U1-PORTB.PB6, U3.SCL; no longer U1-PORTA.PA15
- net SDA: now also U1-PORTB.PB7, U3.SDA; no longer U1-PORTA.PA14
Other:
- note added: "Need Bypass caps"
- note added: "Standard servo pinout: Signal -> Power -> Ground"
- note removed: "Need PCA9685 or something for servos."
- note removed: "Need Power regulation"
- note removed: "We need 12V battery in for Servos"
