File: science_controller/science_controller.sch (EAGLE design)
At the start: 25 parts, among them CON1 UAVCAN_MICRO, CON2 UAVCAN_MICRO, J1 ED350/2, U1 STM32F303CB, U2 AP2112K-3.3TRG1, U3 PCA9685PW, Y1 NX5032

Commit message: Finished first revision of science controller board.
Needs review!
Parts:
- added P1: I2C-PWR, SPEAR-science-controller:I2C-PWR
- added R1, R2: 4k7, resistor:R-EU_R0805
- JP2, JP3, JP4: value (none) -> PINHD-16; device pinhead:PINHD-1X16 -> SPEAR-science-controller:PINHD-16
Connections:
- removed net CAN_RX: U1-PORTA.PA11
- removed net CAN_TX: U1-PORTA.PA12
- net +3V3: now also P1.VCC, R1.2, R2.2
- net CAN_RXD: now also U1-PORTA.PA11
- net CAN_TXD: now also U1-PORTA.PA12
- net GND: now also P1.GND
- net SCL: now also P1.SCL, R1.1
- net SDA: now also P1.SDA, R2.1
- net USART2_RX: now also U1-PORTA.PA3
- net USART2_TX: no longer U1-PORTA.PA3
Other:
- note added: "External I2C Connector"
- note added: "I2C Pullups"
