File: arm_pdu/ARM_PDU.brd (EAGLE design)
At the start: 106.4 x 102.9 mm, 18 parts

Commit message: Tweaked board dimensions
Parts:
- moved 2PIN_CONNECTOR1 5.39 mm to (94.0, 87.6)
- moved 2PIN_CONNECTOR2 5.39 mm to (94.0, 76.2)
- moved 2PIN_CONNECTOR3 5.39 mm to (94.0, 64.8)
- moved 2PIN_CONNECTOR5 5.39 mm to (94.0, 41.9)
- moved U$1 5.39 mm to (64.8, 90.2)
- moved U$2 5.39 mm to (64.8, 78.7)
- moved U$3 5.39 mm to (64.8, 67.3)
- moved 2PIN_CONNECTOR6 5.39 mm to (94.0, 30.5)
- moved U$4 5.39 mm to (30.5, 83.8)
- moved U$5 5.39 mm to (30.5, 63.5)
- moved U$6 5.39 mm to (30.5, 40.6)
- moved U$9 5.39 mm to (59.7, 21.6)
- moved 2PIN_CONNECTOR4 5.39 mm to (94.0, 53.3)
- moved U$14 5.39 mm to (64.8, 55.9)
- moved U$15 5.39 mm to (64.8, 44.5)
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Other:
- board size 106.4 x 102.9 mm -> 100 x 100 mm
