File: arm_pdu/ARM_PDU.brd (EAGLE design)
At the start: 100 x 100 mm, 18 parts

Commit message: fixed issues with board not being in sync with schematic
Parts:
- removed 2PIN_CONNECTOR1, 2PIN_CONNECTOR2, 2PIN_CONNECTOR3, 2PIN_CONNECTOR4, 2PIN_CONNECTOR5, 2PIN_CONNECTOR6: 2PIN_CONNECTOR, 2PIN_CONNECTOR:2PIN_CONNECTOR
- added U$10, U$11, U$12, U$13, U$17, U$18: 2PIN_5MM, SPEAR-arm-pdu:2PIN_5MM
Connections:
- removed net V: 2PIN_CONNECTOR1.P$1, 2PIN_CONNECTOR2.P$1, 2PIN_CONNECTOR3.P$1, 2PIN_CONNECTOR4.P$1, 2PIN_CONNECTOR5.P$1, 2PIN_CONNECTOR6.P$1, U$1.P$1, U$1.P$3, U$14.P$1, U$14.P$3, U$15.P$1, U$15.P$3, U$16.P$1, U$16.P$3, U$2.P$1, U$2.P$3, U$3.P$1, U$3.P$3, U$4.+, U$5.+, U$6.+, U$7.+, U$9.+VIN
- new net +VBAT: U$1.P$1, U$14.P$1, U$15.P$1, U$16.P$1, U$2.P$1, U$3.P$1, U$4.+, U$5.+, U$6.+, U$7.+, U$9.+VIN
- new net OUT1: U$1.P$3, U$13.P$1
- new net OUT2: U$17.P$1, U$2.P$3
- new net OUT3: U$18.P$1, U$3.P$3
- new net OUT4: U$10.P$2, U$16.P$3
- new net OUT5: U$11.P$2, U$15.P$3
- new net OUT6: U$12.P$2, U$14.P$3
- net GND: now also U$10.P$1, U$11.P$1, U$12.P$1, U$13.P$2, U$17.P$2, U$18.P$2; no longer 2PIN_CONNECTOR1.P$2, 2PIN_CONNECTOR2.P$2, 2PIN_CONNECTOR3.P$2, 2PIN_CONNECTOR4.P$2, 2PIN_CONNECTOR5.P$2, 2PIN_CONNECTOR6.P$2
Routing:
- added copper zone on layer 1, net +VBAT
- added copper zone on layer 1, net OUT1
- added copper zone on layer 1, net OUT2
- added copper zone on layer 1, net OUT3
- added copper zone on layer 1, net OUT4
- added copper zone on layer 1, net OUT5
- added copper zone on layer 1, net OUT6
- removed copper zone on layer 1, net V

Commit message: fixed hole size issues
Parts:
- moved U$13 1.38 mm to (95.2, 87.6)
- moved U$11 0.60 mm to (95.2, 40.6)
- moved U$10 0.54 mm to (95.2, 30.5)
- moved U$12 0.46 mm to (95.2, 53.3)
- moved U$17 0.39 mm to (95.2, 76.2)
- moved U$18 0.23 mm to (95.2, 64.8)
Changed lines of the file:
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@@
 <element name="U$15" library="20A_FUSE_HOLDER" package="20A_FUSE_HOLDER" value="20A_FUSE_HOLDER" x="64.77" y="44.45" smashed="yes"/>
 <element name="U$16" library="20A_FUSE_HOLDER" package="20A_FUSE_HOLDER" value="20A_FUSE_HOLDER" x="64.77" y="33.02" smashed="yes"/>
-<element name="U$10" library="SPEAR-arm-pdu" package="2PIN_5MM" value="2PIN_5MM" x="95" y="30" smashed="yes" rot="R90"/>
-<element name="U$11" library="SPEAR-arm-pdu" package="2PIN_5MM" value="2PIN_5MM" x="95" y="41.19" smashed="yes" rot="R90"/>
-<element name="U$12" library="SPEAR-arm-pdu" package="2PIN_5MM" value="2PIN_5MM" x="95" y="53.73" smashed="yes" rot="R90"/>
-<element name="U$13" library="SPEAR-arm-pdu" package="2PIN_5MM" value="2PIN_5MM" x="94.7" y="86.36" smashed="yes" rot="R270"/>
-<element name="U$17" library="SPEAR-arm-pdu" package="2PIN_5MM" value="2PIN_5MM" x="94.86" y="76.2" smashed="yes" rot="R270"/>
-<element name="U$18" library="SPEAR-arm-pdu" package="2PIN_5MM" value="2PIN_5MM" x="95.02" y="64.77" smashed="yes" rot="R270"/>
+<element name="U$10" library="SPEAR-arm-pdu" package="2PIN_5MM" value="2PIN_5MM" x="95.25" y="30.48" smashed="yes" rot="R90"/>
+<element name="U$11" library="SPEAR-arm-pdu" package="2PIN_5MM" value="2PIN_5MM" x="95.25" y="40.64" smashed="yes" rot="R90"/>
+<element name="U$12" library="SPEAR-arm-pdu" package="2PIN_5MM" value="2PIN_5MM" x="95.25" y="53.34" smashed="yes" rot="R90"/>
+<element name="U$13" library="SPEAR-arm-pdu" package="2PIN_5MM" value="2PIN_5MM" x="95.25" y="87.63" smashed="yes" rot="R270"/>
+<element name="U$17" library="SPEAR-arm-pdu" package="2PIN_5MM" value="2PIN_5MM" x="95.25" y="76.2" smashed="yes" rot="R270"/>
+<element name="U$18" library="SPEAR-arm-pdu" package="2PIN_5MM" value="2PIN_5MM" x="95.25" y="64.77" smashed="yes" rot="R270"/>
 </elements>
 <signals>
@@
 <contactref element="U$17" pad="P$2"/>
 <contactref element="U$18" pad="P$2"/>
+<wire x1="95.25" y1="73.7" x2="95.25" y2="62.27" width="0" layer="19" extent="1-1"/>
+<wire x1="95.25" y1="85.13" x2="95.25" y2="73.7" width="0" layer="19" extent="1-1"/>
+<wire x1="95.25" y1="50.84" x2="95.25" y2="85.13" width="0" layer="19" extent="1-1"/>
+<wire x1="95.25" y1="38.14" x2="95.25" y2="50.84" width="0" layer="19" extent="1-1"/>
+<wire x1="95.25" y1="27.98" x2="95.25" y2="38.14" width="0" layer="19" extent="1-1"/>
+<wire x1="30.48" y1="21.717" x2="95.25" y2="27.98" width="0" layer="19" extent="1-1"/>
 </signal>
 <signal name="N$2">
@@
 <contactref element="U$1" pad="P$3"/>
 <contactref element="U$13" pad="P$1"/>
+<wire x1="85.27" y1="90.17" x2="95.25" y2="90.13" width="0" layer="19" extent="1-1"/>
 </signal>
 <signal name="+VBAT">
@@
 <signal name="OUT2">
 <contactref element="U$2" pad="P$3"/>
-<contactref element="U$17" pad="P$1"/>
 <polygon width="0.1524" layer="1">
 <vertex x="80.01" y="81.28"/>
@@
 <vertex x="80.01" y="74.93"/>
 </polygon>
+<contactref element="U$17" pad="P$1"/>
+<wire x1="85.27" y1="78.74" x2="95.25" y2="78.7" width="0" layer="19" extent="1-1"/>
 </signal>
 <signal name="OUT3">
 <contactref element="U$3" pad="P$3"/>
-<contactref element="U$18" pad="P$1"/>
 <polygon width="0.1524" layer="1">
 <vertex x="80.01" y="69.85"/>
@@
 <vertex x="80.01" y="63.5"/>
 </polygon>
+<contactref element="U$18" pad="P$1"/>
+<wire x1="85.27" y1="67.31" x2="95.25" y2="67.27" width="0" layer="19" extent="1-1"/>
 </signal>
 <signal name="OUT4">
 <contactref element="U$16" pad="P$3"/>
-<contactref element="U$10" pad="P$2"/>
 <polygon width="0.1524" layer="1">
 <vertex x="80.01" y="35.56"/>
@@
 <vertex x="80.01" y="29.21"/>
 </polygon>
+<contactref element="U$10" pad="P$2"/>
+<wire x1="85.27" y1="33.02" x2="95.25" y2="32.98" width="0" layer="19" extent="1-1"/>
 </signal>
 <signal name="OUT5">
-<contactref element="U$11" pad="P$2"/>
 <contactref element="U$15" pad="P$3"/>
 <polygon width="0.1524" layer="1">
@@
 <vertex x="80.01" y="40.64"/>
 </polygon>
+<contactref element="U$11" pad="P$2"/>
+<wire x1="85.27" y1="44.45" x2="95.25" y2="43.14" width="0" layer="19" extent="1-1"/>
 </signal>
 <signal name="OUT6">
 <contactref element="U$14" pad="P$3"/>
-<contactref element="U$12" pad="P$2"/>
 <polygon width="0.1524" layer="1">
 <vertex x="80.01" y="59.69"/>
@@
 <vertex x="80.01" y="53.34"/>
 </polygon>
+<contactref element="U$12" pad="P$2"/>
+<wire x1="85.27" y1="55.88" x2="95.25" y2="55.84" width="0" layer="19" extent="1-1"/>
 </signal>
 </signals>
