File: drive_controller/DriveControllerBoard.brd (EAGLE design)
At the start: 100 x 100 mm, 18 parts, among them CON1 UAVCAN_MICRO, CON2 UAVCAN_MICRO, U1 AP2112K-3.3TRG1, U2 STM32F303CB

Commit message: Fixed some things
Parts:
- added C6, C7: 22p, resistor:C0805
- added C8, C9: 0u1, resistor:C0805
- added U$4: AMP-MTE-2MALE, SPEAR-general:AMP-MTE-2MALE
- added Y1: NX5032, SPEAR-general:NX5032
- C1: value (none) -> 4u7
- C2, C3, C4, C5: value (none) -> 0u1
- R1: value (none) -> 10k
- R3, R4, R5, R6: value (none) -> 10K
- U$1, U$2: value ED2732-ND -> AMP-MTE-4MALE; device ED2732-ND:ED2732-ND -> SPEAR-drive-controller:AMP-MTE-4MALE
- moved CON1 75.0 mm to (95.0, 82.0), turned to 90 degrees
- moved CON2 69.4 mm to (95.0, 70.0), turned to 90 degrees
- moved U$2 41.2 mm to (96.0, 54.0), turned to 270 degrees
- moved R1 35.0 mm to (72.0, 59.0)
- moved JP1 31.3 mm to (64.0, 57.9)
- moved R4 26.9 mm to (84.8, 57.1), turned to 90 degrees
- moved R3 25.4 mm to (87.7, 57.1), turned to 90 degrees
- moved C5 25.0 mm to (72.0, 39.0), turned to 90 degrees
- moved U$3 22.5 mm to (77.0, 71.0), turned to 270 degrees
- moved C4 18.8 mm to (69.0, 39.0), turned to 90 degrees
- moved R6 18.8 mm to (88.0, 35.0), turned to 270 degrees
- moved U2 18.4 mm to (76.8, 46.0), turned to 0 degrees
- moved C3 14.0 mm to (66.0, 39.0), turned to 90 degrees
- moved R5 13.9 mm to (84.0, 35.0), turned to 270 degrees
- moved C1 13.6 mm to (60.0, 39.0), turned to 90 degrees
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Connections:
- removed net N$8: R1.2, U2.7
- new net NRST: JP1.10, R1.2, U2.7
- new net OSC_IN: C7.1, U2.5, Y1.P$1
- new net OSC_OUT: C6.1, U2.6, Y1.P$2
- net +3V3: now also C9.1; no longer JP1.10
- net +5V: now also C8.1, U$1.3, U$2.3, U1.3; no longer U$1.P$3, U$2.P$3
- net 1A: now also U$2.1; no longer U$2.P$1
- net 1B: now also U$2.2; no longer U$2.P$2
- net 2A: now also U$1.1; no longer U$1.P$1
- net 2B: now also U$1.2; no longer U$1.P$2
- net GND: now also C6.2, C7.2, C8.2, C9.2, U$1.4, U$2.4, U$4.P$2; no longer U$1.P$4, U$2.P$4
- net USART_3: now also U$4.P$1
Routing:
- net GND: track 238.8 -> 67.5 mm, vias 2 -> 14
- net 1A: track 110.9 -> 22.3 mm
- net N$1: track 109.5 -> 28.7 mm, vias 0 -> 2
- net +3V3: track 172.6 -> 94.6 mm, vias 6 -> 2
- net N$4: track 91.5 -> 30.6 mm
- net 2B: track 74.6 -> 21.1 mm
- net 2A: track 64.9 -> 21.3 mm
- net N$8: track 40.5 -> 0.00 mm
- net 1B: track 62.2 -> 28.3 mm, vias 2 -> 0
- net +5V: track 182.4 -> 149.6 mm, vias 4 -> 5
- net USART_3: track 0.00 -> 32.3 mm
- net NRST: track 0.00 -> 26.2 mm, vias 0 -> 4
- net SWCLK: track 37.8 -> 14.0 mm, vias 2 -> 0
- net TRACESWO: track 34.7 -> 14.0 mm
- net SWDIO: track 35.5 -> 15.2 mm, vias 2 -> 0
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- added copper zone on layer 16, net GND

Commit message: Fixing errors. Still a few to be fixed.
Connections:
- net N$1 renamed CANH
- net N$4 renamed CANL
- net CANRX: now also U2.32; no longer U2.33
- net CANTX: now also U2.33; no longer U2.32
- net GND: now also U$3.8
Routing:
- net CANTX: track 23.4 -> 2.42 mm
- net CANRX: track 19.3 -> 1.77 mm
Changed lines of the file:
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@@
 <?xml version="1.0" encoding="utf-8"?>
 <!DOCTYPE eagle SYSTEM "eagle.dtd">
-<eagle version="9.3.0">
+<eagle version="9.4.1">
 <drawing>
 <settings>
@@
 <wire x1="93.98" y1="72.045" x2="93.98" y2="72.709" width="0.2032" layer="1"/>
 <via x="93.98" y="72.709" extent="1-16" drill="0.35"/>
+<contactref element="U$3" pad="8"/>
+<wire x1="97.35" y1="73.725" x2="93.98" y2="72.709" width="0" layer="19" extent="1-1"/>
+<wire x1="84.381" y1="66.338" x2="93.98" y2="72.045" width="0" layer="19" extent="1-1"/>
+<wire x1="79.75" y1="72.905" x2="82.677" y2="66.359" width="0" layer="19" extent="1-1"/>
+<wire x1="74.25" y1="71.635" x2="79.75" y2="72.905" width="0" layer="19" extent="1-1"/>
+<wire x1="71.374" y1="66.105" x2="73.718" y2="71.635" width="0" layer="19" extent="1-1"/>
+<wire x1="61.976" y1="59.12" x2="69.759" y2="66.132" width="0" layer="19" extent="1-1"/>
+<wire x1="67.056" y1="49.214" x2="64.262" y2="53.405" width="0" layer="19" extent="1-1"/>
+<wire x1="70.612" y1="44.769" x2="66.988" y2="47.8" width="0" layer="19" extent="1-1"/>
+<wire x1="72" y1="38.05" x2="71.591" y2="43.79" width="0" layer="19" extent="1-1"/>
+<wire x1="73.152" y1="30.164" x2="73.914" y2="36.006" width="0" layer="19" extent="1-1"/>
+<wire x1="79.95" y1="28" x2="74.05" y2="28" width="0" layer="19" extent="1-1"/>
+<wire x1="74.5" y1="50.29" x2="70.612" y2="44.769" width="0" layer="19" extent="1-1"/>
+<wire x1="81" y1="48.29" x2="74.5" y2="50.29" width="0" layer="19" extent="1-1"/>
+<wire x1="96" y1="50.19" x2="82.677" y2="48.325" width="0" layer="19" extent="1-1"/>
+<wire x1="96" y1="42.81" x2="96" y2="50.19" width="0" layer="19" extent="1-1"/>
+<wire x1="97" y1="27.73" x2="96" y2="42.81" width="0" layer="19" extent="1-1"/>
 </signal>
-<signal name="N$1">
+<signal name="CANH">
 <contactref element="U$3" pad="7"/>
 <contactref element="CON2" pad="2"/>
@@
 <wire x1="92.867" y1="81.375" x2="94.15" y2="81.375" width="0.2032" layer="1"/>
 </signal>
-<signal name="N$4">
+<signal name="CANL">
 <contactref element="CON1" pad="3"/>
 <contactref element="CON2" pad="3"/>
@@
 </signal>
 <signal name="CANRX">
-<contactref element="U2" pad="33"/>
 <contactref element="U$3" pad="4"/>
-<wire x1="75.5" y1="50.29" x2="75.5" y2="67.845" width="0.2032" layer="1"/>
 <wire x1="75.5" y1="67.845" x2="74.25" y2="69.095" width="0.2032" layer="1"/>
+<contactref element="U2" pad="32"/>
+<wire x1="76" y1="50.29" x2="75.5" y2="67.845" width="0" layer="19" extent="1-1"/>
 </signal>
 <signal name="CANTX">
-<contactref element="U2" pad="32"/>
 <contactref element="U$3" pad="1"/>
 <wire x1="75.1052125" y1="72.189" x2="74.966" y2="72.189" width="0.2032" layer="1"/>
 <wire x1="74.966" y1="72.189" x2="74.25" y2="72.905" width="0.2032" layer="1"/>
-<wire x1="76" y1="50.29" x2="76" y2="71.2942125" width="0.2032" layer="1"/>
 <wire x1="76" y1="71.2942125" x2="75.1052125" y2="72.189" width="0.2032" layer="1"/>
+<contactref element="U2" pad="33"/>
+<wire x1="75.5" y1="50.29" x2="76" y2="71.2942125" width="0" layer="19" extent="1-1"/>
 </signal>
 <signal name="1B">

Commit message: corrected layout issues.
Routing:
- net CANTX: track 2.42 -> 26.9 mm
- net CANRX: track 1.77 -> 19.5 mm
- net GND: track 67.5 -> 70.3 mm, vias 14 -> 15
Changed lines of the file:
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@@
 <setting verticaltext="up"/>
 </settings>
-<grid distance="1" unitdist="mm" unit="mm" style="lines" multiple="1" display="no" altdistance="1" altunitdist="mm" altunit="mm"/>
+<grid distance="10" unitdist="mil" unit="mil" style="lines" multiple="1" display="no" altdistance="1" altunitdist="mm" altunit="mm"/>
 <layers>
 <layer number="1" name="Top" color="4" fill="1" visible="yes" active="yes"/>
@@
 <via x="93.98" y="72.709" extent="1-16" drill="0.35"/>
 <contactref element="U$3" pad="8"/>
+<wire x1="79.75" y1="72.905" x2="82.543" y2="72.905" width="0.254" layer="1"/>
+<wire x1="82.543" y1="72.905" x2="82.55" y2="72.898" width="0.254" layer="1"/>
+<via x="82.55" y="72.898" extent="1-16" drill="0.35"/>
 <wire x1="97.35" y1="73.725" x2="93.98" y2="72.709" width="0" layer="19" extent="1-1"/>
 <wire x1="84.381" y1="66.338" x2="93.98" y2="72.045" width="0" layer="19" extent="1-1"/>
-<wire x1="79.75" y1="72.905" x2="82.677" y2="66.359" width="0" layer="19" extent="1-1"/>
+<wire x1="82.55" y1="72.898" x2="82.677" y2="66.359" width="0" layer="19" extent="1-1"/>
 <wire x1="74.25" y1="71.635" x2="79.75" y2="72.905" width="0" layer="19" extent="1-1"/>
 <wire x1="71.374" y1="66.105" x2="73.718" y2="71.635" width="0" layer="19" extent="1-1"/>
@@
 <signal name="CANRX">
 <contactref element="U$3" pad="4"/>
-<wire x1="75.5" y1="67.845" x2="74.25" y2="69.095" width="0.2032" layer="1"/>
 <contactref element="U2" pad="32"/>
-<wire x1="76" y1="50.29" x2="75.5" y2="67.845" width="0" layer="19" extent="1-1"/>
+<wire x1="76" y1="50.29" x2="76" y2="67.345" width="0.254" layer="1"/>
+<wire x1="76" y1="67.345" x2="74.25" y2="69.095" width="0.254" layer="1"/>
 </signal>
 <signal name="CANTX">
 <contactref element="U$3" pad="1"/>
-<wire x1="75.1052125" y1="72.189" x2="74.966" y2="72.189" width="0.2032" layer="1"/>
-<wire x1="74.966" y1="72.189" x2="74.25" y2="72.905" width="0.2032" layer="1"/>
-<wire x1="76" y1="71.2942125" x2="75.1052125" y2="72.189" width="0.2032" layer="1"/>
 <contactref element="U2" pad="33"/>
-<wire x1="75.5" y1="50.29" x2="76" y2="71.2942125" width="0" layer="19" extent="1-1"/>
+<wire x1="75.5" y1="50.29" x2="75.5" y2="66.232" width="0.254" layer="1"/>
+<wire x1="72.898" y1="69.18813125" x2="73.49546875" y2="69.7856" width="0.254" layer="1"/>
+<wire x1="75.692" y1="70.358" x2="75.692" y2="72.39" width="0.254" layer="1"/>
+<wire x1="75.692" y1="72.39" x2="75.177" y2="72.905" width="0.254" layer="1"/>
+<wire x1="75.177" y1="72.905" x2="74.25" y2="72.905" width="0.254" layer="1"/>
+<wire x1="75.5" y1="66.232" x2="72.898" y2="68.834" width="0.254" layer="1"/>
+<wire x1="72.898" y1="68.834" x2="72.898" y2="69.18813125" width="0.254" layer="1"/>
+<wire x1="75.68813125" y1="70.358" x2="75.692" y2="70.358" width="0.254" layer="1"/>
+<wire x1="75.11573125" y1="69.7856" x2="75.68813125" y2="70.358" width="0.254" layer="1"/>
+<wire x1="73.49546875" y1="69.7856" x2="75.11573125" y2="69.7856" width="0.254" layer="1"/>
 </signal>
 <signal name="1B">
