File: drive_controller/DriveControllerBoard.brd (EAGLE design)
At the start: 100 x 100 mm, 24 parts, among them CON1 UAVCAN_MICRO, CON2 UAVCAN_MICRO, U1 AP2112K-3.3TRG1, U2 STM32F303CB, Y1 NX5032

Commit message: first commit
Parts:
- removed C1: 4u7, resistor:C0805
- removed C3, C4, C5, C8, C9: 0u1, resistor:C0805
- removed C6, C7: 22p, resistor:C0805
- removed CON1, CON2: UAVCAN_MICRO, SPEAR-general:SM04B-GHS-TB
- removed JP1: CORTEX-M-DBG, SPEAR-general:FTSH-105-01-F-DV-007
- removed R1: 10k, resistor:R0805
- removed U1: AP2112K-3.3TRG1, SPEAR-general:SOT25
- removed U2: STM32F303CB, SPEAR-general:LQFP48
- removed Y1: NX5032, SPEAR-general:NX5032
- added D1: CGRM4001-G, diode:SOD-123_MINI-SMA
- added U$5, U$6: AMP-MTE-4MALE, SPEAR-drive-controller:AMP-MTE-4MALE
- C2: value 0u1 -> 100nf; device resistor:C0805 -> rcl:C0805
- U$3: value MCP2562-E/SN -> STM-DEV-BOARD; device SPEAR-general:SOIC8 -> SPEAR:STM-DEV-BOARD
- moved U$3 48.6 mm to (58.9, 25.9), turned to 0 degrees
- moved C2 11.3 mm to (65.5, 27.9), turned to 270 degrees
Connections:
- removed net CANRX: U$3.4, U2.32
- removed net CANTX: U$3.1, U2.33
- removed net N$3: JP1.8
- removed net NRST: JP1.10, R1.2, U2.7
- removed net OSC_IN: C7.1, U2.5, Y1.P$1
- removed net OSC_OUT: C6.1, U2.6, Y1.P$2
- removed net SWCLK: JP1.4, U2.37
- removed net SWDIO: JP1.2, U2.34
- removed net TRACESWO: JP1.6, U2.39
- new net 5V: C2.1, D1.A, U$3.5V, U$5.1, U$6.1
- new net N$5: U$3.GND@3
- net +3V3: now also R3.2, R4.2, R5.2, R6.2, U$1.3, U$2.3, U$3.3.3V; no longer C1.2, C2.2, C3.2, C4.2, C5.2, C9.1, JP1.1, R1.1, U$3.5, U1.5, U2.24, U2.36, U2.48
- net +5V: now also D1.C; no longer C8.1, CON1.1, CON2.1, R3.2, R4.2, R5.2, R6.2, U$1.3, U$2.3, U$3.3, U1.1, U1.3
- net 1A: now also U$3.PA5; no longer U2.29
- net 1B: now also U$3.PA6; no longer U2.30
- net 2A: now also U$3.PA2; no longer U2.10
- net 2B: now also U$3.PA3; no longer U2.11
- net CANH: now also U$3.CANH, U$5.2, U$6.2; no longer CON1.2, CON2.2, U$3.7
- net CANL: now also U$3.CANL, U$5.3, U$6.3; no longer CON1.3, CON2.3, U$3.6
- net GND: now also C2.2, U$3.GND, U$3.GND@2, U$5.4, U$6.4; no longer C1.1, C2.1, C3.1, C4.1, C5.1, C6.2, C7.2, C8.2, C9.2, CON1.4, CON1.TAB_A, CON1.TAB_B, CON2.4, CON2.TAB_A, CON2.TAB_B, JP1.3, JP1.5, JP1.9, U$3.2, U$3.8, U1.2, U2.23, U2.35, U2.47
- net USART_3: now also U$3.PA4; no longer U2.21
Routing:
- net +5V: track 149.6 -> 12.9 mm, vias 5 -> 0
- net 5V: track 0.00 -> 37.5 mm
- net CANTX: track 26.9 -> 0.00 mm
- net NRST: track 26.2 -> 0.00 mm, vias 4 -> 0
- net CANL: track 30.6 -> 53.1 mm, vias 2 -> 0
- net CANRX: track 19.5 -> 0.00 mm
- net CANH: track 28.7 -> 47.2 mm, vias 2 -> 0
- net OSC_OUT: track 17.8 -> 0.00 mm
- net OSC_IN: track 17.2 -> 0.00 mm
- net SWDIO: track 15.2 -> 0.00 mm
- net TRACESWO: track 14.0 -> 0.00 mm
- net SWCLK: track 14.0 -> 0.00 mm
- net +3V3: track 94.6 -> 86.3 mm, vias 2 -> 1
- net USART_3: track 32.3 -> 34.9 mm
- net GND: track 70.3 -> 68.3 mm, vias 15 -> 5
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- added copper zone on layer 1, net GND
- removed copper zone on layer 16, net GND
Other:
- board size 100 x 100 mm -> 47.7 x 100 mm

Commit message: got rid of useless traces
Parts:
- moved D1 5.14 mm to (72.6, 31.2), turned to 90 degrees
Connections:
- removed net 5V: C2.1, D1.A, U$3.5V, U$5.1, U$6.1
- net +5V: now also C2.1, D1.A, U$3.5V, U$5.1, U$6.1
Routing:
- net GND: track 68.3 -> 11.2 mm, vias 5 -> 2
- net 5V: track 37.5 -> 0.00 mm
- net +5V: track 12.9 -> 43.4 mm, vias 0 -> 2
- net +3V3: track 86.3 -> 95.5 mm
- net CANL: track 53.1 -> 58.0 mm
- net 1B: track 26.5 -> 24.7 mm
- net CANH: track 47.2 -> 47.8 mm

Commit message: made the board a bit smaller and other small changes
Parts:
- moved U$1 1.27 mm to (94.7, 39.0)
- moved U$2 1.27 mm to (94.7, 54.0)
Connections:
- removed net N$5: U$3.GND@3
- net GND: now also U$3.GND@3
Routing:
- net GND: track 11.2 -> 6.12 mm, vias 2 -> 1
- net +3V3: track 95.5 -> 99.3 mm
- net 2B: track 21.1 -> 19.8 mm
- net 2A: track 19.8 -> 18.5 mm
- net 1B: track 24.7 -> 23.5 mm
- net 1A: track 20.9 -> 19.9 mm
Other:
- board size 47.7 x 100 mm -> 47.7 x 91 mm
- board text added: "SPEAR 2020 JACK OPGENORTH DRIVE CONTROLLER REVISION"
- board text removed: "SPEAR 2019 JACK DE WIT DRIVE CONTROLLER BOARD"
Changed lines of the file:
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@@
 <board>
 <plain>
-<wire x1="52.324" y1="99.873" x2="52.324" y2="0.889" width="0" layer="20"/>
+<wire x1="52.324" y1="90.873" x2="52.324" y2="0.889" width="0" layer="20"/>
 <wire x1="52.324" y1="0.889" x2="52.705" y2="0" width="0" layer="20" curve="90"/>
 <wire x1="52.705" y1="0" x2="99.365" y2="0" width="0" layer="20"/>
 <wire x1="99.365" y1="0" x2="100" y2="0.635" width="0" layer="20" curve="90"/>
-<wire x1="100" y1="0.635" x2="100" y2="99.365" width="0" layer="20"/>
-<wire x1="100" y1="99.365" x2="99.365" y2="100" width="0" layer="20" curve="90"/>
-<wire x1="99.365" y1="100" x2="52.705" y2="100" width="0" layer="20"/>
-<wire x1="52.705" y1="100" x2="52.324" y2="99.873" width="0" layer="20" curve="90"/>
-<text x="62.752" y="0.934" size="1.778" layer="21">SPEAR 2019
-JACK DE WIT
-DRIVE CONTROLLER BOARD</text>
-<hole x="56.562" y="2.714" drill="4.5"/>
-<hole x="56.816" y="95.254" drill="4.5"/>
+<wire x1="100" y1="0.635" x2="100" y2="90.365" width="0" layer="20"/>
+<wire x1="100" y1="90.365" x2="99.365" y2="91" width="0" layer="20" curve="90"/>
+<wire x1="99.365" y1="91" x2="52.705" y2="91" width="0" layer="20"/>
+<wire x1="52.705" y1="91" x2="52.324" y2="90.873" width="0" layer="20" curve="90"/>
+<text x="59.45" y="0.934" size="1.778" layer="21">SPEAR 2020
+JACK OPGENORTH
+DRIVE CONTROLLER REVISION</text>
+<hole x="56.562" y="4.714" drill="4.5"/>
+<hole x="56.816" y="86.254" drill="4.5"/>
 <hole x="95" y="5" drill="4.5"/>
-<hole x="95" y="95" drill="4.5"/>
+<hole x="95" y="86" drill="4.5"/>
 </plain>
 <attributes>
@@
 </element>
 <element name="U$4" library="SPEAR-general" package="AMP-MTE-2MALE" value="AMP-MTE-2MALE" x="97" y="29" smashed="yes" rot="R270"/>
-<element name="U$2" library="SPEAR-drive-controller" package="AMP-MTE-4MALE" value="AMP-MTE-4MALE" x="96" y="54" smashed="yes" rot="R270"/>
-<element name="U$1" library="SPEAR-drive-controller" package="AMP-MTE-4MALE" value="AMP-MTE-4MALE" x="96" y="39" smashed="yes" rot="R90"/>
+<element name="U$2" library="SPEAR-drive-controller" package="AMP-MTE-4MALE" value="AMP-MTE-4MALE" x="94.73" y="54" smashed="yes" rot="R270"/>
+<element name="U$1" library="SPEAR-drive-controller" package="AMP-MTE-4MALE" value="AMP-MTE-4MALE" x="94.73" y="39" smashed="yes" rot="R90"/>
 <element name="U$3" library="SPEAR" package="STM-DEV-BOARD" value="STM-DEV-BOARD" x="58.928" y="25.908" smashed="yes">
 <attribute name="NAME" x="69.088" y="60.96" size="1.27" layer="25"/>
@@
 <contactref element="U$1" pad="4"/>
 <contactref element="C2" pad="2"/>
-<polygon width="0.1524" layer="1">
-<vertex x="51.562" y="80.264"/>
-<vertex x="51.562" y="-2.032"/>
-<vertex x="53.34" y="-0.254"/>
-<vertex x="100.584" y="-0.254"/>
-<vertex x="100.584" y="80.264"/>
-</polygon>
 <contactref element="U$5" pad="4"/>
 <contactref element="U$6" pad="4"/>
-<contactref element="U$3" pad="GND"/>
-<contactref element="U$3" pad="GND@2"/>
-<via x="53.848" y="10.414" extent="1-16" drill="0.35"/>
-<wire x1="58.674" y1="10.922" x2="54.356" y2="10.922" width="0.3048" layer="1"/>
-<wire x1="54.356" y1="10.922" x2="53.848" y2="10.414" width="0.3048" layer="1"/>
 <via x="70.358" y="23.876" extent="1-16" drill="0.35"/>
 <wire x1="65.532" y1="26.99" x2="67.244" y2="26.99" width="0.381" layer="1"/>
 <wire x1="67.244" y1="26.99" x2="70.358" y2="23.876" width="0.381" layer="1"/>
+<contactref element="U$3" pad="GND"/>
+<contactref element="U$3" pad="GND@3"/>
+<contactref element="U$3" pad="GND@2"/>
+<polygon width="0.1524" layer="1">
+<vertex x="51.816" y="82.042"/>
+<vertex x="78.486" y="82.042"/>
+<vertex x="100.584" y="59.944"/>
+<vertex x="100.584" y="27.94"/>
+<vertex x="94.234" y="21.59"/>
+<vertex x="80.264" y="7.62"/>
+<vertex x="49.784" y="7.62"/>
+<vertex x="49.784" y="80.01"/>
+</polygon>
 </signal>
 <signal name="1B">
@@
 <contactref element="U$2" pad="2"/>
 <contactref element="U$3" pad="PA6"/>
-<wire x1="96.9525" y1="57.41545625" x2="96.9525" y2="58.20454375" width="0.2032" layer="1"/>
-<wire x1="96.9525" y1="58.20454375" x2="96.39454375" y2="58.7625" width="0.2032" layer="1"/>
-<wire x1="96.39454375" y1="58.7625" x2="95.60545625" y2="58.7625" width="0.2032" layer="1"/>
 <wire x1="85.8917875" y1="56.177" x2="84.809" y2="56.177" width="0.2032" layer="1"/>
-<wire x1="86.7957875" y1="57.081" x2="85.8917875" y2="56.177" width="0.2032" layer="1"/>
-<wire x1="95.60545625" y1="58.7625" x2="93.92395625" y2="57.081" width="0.2032" layer="1"/>
-<wire x1="93.92395625" y1="57.081" x2="86.7957875" y2="57.081" width="0.2032" layer="1"/>
-<wire x1="96" y1="55.27" x2="96" y2="56.46295625" width="0.2032" layer="1"/>
-<wire x1="96" y1="56.46295625" x2="96.9525" y2="57.41545625" width="0.2032" layer="1"/>
+<wire x1="85.8917875" y1="56.177" x2="86.7957875" y2="57.081" width="0.2032" layer="1"/>
 <wire x1="78.867" y1="51.308" x2="83.736" y2="56.177" width="0.2032" layer="1"/>
 <wire x1="83.736" y1="56.177" x2="84.809" y2="56.177" width="0.2032" layer="1"/>
+<wire x1="94.33545625" y1="58.7625" x2="95.12454375" y2="58.7625" width="0.2032" layer="1"/>
+<wire x1="95.12454375" y1="58.7625" x2="95.6825" y2="58.20454375" width="0.2032" layer="1"/>
+<wire x1="95.6825" y1="58.20454375" x2="95.6825" y2="57.41545625" width="0.2032" layer="1"/>
+<wire x1="86.7957875" y1="57.081" x2="92.65395625" y2="57.081" width="0.2032" layer="1"/>
+<wire x1="94.73" y1="56.46295625" x2="94.73" y2="55.27" width="0.2032" layer="1"/>
+<wire x1="92.65395625" y1="57.081" x2="94.33545625" y2="58.7625" width="0.2032" layer="1"/>
+<wire x1="95.6825" y1="57.41545625" x2="94.73" y2="56.46295625" width="0.2032" layer="1"/>
 </signal>
 <signal name="2A">
@@
 <contactref element="U$1" pad="1"/>
 <contactref element="U$3" pad="PA2"/>
-<wire x1="96" y1="35.19" x2="88.9992125" y2="35.19" width="0.2032" layer="1"/>
-<wire x1="88.9992125" y1="35.19" x2="88.8552125" y2="35.046" width="0.2032" layer="1"/>
 <wire x1="88.8552125" y1="35.046" x2="84.904" y2="35.046" width="0.2032" layer="1"/>
 <wire x1="84.904" y1="35.046" x2="84" y2="35.95" width="0.2032" layer="1"/>
 <wire x1="84" y1="35.95" x2="78.867" y2="41.083" width="0.2032" layer="1"/>
 <wire x1="78.867" y1="41.083" x2="78.867" y2="41.148" width="0.2032" layer="1"/>
+<wire x1="88.8552125" y1="35.046" x2="94.586" y2="35.046" width="0.2032" layer="1"/>
+<wire x1="94.586" y1="35.046" x2="94.73" y2="35.19" width="0.2032" layer="1"/>
 </signal>
 <signal name="2B">
@@
 <contactref element="U$1" pad="2"/>
 <contactref element="U$3" pad="PA3"/>
-<wire x1="96" y1="37.73" x2="94.22" y2="35.95" width="0.2032" layer="1"/>
-<wire x1="94.22" y1="35.95" x2="88" y2="35.95" width="0.2032" layer="1"/>
 <wire x1="88" y1="35.95" x2="80.262" y2="43.688" width="0.2032" layer="1"/>
 <wire x1="80.262" y1="43.688" x2="78.867" y2="43.688" width="0.2032" layer="1"/>
+<wire x1="88" y1="35.95" x2="92.95" y2="35.95" width="0.2032" layer="1"/>
+<wire x1="92.95" y1="35.95" x2="94.73" y2="37.73" width="0.2032" layer="1"/>
 </signal>
 <signal name="1A">
@@
 <contactref element="U$2" pad="1"/>
 <contactref element="U$3" pad="PA5"/>
-<wire x1="96" y1="57.81" x2="94.367" y2="56.177" width="0.2032" layer="1"/>
-<wire x1="94.367" y1="56.177" x2="87.651" y2="56.177" width="0.2032" layer="1"/>
 <wire x1="87.651" y1="56.177" x2="80.242" y2="48.768" width="0.2032" layer="1"/>
 <wire x1="80.242" y1="48.768" x2="78.867" y2="48.768" width="0.2032" layer="1"/>
+<wire x1="94.27955625" y1="57.35955625" x2="94.73" y2="57.81" width="0.2032" layer="1"/>
+<wire x1="94.27955625" y1="56.9337" x2="94.27955625" y2="57.35955625" width="0.2032" layer="1"/>
+<wire x1="87.651" y1="56.177" x2="93.52285625" y2="56.177" width="0.2032" layer="1"/>
+<wire x1="93.52285625" y1="56.177" x2="94.27955625" y2="56.9337" width="0.2032" layer="1"/>
 </signal>
 <signal name="USART_3">
@@
 <wire x1="97.296" y1="34.05" x2="97.79" y2="34.544" width="0.508" layer="1"/>
 <wire x1="97.79" y1="34.544" x2="97.79" y2="38.48" width="0.508" layer="1"/>
-<wire x1="97.79" y1="38.48" x2="96" y2="40.27" width="0.508" layer="1"/>
-<wire x1="96" y1="40.27" x2="98.044" y2="42.314" width="0.508" layer="16"/>
-<wire x1="98.044" y1="42.314" x2="98.044" y2="44.007" width="0.508" layer="16"/>
+<wire x1="98.044" y1="44.007" x2="98.044" y2="42.314" width="0.508" layer="16"/>
 <wire x1="98.044" y1="44.007" x2="98.044" y2="50.686" width="0.508" layer="1"/>
-<wire x1="98.044" y1="50.686" x2="96" y2="52.73" width="0.508" layer="1"/>
-<wire x1="96" y1="52.73" x2="96" y2="53.70743125" width="0.508" layer="1"/>
-<wire x1="96" y1="53.70743125" x2="98.73" y2="56.43743125" width="0.508" layer="1"/>
+<wire x1="98.73" y1="56.43743125" x2="96" y2="53.70743125" width="0.508" layer="1"/>
 <wire x1="98.73" y1="56.43743125" x2="98.73" y2="59.436" width="0.508" layer="1"/>
 <wire x1="98.73" y1="59.436" x2="96.952" y2="61.214" width="0.508" layer="1"/>
@@
 <wire x1="87.651" y1="59.203" x2="87.651" y2="58.077" width="0.508" layer="1"/>
 <wire x1="87.651" y1="58.077" x2="84.809" y2="58.077" width="0.508" layer="1"/>
-</signal>
-<signal name="N$5">
-<contactref element="U$3" pad="GND@3"/>
+<wire x1="97.79" y1="38.48" x2="96" y2="40.27" width="0.508" layer="1"/>
+<wire x1="96" y1="40.27" x2="94.73" y2="40.27" width="0.508" layer="1"/>
+<wire x1="98.044" y1="42.314" x2="96" y2="40.27" width="0.508" layer="16"/>
+<wire x1="96" y1="40.27" x2="94.73" y2="40.27" width="0.508" layer="16"/>
+<wire x1="98.044" y1="50.686" x2="96" y2="52.73" width="0.508" layer="1"/>
+<wire x1="96" y1="52.73" x2="94.73" y2="52.73" width="0.508" layer="1"/>
+<wire x1="96" y1="53.70743125" x2="96" y2="52.73" width="0.508" layer="1"/>
 </signal>
 </signals>
