File: drive_controller/DriveControllerBoard.sch (EAGLE design)
At the start: 18 parts, among them CON1 UAVCAN_MICRO, CON2 UAVCAN_MICRO, U1 AP2112K-3.3TRG1, U2 STM32F303CB

Commit message: Fixed some things
Parts:
- added C6, C7: 22p, resistor:C-EUC0805
- added C8, C9: 0u1, resistor:C-EUC0805
- added U$4: AMP-MTE-2MALE, SPEAR-general:AMP-MTE-2MALE
- added Y1: NX5032, SPEAR-general:NX5032
- C1: value (none) -> 4u7
- C2, C3, C4, C5: value (none) -> 0u1
- R1: value (none) -> 10k
- R3, R4, R5, R6: value (none) -> 10K
- U$1, U$2: value ED2732-ND -> AMP-MTE-4MALE; device ED2732-ND:ED2732-ND -> SPEAR-drive-controller:AMP-MTE-4MALE
Connections:
- removed net N$8: R1.2, U2-MISC.NRST
- new net NRST: JP1.!RESET, R1.2, U2-MISC.NRST
- new net OSC_IN: C7.1, U2-MISC.PF0/OSC_IN, Y1.1
- new net OSC_OUT: C6.1, U2-MISC.PF1/OSC_OUT, Y1.2
- net +3V3: now also C9.1; no longer JP1.!RESET
- net +5V: now also C8.1, U$1.3, U$2.3, U1.EN; no longer U$1.P$3, U$2.P$3
- net 1A: now also U$2.1; no longer U$2.P$1
- net 1B: now also U$2.2; no longer U$2.P$2
- net 2A: now also U$1.1; no longer U$1.P$1
- net 2B: now also U$1.2; no longer U$1.P$2
- net GND: now also C6.2, C7.2, C8.2, C9.2, U$1.4, U$2.4, U$4.P$2; no longer U$1.P$4, U$2.P$4
- net USART_3: now also U$4.P$1

Commit message: Fixing errors. Still a few to be fixed.
Connections:
- net N$1 renamed CANH
- net N$4 renamed CANL
- net CANRX: now also U2-PORTA.PA11; no longer U2-PORTA.PA12
- net CANTX: now also U2-PORTA.PA12; no longer U2-PORTA.PA11
- net GND: now also U$3.STBY
Changed lines of the file:
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@@
 <?xml version="1.0" encoding="utf-8"?>
 <!DOCTYPE eagle SYSTEM "eagle.dtd">
-<eagle version="9.3.0">
+<eagle version="9.4.1">
 <drawing>
 <settings>
@@
 <part name="GND9" library="supply1" library_urn="urn:adsk.eagle:library:371" deviceset="GND" device=""/>
 <part name="JP1" library="SPEAR-general" deviceset="CORTEX-M-DBG" device=""/>
+<part name="GND10" library="supply1" library_urn="urn:adsk.eagle:library:371" deviceset="GND" device=""/>
 </parts>
 <sheets>
@@
 </instance>
 <instance part="JP1" gate="G$1" x="2.54" y="147.32" smashed="yes"/>
+<instance part="GND10" gate="1" x="22.86" y="86.36" smashed="yes" rot="R90">
+<attribute name="VALUE" x="25.4" y="83.82" size="1.778" layer="96" rot="R90"/>
+</instance>
 </instances>
 <busses>
@@
 <pinref part="GND9" gate="1" pin="GND"/>
 </segment>
+<segment>
+<pinref part="U$3" gate="G$1" pin="STBY"/>
+<wire x1="10.16" y1="86.36" x2="20.32" y2="86.36" width="0.1524" layer="91"/>
+<pinref part="GND10" gate="1" pin="GND"/>
+</segment>
 </net>
-<net name="N$1" class="0">
+<net name="CANH" class="0">
 <segment>
 <wire x1="27.94" y1="99.06" x2="27.94" y2="93.98" width="0.1524" layer="91"/>
@@
 <wire x1="-25.4" y1="93.98" x2="27.94" y2="93.98" width="0.1524" layer="91"/>
 <junction x="27.94" y="93.98"/>
+<label x="17.78" y="76.2" size="1.778" layer="95"/>
 </segment>
 </net>
-<net name="N$4" class="0">
+<net name="CANL" class="0">
 <segment>
 <pinref part="CON1" gate="G$1" pin="CANL"/>
@@
 <wire x1="40.64" y1="71.12" x2="30.48" y2="71.12" width="0.1524" layer="91"/>
 <junction x="30.48" y="71.12"/>
+<label x="17.78" y="71.12" size="1.778" layer="95"/>
 </segment>
 </net>
 <net name="CANRX" class="0">
+<segment>
+<pinref part="U$3" gate="G$1" pin="RXD"/>
+<wire x1="-17.78" y1="71.12" x2="-25.4" y2="71.12" width="0.1524" layer="91"/>
+<label x="-27.94" y="71.12" size="1.778" layer="95"/>
+</segment>
+<segment>
+<pinref part="U2" gate="-PORTA" pin="PA11"/>
+<wire x1="-55.88" y1="111.76" x2="-48.26" y2="111.76" width="0.1524" layer="91"/>
+<label x="-48.26" y="111.76" size="1.778" layer="95"/>
+</segment>
+</net>
+<net name="CANTX" class="0">
+<segment>
+<pinref part="U$3" gate="G$1" pin="TXD"/>
+<wire x1="-17.78" y1="76.2" x2="-25.4" y2="76.2" width="0.1524" layer="91"/>
+<label x="-27.94" y="76.2" size="1.778" layer="95"/>
+</segment>
 <segment>
 <pinref part="U2" gate="-PORTA" pin="PA12"/>
@@
 <label x="-48.26" y="109.22" size="1.778" layer="95"/>
 </segment>
-<segment>
-<pinref part="U$3" gate="G$1" pin="RXD"/>
-<wire x1="-17.78" y1="71.12" x2="-25.4" y2="71.12" width="0.1524" layer="91"/>
-<label x="-27.94" y="71.12" size="1.778" layer="95"/>
-</segment>
 </net>
-<net name="CANTX" class="0">
-<segment>
-<pinref part="U2" gate="-PORTA" pin="PA11"/>
-<wire x1="-55.88" y1="111.76" x2="-48.26" y2="111.76" width="0.1524" layer="91"/>
-<label x="-48.26" y="111.76" size="1.778" layer="95"/>
-</segment>
-<segment>
-<pinref part="U$3" gate="G$1" pin="TXD"/>
-<wire x1="-17.78" y1="76.2" x2="-25.4" y2="76.2" width="0.1524" layer="91"/>
-<label x="-27.94" y="76.2" size="1.778" layer="95"/>
-</segment>
-</net>

Commit message: first commit
Parts:
- removed C1: 4u7, resistor:C-EUC0805
- removed C3, C4, C5, C8, C9: 0u1, resistor:C-EUC0805
- removed C6, C7: 22p, resistor:C-EUC0805
- removed CON1, CON2: UAVCAN_MICRO, SPEAR-general:UAVCAN_MICRO
- removed JP1: CORTEX-M-DBG, SPEAR-general:CORTEX-M-DBG
- removed R1: 10k, resistor:R-EU_R0805
- removed U1: AP2112K-3.3TRG1, SPEAR-general:AP2112K-3.3TRG1
- removed U2: STM32F303CB, SPEAR-general:STM32F303CB
- removed Y1: NX5032, SPEAR-general:NX5032
- added D1: CGRM4001-G, diode:CGRM4001-G
- added U$5, U$6: AMP-MTE-4MALE, SPEAR-drive-controller:AMP-MTE-4MALE
- C2: value 0u1 -> 100nf; device resistor:C-EUC0805 -> rcl:C-EUC0805
- U$3: value MCP2562-E/SN -> STM-DEV-BOARD; device SPEAR-general:MCP2562-E/SN -> SPEAR:STM-DEV-BOARD
Connections:
- removed net CANRX: U$3.RXD, U2-PORTA.PA11
- removed net CANTX: U$3.TXD, U2-PORTA.PA12
- removed net N$3: JP1.NC/TDI
- removed net NRST: JP1.!RESET, R1.2, U2-MISC.NRST
- removed net OSC_IN: C7.1, U2-MISC.PF0/OSC_IN, Y1.1
- removed net OSC_OUT: C6.1, U2-MISC.PF1/OSC_OUT, Y1.2
- removed net SWCLK: JP1.SWCLK/TCK, U2-PORTA.PA14
- removed net SWDIO: JP1.SWDIO/TMS, U2-PORTA.PA13
- removed net TRACESWO: JP1.SWO/TDO, U2-PORTB.PB3
- new net 5V: C2.1, D1.A, U$3.5V, U$5.1, U$6.1
- new net N$5: U$3.GND@3
- net +3V3: now also R3.2, R4.2, R5.2, R6.2, U$1.3, U$2.3, U$3.3.3V@1; no longer C1.2, C2.2, C3.2, C4.2, C5.2, C9.1, JP1.VCC, R1.1, U$3.VIO, U1.VOUT, U2-PWR.VDD_1, U2-PWR.VDD_2, U2-PWR.VDD_3
- net +5V: now also D1.C; no longer C8.1, CON1.+5V, CON2.+5V, R3.2, R4.2, R5.2, R6.2, U$1.3, U$2.3, U$3.VDD, U1.EN, U1.VIN
- net 1A: now also U$3.PA5; no longer U2-PORTA.PA8
- net 1B: now also U$3.PA6; no longer U2-PORTA.PA9
- net 2A: now also U$3.PA2; no longer U2-PORTA.PA0
- net 2B: now also U$3.PA3; no longer U2-PORTA.PA1
- net CANH: now also U$5.2, U$6.2; no longer CON1.CANH, CON2.CANH
- net CANL: now also U$5.3, U$6.3; no longer CON1.CANL, CON2.CANL
- net GND: now also C2.2, U$3.GND@1, U$3.GND@2, U$5.4, U$6.4; no longer C1.1, C2.1, C3.1, C4.1, C5.1, C6.2, C7.2, C8.2, C9.2, CON1.GND, CON1.TABS, CON2.GND, CON2.TABS, JP1.GND_1, JP1.GND_2, JP1.GND_DETECT, U$3.STBY, U$3.VSS, U1.GND, U2-PWR.VSS_1, U2-PWR.VSS_2, U2-PWR.VSS_3
- net USART_3: now also U$3.PA4; no longer U2-PORTB.PB10
Other:
- moved on the sheet: C2

Commit message: got rid of useless traces
Connections:
- removed net 5V: C2.1, D1.A, U$3.5V, U$5.1, U$6.1
- net +5V: now also C2.1, D1.A, U$3.5V, U$5.1, U$6.1
Changed lines of the file:
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@@
 <instance part="D1" gate="G$1" x="-73.66" y="40.64" smashed="yes" rot="R180">
 <attribute name="NAME" x="-76.2" y="40.1574" size="1.778" layer="95" rot="R180"/>
-<attribute name="VALUE" x="-76.2" y="42.9514" size="1.778" layer="96" rot="R180"/>
+<attribute name="VALUE" x="-68.58" y="45.4914" size="1.778" layer="96" rot="R180"/>
 </instance>
 <instance part="U$5" gate="G$1" x="104.14" y="20.32" smashed="yes">
@@
 <label x="-96.52" y="40.64" size="1.778" layer="95"/>
 </segment>
+<segment>
+<pinref part="U$3" gate="G$1" pin="5V"/>
+<label x="-53.34" y="40.64" size="1.778" layer="95"/>
+<pinref part="D1" gate="G$1" pin="A"/>
+<wire x1="-71.12" y1="40.64" x2="-60.96" y2="40.64" width="0.1524" layer="91"/>
+<pinref part="C2" gate="G$1" pin="1"/>
+<wire x1="-60.96" y1="40.64" x2="-45.72" y2="40.64" width="0.1524" layer="91"/>
+<wire x1="-60.96" y1="30.48" x2="-60.96" y2="40.64" width="0.1524" layer="91"/>
+<junction x="-60.96" y="40.64"/>
+</segment>
+<segment>
+<pinref part="U$6" gate="G$1" pin="1"/>
+<wire x1="106.68" y1="5.08" x2="96.52" y2="5.08" width="0.1524" layer="91"/>
+<label x="99.06" y="5.08" size="1.778" layer="95"/>
+</segment>
+<segment>
+<pinref part="U$5" gate="G$1" pin="1"/>
+<wire x1="101.6" y1="25.4" x2="91.44" y2="25.4" width="0.1524" layer="91"/>
+<label x="93.98" y="25.4" size="1.778" layer="95"/>
+</segment>
 </net>
 <net name="CANH" class="0">
@@
 </segment>
 </net>
-<net name="5V" class="0">
-<segment>
-<pinref part="U$5" gate="G$1" pin="1"/>
-<wire x1="101.6" y1="25.4" x2="91.44" y2="25.4" width="0.1524" layer="91"/>
-<label x="93.98" y="25.4" size="1.778" layer="95"/>
-</segment>
-<segment>
-<pinref part="U$6" gate="G$1" pin="1"/>
-<wire x1="106.68" y1="5.08" x2="91.44" y2="5.08" width="0.1524" layer="91"/>
-<label x="93.98" y="5.08" size="1.778" layer="95"/>
-</segment>
-<segment>
-<pinref part="C2" gate="G$1" pin="1"/>
-<wire x1="-60.96" y1="30.48" x2="-60.96" y2="38.1" width="0.1524" layer="91"/>
-<label x="-60.96" y="35.56" size="1.778" layer="95" rot="R90" align="bottom-right"/>
-</segment>
-<segment>
-<pinref part="D1" gate="G$1" pin="A"/>
-<wire x1="-71.12" y1="40.64" x2="-63.5" y2="40.64" width="0.1524" layer="91"/>
-<label x="-66.04" y="40.64" size="1.778" layer="95" align="bottom-right"/>
-</segment>
-<segment>
-<pinref part="U$3" gate="G$1" pin="5V"/>
-<wire x1="-45.72" y1="40.64" x2="-53.34" y2="40.64" width="0.1524" layer="91"/>
-<label x="-50.8" y="40.64" size="1.778" layer="95"/>
-</segment>
-</net>

Commit message: made the board a bit smaller and other small changes
Connections:
- removed net N$5: U$3.GND@3
- net GND: now also U$3.GND@3
Changed lines of the file:
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@@
 <part name="+3V1" library="supply1" library_urn="urn:adsk.eagle:library:371" deviceset="+3V3" device=""/>
 <part name="+3V2" library="supply1" library_urn="urn:adsk.eagle:library:371" deviceset="+3V3" device=""/>
-<part name="GND2" library="supply1" library_urn="urn:adsk.eagle:library:371" deviceset="GND" device=""/>
-<part name="GND3" library="supply1" library_urn="urn:adsk.eagle:library:371" deviceset="GND" device=""/>
 </parts>
 <sheets>
@@
 <attribute name="VALUE" x="-55.88" y="30.48" size="1.778" layer="96" rot="R90"/>
 </instance>
-<instance part="GND2" gate="1" x="-50.8" y="22.86" smashed="yes">
-<attribute name="VALUE" x="-53.34" y="20.32" size="1.778" layer="96"/>
-</instance>
-<instance part="GND3" gate="1" x="5.08" y="116.84" smashed="yes">
-<attribute name="VALUE" x="2.54" y="114.3" size="1.778" layer="96"/>
-</instance>
 </instances>
 <busses>
@@
 <segment>
 <pinref part="U$3" gate="G$1" pin="GND@1"/>
-<wire x1="-45.72" y1="35.56" x2="-50.8" y2="35.56" width="0.1524" layer="91"/>
-<wire x1="-50.8" y1="35.56" x2="-50.8" y2="25.4" width="0.1524" layer="91"/>
-<pinref part="GND2" gate="1" pin="GND"/>
+<wire x1="-45.72" y1="35.56" x2="-55.88" y2="35.56" width="0.1524" layer="91"/>
+<label x="-53.34" y="35.56" size="1.778" layer="95"/>
+</segment>
+<segment>
+<pinref part="U$3" gate="G$1" pin="GND@3"/>
+<wire x1="-7.62" y1="127" x2="2.54" y2="127" width="0.1524" layer="91"/>
+<label x="5.08" y="127" size="1.778" layer="95" align="bottom-right"/>
 </segment>
 <segment>
 <pinref part="U$3" gate="G$1" pin="GND@2"/>
-<wire x1="-7.62" y1="121.92" x2="5.08" y2="121.92" width="0.1524" layer="91"/>
-<pinref part="GND3" gate="1" pin="GND"/>
-<wire x1="5.08" y1="121.92" x2="5.08" y2="119.38" width="0.1524" layer="91"/>
+<wire x1="-7.62" y1="121.92" x2="2.54" y2="121.92" width="0.1524" layer="91"/>
+<label x="7.62" y="121.92" size="1.778" layer="95" align="bottom-right"/>
 </segment>
 </net>
@@
 </segment>
 </net>
-<net name="N$5" class="0">
-<segment>
-<pinref part="U$3" gate="G$1" pin="GND@3"/>
-<wire x1="-7.62" y1="127" x2="5.08" y2="127" width="0.1524" layer="91"/>
-</segment>
-</net>
