File: spear-dev-board/Green Pill Sparkfun.sch (EAGLE design)
At the start: 41 parts, among them IC1 STM32F103C8T6, IC2 STM32F103C8T6, U1 3.3V, X1 8MHz, X2 8MHz

Commit message: uploaded bom, PnP, and change some board layout:
Parts:
- removed R11, R12: 4.7k, rcl:R-US_R0603
- removed R13: 1k, rcl:R-US_R0603
- added C6, C7: 22pF, resistor:C-EUC0603
- added U$1: 32.768kHz, SPEAR:KX-327
- R1, R3: value 100k -> 10k
- R7: value 1.5k -> 10k
- R9: value 100 -> 1k
Connections:
- removed net LED_STLINK: IC1.PA9, R13.1
- removed net PA0: IC1.PA0-WKUP, R11.1, R12.2
- removed net RST: IC1.NRST, R4.1
- net 3.3V: now also R9.2; no longer IC1.VBAT, R11.2, R4.2
- net GND: now also C6.2, C7.2, R4.2; no longer IC1.PB2, LED1.C, R12.1
- net N$5: now also IC1.PB2, R4.1; no longer IC1.PC13-TAMPER-RTC, R2.1
- net N$7: now also IC1.PC14-OSC32_IN, LED1.C; no longer LED1.A, R13.2
- net N$8: now also LED1.A; no longer IC1.PB12
- net OSC32_IN: now also C7.1, U$1.2
- net OSC32_OUT: now also C6.1, U$1.1
- net PA10: now also IC1.PA2
- net PA2: no longer IC1.PA3
- net PA3: no longer IC1.PA2
- net PA9: now also IC1.PA3
- net PB2: now also R2.1; no longer JP2.19
- net PC13: now also JP2.19
- net SWCLK: no longer IC1.PB13
- net SWDIO: no longer R9.2
Other:
- note added: "BLACK MAGIC PROBE"
- note removed: "Compatible MCU: * STM32F303CC * STM32F303CB * STM32F103CB * STM32F103C8 * STM32L151C8 * STM32F072C8"
- note removed: "STLINK V2.1"
- moved on the sheet: LED1, R2, R4, R9
