File: spear-dev-board/Green Pill stlink.sch (EAGLE design)
At the start: 41 parts, among them IC1 STM32F103C8T6, IC2 STM32F103C8T6, U1 3.3V, X1 8MHz, X2 8MHz

Commit message: added jumper for MCO switch, updated design
Parts:
- removed C6, C7: 22pF, resistor:C-EUC0603
- removed DCLK, DIO: (no value), wirepad:SMD2
- added JP3: (no value), pinhead:PINHD-1X2
- added R11, R12: 4.7k, rcl:R-US_R0603
- added R13: 1k, rcl:R-US_R0603
- added SJ1: SOLDERJUMPERNC2, SparkFun-Retired:SOLDERJUMPERNC2
- R1, R3: value 10k -> 100k
- R7: value 10k -> 1.5k
- R9: value 1k -> 100
- U$1: value 32.768kHz -> MCP2562-E/SN; device SPEAR:KX-327 -> SPEAR:MCP2562-E/SN
Connections:
- new net CANH: JP1.12, U$1.CANH
- new net CANL: JP1.13, U$1.CANL
- new net LED_STLINK: IC1.PA9, R13.1
- new net N$10: IC1.PA8, SJ1.1
- new net PA0: IC1.PA0-WKUP, R11.1, R12.2
- new net RST: IC1.NRST, R4.1
- net 3.3V: now also IC1.VBAT, R11.2, R4.2, U$1.VIO; no longer R9.2
- net 5V: now also U$1.VDD
- net DCLK: now also JP3.1; no longer DCLK.P
- net DIO: now also JP3.2; no longer DIO.P
- net GND: now also IC1.PB2, LED1.C, R12.1, U$1.STBY, U$1.VSS; no longer C6.2, C7.2, R4.2
- net N$5: now also IC1.PC13-TAMPER-RTC, R2.1; no longer IC1.PB2, R4.1
- net N$7: now also LED1.A, R13.2; no longer IC1.PC14-OSC32_IN, LED1.C
- net N$8: now also IC1.PB12; no longer LED1.A
- net OSC32_IN: no longer C7.1, U$1.2
- net OSC32_OUT: no longer C6.1, U$1.1
- net OSC_IN: now also SJ1.2
- net PA10: no longer IC1.PA2
- net PA11: now also U$1.RXD; no longer JP1.13
- net PA12: now also U$1.TXD; no longer JP1.12
- net PA2: now also IC1.PA3
- net PA3: now also IC1.PA2
- net PA9: no longer IC1.PA3
- net PB2: now also JP2.19; no longer R2.1
- net PC13: no longer JP2.19
- net SWCLK: now also IC1.PB13
- net SWDIO: now also R9.2
Other:
- note added: "CAN BUS"
- note added: "Compatible MCU: * STM32F303CC * STM32F303CB * STM32F103CB * STM32F103C8 * STM32L151C8 * STM32F072C8"
- note added: "STLINK V2.1"
- note removed: "BLACK MAGIC PROBE"
- moved on the sheet: LED1, R2, R4, R6, R9
