File: comp-pdu/Comp PDU.brd (EAGLE design)
At the start: 100 x 70 mm, 39 parts, among them IC1 788TV, J1 POWER_JACK, K1 RELAY-SPDT-JZC-11F, Q1 BCX70SMD, Q2 SMP3003-DL-1E, Q3 SMP3003-DL-1E, U1 3568

Commit message: updated to new relay to commonly used songle 10A, minor changes to layout.
Parts:
- removed JP4: (no value), pinhead:1X02
- removed Q1: BCX70SMD, transistor-npn:SOT23
- removed Q2, Q3: SMP3003-DL-1E, SPEAR:BBS3002DL1E
- removed R10, R11: 100k, rcl:R0805
- removed R9: 1k, rcl:R0805
- added C7: 10uF, rcl:C0805
- added D3: (no value), adafruit:DO-1N4148
- added SWITCH: (no value), pinhead:1X01
- D1: value CGRM4004-G -> (none); device diode:SOD-123_MINI-SMA -> diode:DO214AA
- K1: value RELAY-SPDT-JZC-11F -> SRD-05VDC-SL-C; device SparkFun-Electromechanical:RELAY-JZC -> SPEAR:RELAY_SRD-05VDC-SL-C
- moved D1 53.9 mm to (65.9, 12.1), turned to 180 degrees
- moved K1 2.39 mm to (86.0, 35.7), turned to 0 degrees
Connections:
- removed net N$10: Q2.1, R10.2
- removed net N$5: Q3.1, R11.2
- removed net SW: JP4.2, R9.1
- removed net VOUT1: J1.PWR, Q2.3
- removed net VOUT2: J2.2, Q3.3
- net +5V: no longer D1.C
- net GND: now also C7.2, D3.A, K1.A2; no longer JP4.1, Q1.2, R10.1, R11.1
- net N$4: now also D1.C, J2.2; no longer Q1.1, R9.2
- net N$7: now also D3.C, K1.A1, SWITCH.1; no longer D1.A, K1.1, K1.5, Q1.3
- net VBAT: now also K1.COM; no longer K1.4
- net VIN: now also K1.NO; no longer K1.3
- net VIOUT: now also C7.1
- net VOUT1_FIXED: now also J1.PWR; no longer Q2.2
- net VOUT2_FIXED: now also D1.A; no longer Q3.2
Routing:
- net N$7: track 36.1 -> 22.0 mm
- net CANL: track 72.1 -> 79.7 mm
- net N$10: track 5.39 -> 0.00 mm
- net N$5: track 4.30 -> 0.00 mm
- net SW: track 3.07 -> 0.00 mm
- net N$4: track 2.74 -> 0.00 mm
- net VIOUT: track 5.53 -> 8.06 mm
- net +5V: track 124.0 -> 121.7 mm
- added copper zone on layer 1, net N$4
- removed copper zone on layer 1, net VOUT1
- removed copper zone on layer 1, net VOUT2

Commit message: add connectors for battery monitoring, add more protection to ADC Lines
Parts:
- added C10, C11, C12, C8, C9: 100nF, rcl:C0805
- added D4: (no value), diode:DO-214AC
- added D5, D6, D7, D8, D9: BAT54S, diode:SOT23
- added JP4: (no value), pinhead:1X04
- added R10, R11, R9: 1k, rcl:R0805
- C7: value 10uF -> 100nF
- D2: value 3.6V -> BAT54S; device SparkFun-DiscreteSemi:SOD-323 -> diode:SOT23
- K1: value SRD-05VDC-SL-C -> SRD-24VDC-SL-C
- moved D2 24.5 mm to (34.8, 59.7), turned to 0 degrees
- moved R8 5.72 mm to (40.9, 62.7)
- moved R7 5.71 mm to (40.9, 64.9)
- moved C7 4.07 mm to (35.8, 63.9), turned to 270 degrees
- moved C2 1.09 mm to (61.5, 63.0)
- moved C3 0.90 mm to (76.4, 62.8)
- moved R3 0.28 mm to (6.48, 41.8)
Connections:
- new net N$13: D5.3, JP4.1, R10.1
- new net N$5: D2.3, R7.1, R8.2, R9.1
- new net N$9: D6.3, JP4.4, R11.1
- new net VIOUT1: C8.1, R11.2, U$1.PA4
- new net VIOUT2: C9.1, R10.2, U$1.PA5
- net +3V3: now also D2.2, D5.2, D6.2, D7.2, D8.2, D9.2
- net AIOUT1: now also C10.1, D8.3
- net AIOUT2: now also C11.1, D7.3
- net AIOUT3: now also C12.1, D9.3
- net GND: now also C10.2, C11.2, C12.2, C8.2, C9.2, D2.1, D4.A, D5.1, D6.1, D7.1, D8.1, D9.1, JP4.2, JP4.3; no longer D2.A
- net VIN: now also D4.C; no longer D2.C
- net VIOUT: now also R9.2; no longer R7.1, R8.2
Routing:
- net +3V3: track 67.5 -> 151.3 mm, vias 1 -> 3
- net N$13: track 0.00 -> 63.8 mm, vias 0 -> 2
- net N$9: track 0.00 -> 61.2 mm, vias 0 -> 1
- net N$5: track 0.00 -> 9.03 mm
- net AIOUT1: track 37.2 -> 44.1 mm, vias 0 -> 1
- net AIOUT2: track 36.2 -> 42.8 mm, vias 0 -> 1
- net N$3: track 26.1 -> 20.4 mm
- net VIOUT2: track 0.00 -> 5.22 mm
- net VIOUT1: track 0.00 -> 5.12 mm
- net AIOUT3: track 63.0 -> 67.0 mm, vias 0 -> 1
- net VIOUT: track 8.06 -> 4.91 mm
- net VIN: track 32.1 -> 35.2 mm
- net +5V: track 121.7 -> 122.4 mm
