File: comp-pdu/Comp PDU.sch (EAGLE design)
At the start: 39 parts, among them IC1 788TV, J1 POWER_JACK, K1 RELAY-SPDT-JZC-11F, Q1 BCX70SMD, Q2 SMP3003-DL-1E, Q3 SMP3003-DL-1E, U1 3568

Commit message: updated to new relay to commonly used songle 10A, minor changes to layout.
Parts:
- removed JP4: (no value), pinhead:PINHD-1X2
- removed Q1: BCX70SMD, transistor-npn:BCX70SMD
- removed Q2, Q3: SMP3003-DL-1E, SPEAR:SMP3003-DL-1E
- removed R10, R11: 100k, rcl:R-US_R0805
- removed R9: 1k, rcl:R-US_R0805
- added C7: 10uF, rcl:C-EUC0805
- added D3: (no value), adafruit:DIODEDO-1N4148
- added SWITCH: (no value), pinhead:PINHD-1X1
- D1: value CGRM4004-G -> (none); device diode:CGRM4004-G -> diode:DIODE-DO214AA
- K1: value RELAY-SPDT-JZC-11F -> SRD-05VDC-SL-C; device SparkFun-Electromechanical:RELAY-SPDT-JZC-11F -> SPEAR:SRD-05VDC-SL-C
Connections:
- removed net N$10: Q2.G, R10.2
- removed net N$5: Q3.G, R11.2
- removed net SW: JP4.2, R9.1
- removed net VOUT1: J1.PWR, Q2.S
- removed net VOUT2: J2.2, Q3.S
- net +5V: no longer D1.C
- net GND: now also C7.2, D3.A, K1.A2; no longer JP4.1, Q1.E, R10.1, R11.1
- net N$4: now also D1.C, J2.2; no longer Q1.B, R9.2
- net N$7: now also D3.C, K1.A1, SWITCH.1; no longer D1.A, K1.COIL1, K1.COIL2, Q1.C
- net VBAT: now also K1.COM; no longer K1.MAIN
- net VIOUT: now also C7.1
- net VOUT1_FIXED: now also J1.PWR; no longer Q2.D
- net VOUT2_FIXED: now also D1.A; no longer Q3.D
Other:
- moved on the sheet: D1, J2

Commit message: add connectors for battery monitoring, add more protection to ADC Lines
Parts:
- added C10, C11, C12, C8, C9: 100nF, rcl:C-EUC0805
- added D4: (no value), diode:DIODE-DO-214AC
- added D5, D6, D7, D8, D9: BAT54S, diode:BAT54S
- added JP4: (no value), pinhead:PINHD-1X4
- added R10, R11, R9: 1k, rcl:R-US_R0805
- C7: value 10uF -> 100nF
- D2: value 3.6V -> BAT54S; device SparkFun-DiscreteSemi:DIODE-ZENER-BZT52C3V6S -> diode:BAT54S
- K1: value SRD-05VDC-SL-C -> SRD-24VDC-SL-C
Connections:
- new net N$13: D5.C1A2, JP4.1, R10.1
- new net N$5: D2.C1A2, R7.1, R8.2, R9.1
- new net N$9: D6.C1A2, JP4.4, R11.1
- new net VIOUT1: C8.1, R11.2, U$1.PA4
- new net VIOUT2: C9.1, R10.2, U$1.PA5
- net +3V3: now also D2.C2, D5.C2, D6.C2, D7.C2, D8.C2, D9.C2
- net AIOUT1: now also C10.1, D8.C1A2
- net AIOUT2: now also C11.1, D7.C1A2
- net AIOUT3: now also C12.1, D9.C1A2
- net GND: now also C10.2, C11.2, C12.2, C8.2, C9.2, D2.A1, D4.A, D5.A1, D6.A1, D7.A1, D8.A1, D9.A1, JP4.2, JP4.3; no longer D2.A
- net VIN: now also D4.C; no longer D2.C
- net VIOUT: now also R9.2; no longer R7.1, R8.2
Other:
- moved on the sheet: C7, R4, R5, R6, R7, R8
