File: sub_sys_pdu/sub_sys_pdu.sch (EAGLE design)
At the start: 38 parts, among them Q1 XT60_YELLOW, Q3 XT60_YELLOW

Commit message: fixed schematic, started board
Parts:
- C3, C6: value 100uf -> 100nF; device rcl:CPOL-EUE5-10.5 -> rcl:C-USC0805
Connections:
- net GND: now also C3.2, C6.2; no longer C3.-, C6.-
- net VCC: now also C3.1, C6.1; no longer C3.+, C6.+
Changed lines of the file:
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@@
 <part name="C1" library="rcl" library_urn="urn:adsk.eagle:library:334" deviceset="C-US" device="C0805" package3d_urn="urn:adsk.eagle:package:23617/2" value="100nF"/>
 <part name="C2" library="rcl" library_urn="urn:adsk.eagle:library:334" deviceset="CPOL-EU" device="E5-10.5" package3d_urn="urn:adsk.eagle:package:23372/2" value="100uf"/>
-<part name="C3" library="rcl" library_urn="urn:adsk.eagle:library:334" deviceset="CPOL-EU" device="E5-10.5" package3d_urn="urn:adsk.eagle:package:23372/2" value="100uf"/>
 <part name="Q3" library="XT60_YELLOW" deviceset="XT60_YELLOW" device=""/>
 <part name="C4" library="rcl" library_urn="urn:adsk.eagle:library:334" deviceset="C-US" device="C0805" package3d_urn="urn:adsk.eagle:package:23617/2" value="100nF"/>
 <part name="C5" library="rcl" library_urn="urn:adsk.eagle:library:334" deviceset="CPOL-EU" device="E5-10.5" package3d_urn="urn:adsk.eagle:package:23372/2" value="100uf"/>
-<part name="C6" library="rcl" library_urn="urn:adsk.eagle:library:334" deviceset="CPOL-EU" device="E5-10.5" package3d_urn="urn:adsk.eagle:package:23372/2" value="100uf"/>
 <part name="C7" library="rcl" library_urn="urn:adsk.eagle:library:334" deviceset="C-US" device="C0805" package3d_urn="urn:adsk.eagle:package:23617/2" value="100nF"/>
 <part name="C8" library="rcl" library_urn="urn:adsk.eagle:library:334" deviceset="CPOL-EU" device="E5-10.5" package3d_urn="urn:adsk.eagle:package:23372/2" value="100uf"/>
@@
 <part name="C21" library="rcl" library_urn="urn:adsk.eagle:library:334" deviceset="C-US" device="C0805" package3d_urn="urn:adsk.eagle:package:23617/2" value="100nF"/>
 <part name="C24" library="rcl" library_urn="urn:adsk.eagle:library:334" deviceset="C-US" device="C0805" package3d_urn="urn:adsk.eagle:package:23617/2" value="100nF"/>
+<part name="C3" library="rcl" library_urn="urn:adsk.eagle:library:334" deviceset="C-US" device="C0805" package3d_urn="urn:adsk.eagle:package:23617/2" value="100nF"/>
+<part name="C6" library="rcl" library_urn="urn:adsk.eagle:library:334" deviceset="C-US" device="C0805" package3d_urn="urn:adsk.eagle:package:23617/2" value="100nF"/>
 </parts>
 <sheets>
@@
 <attribute name="VALUE" x="74.803" y="61.4426" size="1.778" layer="96"/>
 </instance>
-<instance part="C3" gate="G$1" x="48.26" y="66.04" smashed="yes">
-<attribute name="NAME" x="49.403" y="66.5226" size="1.778" layer="95"/>
-<attribute name="VALUE" x="49.403" y="61.4426" size="1.778" layer="96"/>
-</instance>
 <instance part="Q3" gate="G$1" x="96.52" y="50.8" smashed="yes">
 <attribute name="NAME" x="93.9562" y="53.3579" size="1.78218125" layer="95"/>
@@
 <attribute name="NAME" x="74.803" y="51.2826" size="1.778" layer="95"/>
 <attribute name="VALUE" x="74.803" y="46.2026" size="1.778" layer="96"/>
-</instance>
-<instance part="C6" gate="G$1" x="48.26" y="50.8" smashed="yes">
-<attribute name="NAME" x="49.403" y="51.2826" size="1.778" layer="95"/>
-<attribute name="VALUE" x="49.403" y="46.2026" size="1.778" layer="96"/>
 </instance>
 <instance part="C7" gate="G$1" x="43.18" y="233.68" smashed="yes">
@@
 <attribute name="NAME" x="31.496" y="114.935" size="1.778" layer="95"/>
 <attribute name="VALUE" x="31.496" y="110.109" size="1.778" layer="96"/>
+</instance>
+<instance part="C3" gate="G$1" x="48.26" y="66.04" smashed="yes">
+<attribute name="NAME" x="49.276" y="66.675" size="1.778" layer="95"/>
+<attribute name="VALUE" x="49.276" y="61.849" size="1.778" layer="96"/>
+</instance>
+<instance part="C6" gate="G$1" x="48.26" y="50.8" smashed="yes">
+<attribute name="NAME" x="49.276" y="51.435" size="1.778" layer="95"/>
+<attribute name="VALUE" x="49.276" y="46.609" size="1.778" layer="96"/>
 </instance>
 </instances>
@@
 <wire x1="73.66" y1="68.58" x2="60.96" y2="68.58" width="0.1524" layer="91"/>
 <junction x="73.66" y="68.58"/>
-<pinref part="C3" gate="G$1" pin="+"/>
 <wire x1="60.96" y1="68.58" x2="48.26" y2="68.58" width="0.1524" layer="91"/>
 <junction x="60.96" y="68.58"/>
+<pinref part="C3" gate="G$1" pin="1"/>
 </segment>
 <segment>
@@
 <wire x1="73.66" y1="53.34" x2="60.96" y2="53.34" width="0.1524" layer="91"/>
 <junction x="73.66" y="53.34"/>
-<pinref part="C6" gate="G$1" pin="+"/>
 <wire x1="60.96" y1="53.34" x2="48.26" y2="53.34" width="0.1524" layer="91"/>
 <junction x="60.96" y="53.34"/>
+<pinref part="C6" gate="G$1" pin="1"/>
 </segment>
 </net>
@@
 <wire x1="91.44" y1="63.5" x2="86.36" y2="63.5" width="0.1524" layer="91"/>
 <label x="86.36" y="63.5" size="1.778" layer="95"/>
-<pinref part="C3" gate="G$1" pin="-"/>
 <pinref part="C1" gate="G$1" pin="2"/>
 <wire x1="48.26" y1="60.96" x2="60.96" y2="60.96" width="0.1524" layer="91"/>
@@
 <junction x="73.66" y="60.96"/>
 <wire x1="86.36" y1="60.96" x2="86.36" y2="63.5" width="0.1524" layer="91"/>
+<pinref part="C3" gate="G$1" pin="2"/>
 </segment>
 <segment>
@@
 <wire x1="91.44" y1="48.26" x2="86.36" y2="48.26" width="0.1524" layer="91"/>
 <label x="86.36" y="48.26" size="1.778" layer="95"/>
-<pinref part="C6" gate="G$1" pin="-"/>
 <pinref part="C4" gate="G$1" pin="2"/>
 <wire x1="48.26" y1="45.72" x2="60.96" y2="45.72" width="0.1524" layer="91"/>
@@
 <junction x="73.66" y="45.72"/>
 <wire x1="86.36" y1="45.72" x2="86.36" y2="48.26" width="0.1524" layer="91"/>
+<pinref part="C6" gate="G$1" pin="2"/>
 </segment>
 </net>

Commit message: submitting for review
Parts:
- removed JP1, JP2, JP3, JP4, JP5, JP6: (no value), pinhead:PINHD-1X2
- added J1, J2, J3, J4, J5, J6: 1017503, 1017503:1017503
Connections:
- removed net GND1: C7.2, C8.-, C9.2, JP1.2
- removed net GND2: C10.2, C11.-, C12.2, JP2.2
- removed net GND3: C13.2, C14.-, C15.2, JP3.2
- removed net GND4: C16.2, C17.-, C18.2, JP4.2
- removed net GND5: C19.2, C20.-, C21.2, JP5.2
- removed net GND6: C22.2, C23.-, C24.2, JP6.2
- removed net N$7: F6.2, JP6.1
- removed net VCC1: C7.1, C8.+, C9.1, F1.1
- removed net VCC2: C10.1, C11.+, C12.1, F2.1
- removed net VCC3: C13.1, C14.+, C15.1, F3.1
- removed net VCC4: C16.1, C17.+, C18.1, F4.1
- removed net VCC5: C19.1, C20.+, C21.1, F5.1
- removed net VCC6: C22.1, C23.+, C24.1, F6.1
- new net N$2: C10.1, C11.+, C12.1, F2.2, J2.3, J2.4
- net GND: now also C10.2, C11.-, C12.2, C13.2, C14.-, C15.2, C16.2, C17.-, C18.2, C19.2, C20.-, C21.2, C22.2, C23.-, C24.2, C7.2, C8.-, C9.2, J1.1, J1.2, J2.1, J2.2, J3.1, J3.2, J4.1, J4.2, J5.1, J5.2, J6.1, J6.2
- net N$1: now also C7.1, C8.+, C9.1, J1.3, J1.4; no longer JP1.1
- net N$3: now also C13.1, C14.+, C15.1, F3.2, J3.3, J3.4; no longer F2.2, JP2.1
- net N$4: now also C16.1, C17.+, C18.1, F4.2, J4.3, J4.4; no longer F3.2, JP3.1
- net N$5: now also C19.1, C20.+, C21.1, F5.2, J5.3, J5.4; no longer F4.2, JP4.1
- net N$6: now also C22.1, C23.+, C24.1, F6.2, J6.3, J6.4; no longer F5.2, JP5.1
- net VCC: now also F1.1, F2.1, F3.1, F4.1, F5.1, F6.1
Other:
- moved on the sheet: C10, C11, C12, C13, C14, C15, C16, C17, C18, C19, C20, C21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
