File: sub_sys_pdu/sub_sys_pdu.brd (EAGLE design)
At the start: 100 x 110 mm, 38 parts, among them Q1 XT60_YELLOW, Q3 XT60_YELLOW

Commit message: submitting for review
Parts:
- removed JP1, JP2, JP3, JP4, JP5, JP6: (no value), pinhead:1X02
- added J1, J2, J3, J4, J5, J6: 1017503, 1017503:1017503
- moved C21 165.8 mm to (95.2, 88.9)
- moved C17 160.6 mm to (87.6, 55.9), turned to 90 degrees
- moved C19 158.8 mm to (95.2, 83.8)
- moved C18 151.5 mm to (95.2, 53.3)
- moved C16 144.9 mm to (95.2, 57.1)
- moved F4 135.6 mm to (73.7, 55.9)
- moved C15 129.5 mm to (72.4, 5.08), turned to 270 degrees
- moved C14 128.4 mm to (69.8, 12.7)
- moved C6 127.0 mm to (62.2, 77.5), turned to 90 degrees
- moved C13 119.4 mm to (67.3, 5.08), turned to 270 degrees
- moved C20 117.4 mm to (87.6, 86.4), turned to 270 degrees
- moved C4 113.4 mm to (54.6, 77.5), turned to 90 degrees
- moved C2 110.0 mm to (44.5, 69.8)
- moved F5 109.8 mm to (73.7, 86.4)
- moved F3 109.4 mm to (69.8, 26.7), turned to 270 degrees
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Connections:
- removed net GND1: C7.2, C8.-, C9.2, JP1.2
- removed net GND2: C10.2, C11.-, C12.2, JP2.2
- removed net GND3: C13.2, C14.-, C15.2, JP3.2
- removed net GND4: C16.2, C17.-, C18.2, JP4.2
- removed net GND5: C19.2, C20.-, C21.2, JP5.2
- removed net GND6: C22.2, C23.-, C24.2, JP6.2
- removed net N$7: F6.2, F6.4, JP6.1
- removed net VCC1: C7.1, C8.+, C9.1, F1.1, F1.3
- removed net VCC2: C10.1, C11.+, C12.1, F2.1, F2.3
- removed net VCC3: C13.1, C14.+, C15.1, F3.1, F3.3
- removed net VCC4: C16.1, C17.+, C18.1, F4.1, F4.3
- removed net VCC5: C19.1, C20.+, C21.1, F5.1, F5.3
- removed net VCC6: C22.1, C23.+, C24.1, F6.1, F6.3
- new net N$2: C10.1, C11.+, C12.1, F2.2, F2.4, J2.3, J2.4
- net GND: now also C10.2, C11.-, C12.2, C13.2, C14.-, C15.2, C16.2, C17.-, C18.2, C19.2, C20.-, C21.2, C22.2, C23.-, C24.2, C7.2, C8.-, C9.2, J1.1, J1.2, J2.1, J2.2, J3.1, J3.2, J4.1, J4.2, J5.1, J5.2, J6.1, J6.2
- net N$1: now also C7.1, C8.+, C9.1, J1.3, J1.4; no longer JP1.1
- net N$3: now also C13.1, C14.+, C15.1, F3.2, F3.4, J3.3, J3.4; no longer F2.2, F2.4, JP2.1
- net N$4: now also C16.1, C17.+, C18.1, F4.2, F4.4, J4.3, J4.4; no longer F3.2, F3.4, JP3.1
- net N$5: now also C19.1, C20.+, C21.1, F5.2, F5.4, J5.3, J5.4; no longer F4.2, F4.4, JP4.1
- net N$6: now also C22.1, C23.+, C24.1, F6.2, F6.4, J6.3, J6.4; no longer F5.2, F5.4, JP5.1
- net VCC: now also F1.1, F1.3, F2.1, F2.3, F3.1, F3.3, F4.1, F4.3, F5.1, F5.3, F6.1, F6.3
Routing:
- added copper zone on layer 16, net GND
- added copper zone on layer 1, net N$1
- added copper zone on layer 1, net N$2
- added copper zone on layer 1, net N$3
- added copper zone on layer 1, net N$4
- added copper zone on layer 1, net N$5
- added copper zone on layer 1, net N$6
- added copper zone on layer 1, net VCC

Commit message: renamed vias to GND and fixed drill size
Changed lines of the file:
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@@
 <vertex x="15.24" y="1.27"/>
 </polygon>
+<via x="-37.846" y="6.35" extent="1-16" drill="0.35" diameter="1.2" shape="square"/>
 <wire x1="96.2" y1="83.82" x2="96.2" y2="88.9" width="0" layer="19" extent="1-1"/>
 <wire x1="87.63" y1="83.82" x2="96.2" y2="83.82" width="0" layer="19" extent="1-1"/>
-<wire x1="54.61" y1="78.42" x2="54.61" y2="69.85" width="0" layer="19" extent="1-1"/>
+<wire x1="39.37" y1="78.42" x2="-37.846" y2="6.35" width="0" layer="19" extent="1-1"/>
+<wire x1="46.99" y1="78.42" x2="-37.846" y2="6.35" width="0" layer="19" extent="1-1"/>
+<wire x1="54.61" y1="78.42" x2="46.99" y2="78.42" width="0" layer="19" extent="1-1"/>
 <wire x1="62.23" y1="78.42" x2="54.61" y2="78.42" width="0" layer="19" extent="1-1"/>
-<wire x1="46.99" y1="78.42" x2="54.61" y2="78.42" width="0" layer="19" extent="1-1"/>
-<wire x1="39.37" y1="78.42" x2="46.99" y2="78.42" width="0" layer="19" extent="1-1"/>
 <wire x1="72.39" y1="4.13" x2="72.39" y2="12.7" width="0" layer="19" extent="1-1"/>
 <wire x1="67.31" y1="4.13" x2="72.39" y2="4.13" width="0" layer="19" extent="1-1"/>
@@
 <wire x1="96.2" y1="57.15" x2="87.63" y2="58.42" width="0" layer="19" extent="1-1"/>
 <wire x1="96.2" y1="53.34" x2="96.2" y2="57.15" width="0" layer="19" extent="1-1"/>
+<via x="4.064" y="72.39" extent="1-16" drill="0.35" diameter="1.2" shape="square"/>
+<via x="-37.846" y="13.97" extent="1-16" drill="0.35" diameter="1.2" shape="square"/>
+<via x="-37.846" y="21.59" extent="1-16" drill="0.35" diameter="1.2" shape="square"/>
+<via x="-37.846" y="29.21" extent="1-16" drill="0.35" diameter="1.2" shape="square"/>
+<via x="4.064" y="67.31" extent="1-16" drill="0.35" diameter="1.2" shape="square"/>
+<via x="4.064" y="41.91" extent="1-16" drill="0.35" diameter="1.2" shape="square"/>
+<via x="4.064" y="36.83" extent="1-16" drill="0.35" diameter="1.2" shape="square"/>
+<via x="36.83" y="4.064" extent="1-16" drill="0.35" diameter="1.2" shape="square"/>
+<via x="41.91" y="4.064" extent="1-16" drill="0.35" diameter="1.2" shape="square"/>
+<via x="67.31" y="4.064" extent="1-16" drill="0.35" diameter="1.2" shape="square"/>
+<via x="72.39" y="4.064" extent="1-16" drill="0.35" diameter="1.2" shape="square"/>
+<via x="96.266" y="53.34" extent="1-16" drill="0.35" diameter="1.2" shape="square"/>
+<via x="96.266" y="57.15" extent="1-16" drill="0.35" diameter="1.2" shape="square"/>
+<via x="96.266" y="83.82" extent="1-16" drill="0.35" diameter="1.2" shape="square"/>
+<via x="96.266" y="88.9" extent="1-16" drill="0.35" diameter="1.2" shape="square"/>
 </signal>
 <signal name="N$6">
@@
 </polygon>
 </signal>
-<signal name="N$7">
-<via x="4.064" y="72.39" extent="1-16" drill="0.2" diameter="1.2" shape="square"/>
-</signal>
-<signal name="N$8">
-<via x="4.064" y="67.31" extent="1-16" drill="0.2" diameter="1.2" shape="square"/>
-</signal>
-<signal name="N$9">
-<via x="4.064" y="41.91" extent="1-16" drill="0.2" diameter="1.2" shape="square"/>
-</signal>
-<signal name="N$10">
-<via x="4.064" y="36.83" extent="1-16" drill="0.2" diameter="1.2" shape="square"/>
-</signal>
-<signal name="N$11">
-<via x="36.83" y="4.064" extent="1-16" drill="0.2" diameter="1.2" shape="square"/>
-</signal>
-<signal name="N$12">
-<via x="41.91" y="4.064" extent="1-16" drill="0.2" diameter="1.2" shape="square"/>
-</signal>
-<signal name="N$13">
-<via x="67.31" y="4.064" extent="1-16" drill="0.2" diameter="1.2" shape="square"/>
-</signal>
-<signal name="N$14">
-<via x="72.39" y="4.064" extent="1-16" drill="0.2" diameter="1.2" shape="square"/>
-</signal>
-<signal name="N$15">
-<via x="96.266" y="53.34" extent="1-16" drill="0.2" diameter="1.2" shape="square"/>
-</signal>
-<signal name="N$16">
-<via x="96.266" y="57.15" extent="1-16" drill="0.2" diameter="1.2" shape="square"/>
-</signal>
-<signal name="N$17">
-<via x="96.266" y="83.82" extent="1-16" drill="0.2" diameter="1.2" shape="square"/>
-</signal>
-<signal name="N$18">
-<via x="96.266" y="88.9" extent="1-16" drill="0.2" diameter="1.2" shape="square"/>
-</signal>
-<signal name="N$19">
-<via x="39.37" y="78.486" extent="1-16" drill="0.2" diameter="1.2" shape="square"/>
-</signal>
-<signal name="N$20">
-<via x="46.99" y="78.486" extent="1-16" drill="0.2" diameter="1.2" shape="square"/>
-</signal>
-<signal name="N$21">
-<via x="54.61" y="78.486" extent="1-16" drill="0.2" diameter="1.2" shape="square"/>
-</signal>
-<signal name="N$22">
-<via x="62.23" y="78.486" extent="1-16" drill="0.2" diameter="1.2" shape="square"/>
-</signal>
 <signal name="N$23">

Commit message: fixed some issues and put board name and author on board
Other:
- board text added: "Jarrett Yu"
- board text added: "SPEAR"
- board text added: "Sub-system PDU 1.0"
Changed lines of the file:
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@@
 <dimension x1="95" y1="105" x2="95" y2="5" x3="105" y3="55" textsize="1.778" layer="1"/>
 <dimension x1="5" y1="5" x2="95" y2="5" x3="50" y3="-5" textsize="1.778" layer="1"/>
+<text x="29.21" y="57.15" size="2.5" layer="25">SPEAR</text>
+<text x="29.21" y="53.34" size="2.5" layer="25">Sub-system PDU 1.0</text>
+<text x="29.21" y="49.53" size="2.5" layer="25">Jarrett Yu</text>
 </plain>
 <attributes>
@@
 <vertex x="15.24" y="1.27"/>
 </polygon>
-<via x="-37.846" y="6.35" extent="1-16" drill="0.35" diameter="1.2" shape="square"/>
-<wire x1="96.2" y1="83.82" x2="96.2" y2="88.9" width="0" layer="19" extent="1-1"/>
-<wire x1="87.63" y1="83.82" x2="96.2" y2="83.82" width="0" layer="19" extent="1-1"/>
-<wire x1="39.37" y1="78.42" x2="-37.846" y2="6.35" width="0" layer="19" extent="1-1"/>
-<wire x1="46.99" y1="78.42" x2="-37.846" y2="6.35" width="0" layer="19" extent="1-1"/>
-<wire x1="54.61" y1="78.42" x2="46.99" y2="78.42" width="0" layer="19" extent="1-1"/>
-<wire x1="62.23" y1="78.42" x2="54.61" y2="78.42" width="0" layer="19" extent="1-1"/>
-<wire x1="72.39" y1="4.13" x2="72.39" y2="12.7" width="0" layer="19" extent="1-1"/>
-<wire x1="67.31" y1="4.13" x2="72.39" y2="4.13" width="0" layer="19" extent="1-1"/>
-<wire x1="4.13" y1="67.31" x2="12.7" y2="67.31" width="0" layer="19" extent="1-1"/>
-<wire x1="4.13" y1="72.39" x2="4.13" y2="67.31" width="0" layer="19" extent="1-1"/>
-<wire x1="41.91" y1="4.13" x2="41.91" y2="12.7" width="0" layer="19" extent="1-1"/>
-<wire x1="36.83" y1="4.13" x2="41.91" y2="4.13" width="0" layer="19" extent="1-1"/>
-<wire x1="4.13" y1="36.83" x2="12.7" y2="36.83" width="0" layer="19" extent="1-1"/>
-<wire x1="4.13" y1="41.91" x2="4.13" y2="36.83" width="0" layer="19" extent="1-1"/>
-<wire x1="96.2" y1="57.15" x2="87.63" y2="58.42" width="0" layer="19" extent="1-1"/>
-<wire x1="96.2" y1="53.34" x2="96.2" y2="57.15" width="0" layer="19" extent="1-1"/>
+<via x="39.37" y="78.486" extent="1-16" drill="0.35" diameter="1.2" shape="square"/>
 <via x="4.064" y="72.39" extent="1-16" drill="0.35" diameter="1.2" shape="square"/>
-<via x="-37.846" y="13.97" extent="1-16" drill="0.35" diameter="1.2" shape="square"/>
-<via x="-37.846" y="21.59" extent="1-16" drill="0.35" diameter="1.2" shape="square"/>
-<via x="-37.846" y="29.21" extent="1-16" drill="0.35" diameter="1.2" shape="square"/>
+<via x="46.99" y="78.486" extent="1-16" drill="0.35" diameter="1.2" shape="square"/>
+<via x="54.61" y="78.486" extent="1-16" drill="0.35" diameter="1.2" shape="square"/>
+<via x="62.23" y="78.486" extent="1-16" drill="0.35" diameter="1.2" shape="square"/>
 <via x="4.064" y="67.31" extent="1-16" drill="0.35" diameter="1.2" shape="square"/>
 <via x="4.064" y="41.91" extent="1-16" drill="0.35" diameter="1.2" shape="square"/>
@@
 <via x="96.266" y="83.82" extent="1-16" drill="0.35" diameter="1.2" shape="square"/>
 <via x="96.266" y="88.9" extent="1-16" drill="0.35" diameter="1.2" shape="square"/>
+<wire x1="96.266" y1="88.9" x2="96.2" y2="88.9" width="0" layer="19" extent="1-1"/>
+<wire x1="96.2" y1="83.82" x2="96.266" y2="83.82" width="0" layer="19" extent="1-1"/>
+<wire x1="96.2" y1="57.15" x2="96.266" y2="57.15" width="0" layer="19" extent="1-1"/>
+<wire x1="96.2" y1="53.34" x2="96.266" y2="53.34" width="0" layer="19" extent="1-1"/>
+<wire x1="62.23" y1="78.42" x2="62.23" y2="78.486" width="0" layer="19" extent="1-1"/>
+<wire x1="54.61" y1="78.42" x2="54.61" y2="78.486" width="0" layer="19" extent="1-1"/>
+<wire x1="46.99" y1="78.42" x2="46.99" y2="78.486" width="0" layer="19" extent="1-1"/>
+<wire x1="39.37" y1="78.42" x2="39.37" y2="78.486" width="0" layer="19" extent="1-1"/>
+<wire x1="4.13" y1="72.39" x2="4.064" y2="72.39" width="0" layer="19" extent="1-1"/>
+<wire x1="72.39" y1="4.13" x2="72.39" y2="4.064" width="0" layer="19" extent="1-1"/>
+<wire x1="4.13" y1="67.31" x2="4.064" y2="67.31" width="0" layer="19" extent="1-1"/>
+<wire x1="67.31" y1="4.13" x2="67.31" y2="4.064" width="0" layer="19" extent="1-1"/>
+<wire x1="4.13" y1="41.91" x2="4.064" y2="41.91" width="0" layer="19" extent="1-1"/>
+<wire x1="41.91" y1="4.13" x2="41.91" y2="4.064" width="0" layer="19" extent="1-1"/>
+<wire x1="4.13" y1="36.83" x2="4.064" y2="36.83" width="0" layer="19" extent="1-1"/>
+<wire x1="36.83" y1="4.13" x2="36.83" y2="4.064" width="0" layer="19" extent="1-1"/>
 </signal>
 <signal name="N$6">
