File: Inertial_measurement_unit/IMU.brd (EAGLE design)
At the start: 21.3 x 53.7 mm, 16 parts, among them IC1 BNO055, Y1 ECS-.327-12.5-39-TR

Commit message: Fixed traces, added BOM
Parts:
- added R2: 10K, resistor:R0805
- moved R3 0.28 mm to (35.0, 15.0)
Connections:
- new net NBOOT: IC1.4, R2.1
- net +3V3: now also R2.2; no longer IC1.4
Routing:
- net NBOOT: track 0.00 -> 12.9 mm, vias 0 -> 2
- net +3V3: track 60.6 -> 70.3 mm, vias 4 -> 6
- net UART_CTS: track 25.2 -> 28.9 mm
- net NRESET: track 32.9 -> 30.9 mm
- net SCL: track 30.3 -> 32.1 mm, vias 2 -> 0
- net UART_RTS: track 29.5 -> 27.8 mm
- net UART_TX: track 39.7 -> 38.1 mm
- net UART_RX: track 34.0 -> 35.2 mm
- net SDA: track 38.4 -> 37.4 mm
- added copper zone on layer 16, net GND
