File: main-pdu/Main PDU.brd (EAGLE design)
At the start: 100 x 70 mm, 37 parts, among them J1 VCF4-1000, J2 VCF4-1000

Commit message: added minh's revisions to pdu
Parts:
- added U1, U2, U3, U4, U5, U6: 3568, LCSC:3568
- moved D2 26.1 mm to (47.2, 49.5)
- moved C4 26.0 mm to (39.5, 80.5)
- moved PS2 26.0 mm to (36.3, 80.5)
- moved R10 26.0 mm to (8.00, 72.7)
- moved R6 26.0 mm to (16.1, 72.7)
- moved R7 26.0 mm to (14.1, 72.7)
- moved R8 26.0 mm to (12.1, 72.7)
- moved R9 26.0 mm to (10.0, 72.7)
- moved D1 26.0 mm to (52.1, 49.4)
- moved SWITCH 26.0 mm to (2.03, 53.1)
- moved C1 26.0 mm to (75.9, 80.6)
- moved C10 26.0 mm to (9.65, 48.9)
- moved C11 26.0 mm to (78.6, 71.0)
- moved C3 26.0 mm to (78.2, 80.6)
- moved C5 26.0 mm to (48.5, 79.3)
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Connections:
- new net N$11: U$8.+, U1.1, U1.2
- new net N$12: U$4.+, U6.1, U6.2
- new net N$13: U$10.+, U3.1, U3.2
- new net N$15: U$7.+, U2.1, U2.2
- new net N$16: U$3.+, U5.1, U5.2
- new net N$18: U$6.+, U4.1, U4.2
- net REG1: now also U4.3, U4.4, U5.3, U5.4, U6.3, U6.4; no longer U$3.+, U$4.+, U$6.+
- net REG2: now also U1.3, U1.4, U2.3, U2.4, U3.3, U3.4; no longer U$10.+, U$7.+, U$8.+
Routing:
- added copper zone on layer 1, net N$11
- added copper zone on layer 1, net N$12
- added copper zone on layer 1, net N$13
- added copper zone on layer 1, net N$15
- added copper zone on layer 1, net N$16
- added copper zone on layer 1, net N$18
Other:
- board size 100 x 70 mm -> 100 x 96 mm
