File: main-pdu/Main PDU.sch (EAGLE design)
At the start: 37 parts, among them J1 VCF4-1000, J2 VCF4-1000

Commit message: added minh's revisions to pdu
Parts:
- added U1, U2, U3, U4, U5, U6: 3568, LCSC:3568
Connections:
- new net N$11: U$8.VCC, U1.1, U1.2
- new net N$12: U$4.VCC, U6.1, U6.2
- new net N$13: U$10.VCC, U3.1, U3.2
- new net N$15: U$7.VCC, U2.1, U2.2
- new net N$16: U$3.VCC, U5.1, U5.2
- new net N$18: U$6.VCC, U4.1, U4.2
- net REG1: now also U4.3, U4.4, U5.3, U5.4, U6.3, U6.4; no longer U$3.VCC, U$4.VCC, U$6.VCC
- net REG2: now also U1.3, U1.4, U2.3, U2.4, U3.3, U3.4; no longer U$10.VCC, U$7.VCC, U$8.VCC
