File: kicad/speedy-breakout/speedy-breakout.kicad_sch (KiCad schematic)
At the start: 9 parts, among them J1 Pin Socket 1x20, J2 Pin Socket 1x20, J3 Molex Mini-Lock 53426, J4 Molex Mini-Lock 53426, J5 CUI TLB009-254, J6 CUI TBL009-254, J7 Conn_01x02

Commit message: speedy-breakout: Complete Rev 1.0 Schematics/Layout
Parts:
- R1: footprint (none) -> Resistor_SMD:R_0805_2012Metric_Pad1.20x1.40mm_HandSolder
Connections:
- net CAN_H is gone; now on net CANL: R1.1
- net CAN_L is gone; now on an unnamed net: J7.2 (Pin_2)
- net CANH: now also J7.1 (Pin_1)
- net PA0: now also J6.2 (Pin_2)
- net PA1: now also J6.1 (Pin_1)
- net PA2: now also J5.2 (Pin_2)
- net PA3: now also J5.1 (Pin_1)
- net at R1.2: no longer J7.1 (Pin_1)
- net OSC32_OUT: now reaches J2.17 (Pin_17)
- net OSC32_IN: now reaches J2.18 (Pin_18)
- no-connect marks 0 -> 28
Other:
- note added: "Motor 1 Direction"
- note added: "Motor 1 PWM/Step"
- note added: "Motor 2 Direction"
- note added: "Motor 2 PWM/Step"
- note added: "Motor driver interface"
- note removed: "Motor controllers"
- moved on the sheet: D1, J1, J2, J3, J4, J5, J6, J7, R1

Commit message: speedy-breakout: Add headers for feedback expansion
This consists of a footprint for an arbitrary 2.54 mm connector, with
traces to another header which can be used to easily solder wires to
make arbitrary connections to the Speedy breakout through-holes
depending on the desired application. A 6 pin footprint was used which
should give enough for power + ground and up to a full 4 pin SPI
interface. Pin 6 is tied to ground.
Parts:
- added J10, J11, J8, J9: Conn_01x06, Connector_PinHeader_2.54mm:PinHeader_1x06_P2.54mm_Vertical, symbol Connector_Generic:Conn_01x06
Connections:
- net GND: now also J10.6 (Pin_6), J11.6 (Pin_6), J8.6 (Pin_6), J9.6 (Pin_6)
- new net: J10.1 (Pin_1), J8.1 (Pin_1)
- new net: J10.2 (Pin_2), J8.2 (Pin_2)
- new net: J10.3 (Pin_3), J8.3 (Pin_3)
- new net: J10.4 (Pin_4), J8.4 (Pin_4)
- new net: J10.5 (Pin_5), J8.5 (Pin_5)
- new net: J11.1 (Pin_1), J9.1 (Pin_1)
- new net: J11.2 (Pin_2), J9.2 (Pin_2)
- new net: J11.3 (Pin_3), J9.3 (Pin_3)
- new net: J11.4 (Pin_4), J9.4 (Pin_4)
- new net: J11.5 (Pin_5), J9.5 (Pin_5)
Other:
- note added: "Expansion headers"
- moved on the sheet: D1, J1, J2, J3, J4, J5, J6, J7, R1
